File: hardware/sensor_board/sensor_board.sch (KiCad schematic (older format))
At the start: 72 parts

Commit message: sendor_board bigger controller
Parts:
- removed IC?: ATMEGA328P-A, TQFP32, symbol ATMEGA328P-A
- removed P?: SPI, ~, symbol CONN_4
- added D?: LED2, ~, symbol LED
- added D?: LED3, ~, symbol LED
- added IC?: ATMEGA164P-A, TQFP44, symbol ATMEGA164P-A
- added J? (x5): RJ45, ~, symbol RJ45
- added K?: I2C, ~, symbol CONN_3
- added P?: SPI, ~, symbol CONN_5
- added P?: 5Vin, ~, symbol CONN_2
- added R? (x2): R, ~, symbol R
- added R? (x5): 120, ~, symbol R
- added R? (x10): 1k, ~, symbol R
- added U? (x5): ST485, ~, symbol ST485
- D?: value LED_DEBUG -> LED1
- P?: value POWER -> 12Vin
Connections:
- net labels added: LED1, LED2, LED3, SCL, SDA, SS, ZAC_12, ZAC_13, ZAC_14, ZAC_15, ZAC_16
- wire segments 331 -> 479
Other:
- moved on the sheet: C?, D?, K?, P?, R?, SW?, U?, X?

Commit message: sensor board: led fix
Parts:
- added R? (x4): 150, ~, symbol R
- C?: value C -> 100n
- R?: value R -> 10k
- R? (x2): value R -> 2k2
- X?: value CRYSTAL -> 20MHz
Connections:
- wire segments 479 -> 483
Other:
- moved on the sheet: D?
Changed lines of the file:
@@
 Sheet 1 1
 Title ""
-Date "23 mar 2014"
+Date "24 mar 2014"
 Rev ""
 Comp ""
@@
 P 2650 1850
 F 0 "C?" H 2650 1950 40  0000 L CNN
-F 1 "C" H 2656 1765 40  0000 L CNN
+F 1 "100n" H 2656 1765 40  0000 L CNN
 F 2 "~" H 2688 1700 30  0000 C CNN
 F 3 "~" H 2650 1850 60  0000 C CNN
@@
 P 1900 3250
 F 0 "X?" H 1900 3400 60  0000 C CNN
-F 1 "CRYSTAL" H 1900 3100 60  0000 C CNN
+F 1 "20MHz" H 1900 3100 60  0000 C CNN
 F 2 "~" H 1900 3250 60  0000 C CNN
 F 3 "~" H 1900 3250 60  0000 C CNN
@@
 P 4050 8000
 F 0 "R?" V 4130 8000 40  0000 C CNN
-F 1 "R" V 4057 8001 40  0000 C CNN
+F 1 "10k" V 4057 8001 40  0000 C CNN
 F 2 "~" V 3980 8000 30  0000 C CNN
 F 3 "~" H 4050 8000 30  0000 C CNN
@@
 L VCC #PWR?
 U 1 1 532E062B
-P 3900 11400
-F 0 "#PWR?" H 3900 11500 30  0001 C CNN
-F 1 "VCC" H 3900 11500 30  0000 C CNN
-F 2 "" H 3900 11400 60  0000 C CNN
-F 3 "" H 3900 11400 60  0000 C CNN
-	1    3900 11400
+P 3200 11400
+F 0 "#PWR?" H 3200 11500 30  0001 C CNN
+F 1 "VCC" H 3200 11500 30  0000 C CNN
+F 2 "" H 3200 11400 60  0000 C CNN
+F 3 "" H 3200 11400 60  0000 C CNN
+	1    3200 11400
 	1    0    0    -1
 $EndComp
@@
 Connection ~ 5000 10500
 Wire Wire Line
-	3900 11400 3900 11500
-Wire Wire Line
 	3900 11500 4150 11500
 Wire Wire Line
@@
 L LED D?
 U 1 1 532E0BA2
-P 3400 13750
-F 0 "D?" H 3400 13850 50  0000 C CNN
-F 1 "LED1" H 3400 13650 50  0000 C CNN
-F 2 "~" H 3400 13750 60  0000 C CNN
-F 3 "~" H 3400 13750 60  0000 C CNN
-	1    3400 13750
+P 3100 13500
+F 0 "D?" H 3100 13600 50  0000 C CNN
+F 1 "LED1" H 3100 13400 50  0000 C CNN
+F 2 "~" H 3100 13500 60  0000 C CNN
+F 3 "~" H 3100 13500 60  0000 C CNN
+	1    3100 13500
 	-1   0    0    1
 $EndComp
@@
 L VCC #PWR?
 U 1 1 532E0C50
-P 3950 13650
-F 0 "#PWR?" H 3950 13750 30  0001 C CNN
-F 1 "VCC" H 3950 13750 30  0000 C CNN
-F 2 "" H 3950 13650 60  0000 C CNN
-F 3 "" H 3950 13650 60  0000 C CNN
-	1    3950 13650
+P 4300 13400
+F 0 "#PWR?" H 4300 13500 30  0001 C CNN
+F 1 "VCC" H 4300 13500 30  0000 C CNN
+F 2 "" H 4300 13400 60  0000 C CNN
+F 3 "" H 4300 13400 60  0000 C CNN
+	1    4300 13400
 	1    0    0    -1
 $EndComp
-Wire Wire Line
-	3950 13650 3950 13750
-Wire Wire Line
-	3950 13750 3600 13750
 $Comp
 L ST485 U?
@@
 P 2400 9700
 F 0 "R?" V 2480 9700 40  0000 C CNN
-F 1 "R" V 2407 9701 40  0000 C CNN
+F 1 "2k2" V 2407 9701 40  0000 C CNN
 F 2 "~" V 2330 9700 30  0000 C CNN
 F 3 "~" H 2400 9700 30  0000 C CNN
@@
 P 2600 9700
 F 0 "R?" V 2680 9700 40  0000 C CNN
-F 1 "R" V 2607 9701 40  0000 C CNN
+F 1 "2k2" V 2607 9701 40  0000 C CNN
 F 2 "~" V 2530 9700 30  0000 C CNN
 F 3 "~" H 2600 9700 30  0000 C CNN
@@
 Text Label 4800 3250 2    60   ~ 0
 LED3
-Text Label 2850 13750 0    60   ~ 0
+Text Label 2550 13500 0    60   ~ 0
 LED1
 Wire Wire Line
-	2850 13750 3200 13750
+	2550 13500 2900 13500
 $Comp
 L LED D?
 U 1 1 532EDB27
-P 3400 14050
-F 0 "D?" H 3400 14150 50  0000 C CNN
-F 1 "LED2" H 3400 13950 50  0000 C CNN
-F 2 "~" H 3400 14050 60  0000 C CNN
-F 3 "~" H 3400 14050 60  0000 C CNN
-	1    3400 14050
+P 3100 13800
+F 0 "D?" H 3100 13900 50  0000 C CNN
+F 1 "LED2" H 3100 13700 50  0000 C CNN
+F 2 "~" H 3100 13800 60  0000 C CNN
+F 3 "~" H 3100 13800 60  0000 C CNN
+	1    3100 13800
 	-1   0    0    1
 $EndComp
@@
 L VCC #PWR?
 U 1 1 532EDB2D
-P 3950 13950
-F 0 "#PWR?" H 3950 14050 30  0001 C CNN
-F 1 "VCC" H 3950 14050 30  0000 C CNN
-F 2 "" H 3950 13950 60  0000 C CNN
-F 3 "" H 3950 13950 60  0000 C CNN
-	1    3950 13950
+P 4300 13700
+F 0 "#PWR?" H 4300 13800 30  0001 C CNN
+F 1 "VCC" H 4300 13800 30  0000 C CNN
+F 2 "" H 4300 13700 60  0000 C CNN
+F 3 "" H 4300 13700 60  0000 C CNN
+	1    4300 13700
 	1    0    0    -1
 $EndComp
 Wire Wire Line
-	3950 13950 3950 14050
-Wire Wire Line
-	3950 14050 3600 14050
-Wire Wire Line
-	2850 14050 3200 14050
+	2550 13800 2900 13800
 $Comp
 L LED D?
 U 1 1 532EDB3C
-P 3400 14350
-F 0 "D?" H 3400 14450 50  0000 C CNN
-F 1 "LED3" H 3400 14250 50  0000 C CNN
-F 2 "~" H 3400 14350 60  0000 C CNN
-F 3 "~" H 3400 14350 60  0000 C CNN
-	1    3400 14350
+P 3100 14100
+F 0 "D?" H 3100 14200 50  0000 C CNN
+F 1 "LED3" H 3100 14000 50  0000 C CNN
+F 2 "~" H 3100 14100 60  0000 C CNN
+F 3 "~" H 3100 14100 60  0000 C CNN
+	1    3100 14100
 	-1   0    0    1
 $EndComp
@@
 L VCC #PWR?
 U 1 1 532EDB42
-P 3950 14250
-F 0 "#PWR?" H 3950 14350 30  0001 C CNN
-F 1 "VCC" H 3950 14350 30  0000 C CNN
-F 2 "" H 3950 14250 60  0000 C CNN
-F 3 "" H 3950 14250 60  0000 C CNN
-	1    3950 14250
+P 4300 14000
+F 0 "#PWR?" H 4300 14100 30  0001 C CNN
+F 1 "VCC" H 4300 14100 30  0000 C CNN
+F 2 "" H 4300 14000 60  0000 C CNN
+F 3 "" H 4300 14000 60  0000 C CNN
+	1    4300 14000
 	1    0    0    -1
 $EndComp
 Wire Wire Line
-	3950 14250 3950 14350
-Wire Wire Line
-	3950 14350 3600 14350
-Wire Wire Line
-	2850 14350 3200 14350
-Text Label 2850 14050 0    60   ~ 0
+	2550 14100 2900 14100
+Text Label 2550 13800 0    60   ~ 0
 LED2
-Text Label 2850 14350 0    60   ~ 0
+Text Label 2550 14100 0    60   ~ 0
 LED3
 Wire Wire Line
@@
 	19150 11350 19000 11350
 Connection ~ 19000 11350
+$Comp
+L R R?
+U 1 1 53302FA3
+P 3800 13500
+F 0 "R?" V 3880 13500 40  0000 C CNN
+F 1 "150" V 3807 13501 40  0000 C CNN
+F 2 "~" V 3730 13500 30  0000 C CNN
+F 3 "~" H 3800 13500 30  0000 C CNN
+	1    3800 13500
+	0    -1   -1   0
+$EndComp
+$Comp
+L R R?
+U 1 1 53302FB0
+P 3800 13800
+F 0 "R?" V 3880 13800 40  0000 C CNN
+F 1 "150" V 3807 13801 40  0000 C CNN
+F 2 "~" V 3730 13800 30  0000 C CNN
+F 3 "~" H 3800 13800 30  0000 C CNN
+	1    3800 13800
+	0    -1   -1   0
+$EndComp
+$Comp
+L R R?
+U 1 1 53302FB6
+P 3800 14100
+F 0 "R?" V 3880 14100 40  0000 C CNN
+F 1 "150" V 3807 14101 40  0000 C CNN
+F 2 "~" V 3730 14100 30  0000 C CNN
+F 3 "~" H 3800 14100 30  0000 C CNN
+	1    3800 14100
+	0    -1   -1   0
+$EndComp
+Wire Wire Line
+	3300 13500 3550 13500
+Wire Wire Line
+	3300 13800 3550 13800
+Wire Wire Line
+	3300 14100 3550 14100
+Wire Wire Line
+	4050 14100 4300 14100
+Wire Wire Line
+	4300 14100 4300 14000
+Wire Wire Line
+	4050 13800 4300 13800
+Wire Wire Line
+	4300 13800 4300 13700
+Wire Wire Line
+	4050 13500 4300 13500
+Wire Wire Line
+	4300 13500 4300 13400
+$Comp
+L R R?
+U 1 1 533043ED
+P 3650 11500
+F 0 "R?" V 3730 11500 40  0000 C CNN
+F 1 "150" V 3657 11501 40  0000 C CNN
+F 2 "~" V 3580 11500 30  0000 C CNN
+F 3 "~" H 3650 11500 30  0000 C CNN
+	1    3650 11500
+	0    -1   -1   0
+$EndComp
+Wire Wire Line
+	3200 11400 3200 11500
+Wire Wire Line
+	3200 11500 3400 11500
 $EndSCHEMATC

Commit message: sensor_board updated
Parts:
- added J? (x2): RJ45, ~, symbol RJ45
- added R? (x2): 120, ~, symbol R
- added R? (x4): 1k, ~, symbol R
- added U? (x2): ST485, ~, symbol ST485
Connections:
- net labels added: ZAC_17, ZAC_18
- wire segments 483 -> 529

Commit message: hardware + bestellungen
Parts:
- removed C?: 100n, ~, symbol C
- removed C? (x2): C, ~, symbol C
- removed D?: LED3, ~, symbol LED
- removed IC?: ATMEGA164P-A, TQFP44, symbol ATMEGA164P-A
- removed J? (x17): RJ45, ~, symbol RJ45
- removed K?: POW_sel, ~, symbol CONN_3
- removed P?: SPI, ~, symbol CONN_5
- removed R? (x17): 120, ~, symbol R
- removed R? (x34): 1k, ~, symbol R
- removed R?: 150, ~, symbol R
- removed U? (x17): ST485, ~, symbol ST485
- removed X?: 20MHz, ~, symbol CRYSTAL
- added C? (x2): C, ~, symbol C
- added C? (x2): 100n, ~, symbol C
- added IC?: ATMEGA88A-A, TQFP32, symbol ATMEGA88A-A
- added K?: I2C, ~, symbol CONN_3
- added P?: I2C_pull_enable, ~, symbol CONN_2X2
- added P?: 5Vin, ~, symbol CONN_2
- added X?: 20MHz, ~, symbol CRYSTAL
- R? (x2): value 1k -> 22k
Connections:
- net labels added: XTAL1, XTAL2
- net labels removed: LED3, SS, Vsup, ZAC_11, ZAC_12, ZAC_13, ZAC_14, ZAC_15, ZAC_16, ZAC_17, ZAC_18
- wire segments 529 -> 142
Other:
- moved on the sheet: C?, D?, K?, P?, R?, SW?, U?

Commit message: schematic sensor board
Parts:
- removed J?: RJ45, ~, symbol RJ45
- removed K? (x2): I2C, ~, symbol CONN_3
- removed P?: 5Vin, ~, symbol CONN_2
- removed P?: I2C_pull_enable, ~, symbol CONN_2X2
- removed U?: ST485, ~, symbol ST485
- added C? (x7): 100n, ~, symbol C
- added J?: RJ45_8P8C_8FACH, ~, symbol RJ45_8P8C_8FACH
- added K?: pow_sel, ~, symbol CONN_3
- added P?: HOHLBUCHSE, ~, symbol HOHLBUCHSE
- added P?: i2c_pow, ~, symbol CONN_3X2
- added P?: i2c_chain, ~, symbol CONN_3X2
- added P?: Shield, ~, symbol CONN_1
- added R? (x7): 120, ~, symbol R
- added R? (x14): 22k, ~, symbol R
- added SW?: SCHALTER_2POL, ~, symbol SCHALTER_2POL
- added U? (x8): ST485, ~, symbol ST485
- C? (x2): value C -> 22p
Connections:
- net labels added: Vi2c, Vreg
- net labels removed: ZAC_09, ZAC_10
- wire segments 142 -> 335
- no-connect marks 0 -> 1
Other:
- moved on the sheet: C?, D?, P?, R?, U?

Commit message: modules
Parts:
- removed J?: RJ45_8P8C_8FACH, ~, symbol RJ45_8P8C_8FACH
- added J?: RJ45_8P8C_8FACH, ~, symbol RJ45_8P8C_8FACH
Connections:
- wire segments 335 -> 425

Commit message: 7805 schematic library
Parts:
- removed U?: LM7805, ~, symbol LM7805
- added C?: 10u, ~, symbol C
- added C? (x8): 100n, ~, symbol C
- added D?: LED1, ~, symbol LED
- added D?: LED2, ~, symbol LED
- added P?: 5Vin, ~, symbol CONN_2
- added R?: 10k, ~, symbol R
- added R? (x2): 150, ~, symbol R
- added SW?: SW1, ~, symbol SW_PUSH
- added U?: LM7805, ~, symbol 7805_CORRECT_PINS
- SW?: value SW_PUSH -> SW_RESET
Connections:
- net labels added: LED3, LED4, SW1
- wire segments 425 -> 466
Other:
- moved on the sheet: P?

Commit message: board started
Parts:
- P7: renamed from P?; value 5Vin -> Vccin
- gave numbers to parts that had none: 84
Connections:
- net labels added: z1a, z1b, z2a, z2b, z3a, z3b, z4a, z4b, z5a, z5b, z6a, z6b, z7a, z7b, z8a, z8b
- wire segments 466 -> 450
