File: hardware/sensor_board/sensor_board.sch (KiCad schematic (older format))
At the start: 85 parts, among them IC1 ATMEGA88A-A, J1 RJ45_8P8C_8FACH, K1 pow_sel, P1 UART, P2 Shield, P3 i2c_pow, P4 i2c_chain, P5 12Vin, P6 HOHLBUCHSE, P7 Vccin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

Commit message: sensor board pcb routing started
Parts:
- D3: value LED1 -> LED3
- D4: value LED2 -> LED4
Connections:
- wire segments 450 -> 358

Commit message: fixed unconnected zac wire
Changed lines of the file:
@@
 z8a
 Wire Wire Line
-	18150 3400 18600 3400
+	18125 3400 18600 3400
 Wire Wire Line
 	18600 3500 18125 3500

Commit message: sensor_board complete
Parts:
- added C23, C24: 10u, ~, symbol C
- added C25, C26, C27, C28, C29, C30, C31, C32: 100n, ~, symbol C
- added R34: 0, ~, symbol R
Connections:
- wire segments 358 -> 379
Other:
- moved on the sheet: P2

Commit message: report schematic images
Connections:
- wire segments 379 -> 471
Other:
- moved on the sheet: C10, C11, C12, C13, C14, C15, C16, C17, C18, C19, C20, C21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
