File: hardware/sensor_board/sensor_board.kicad_pcb (KiCad board)
At the start: 2 copper layers, 65 x 137 mm, 99 parts, among them IC1 ATMEGA88A-A, J1 RJ45_8P8C_8FACH, K1 pow_sel, P1 UART, P2 Shield, P3 i2c_pow, P4 i2c_chain, P5 12Vin, P6 HOHLBUCHSE, P7 Vccin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

Commit message: finalized boards for production
Routing:
- net GND: track 884.0 -> 883.2 mm
Changed lines of the file:
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@@
     (links 278)
     (no_connects 0)
-    (area 190 34.150001 281.714285 190.000001)
+    (area 190 34.150001 287.214286 190.000001)
     (thickness 1.6)
-    (drawings 17)
-    (tracks 1182)
+    (drawings 15)
+    (tracks 1183)
     (zones 0)
     (modules 99)
@@
     )
   )
-  (dimension 137 (width 0.3) (layer Cmts.User)
-    (gr_text "137.000 mm" (at 279.85 112.5 90) (layer Cmts.User)
-      (effects (font (size 1.5 1.5) (thickness 0.3)))
-    )
-    (feature1 (pts (xy 263 44) (xy 281.2 44)))
-    (feature2 (pts (xy 263 181) (xy 281.2 181)))
-    (crossbar (pts (xy 278.5 181) (xy 278.5 44)))
-    (arrow1a (pts (xy 278.5 44) (xy 279.08642 45.126503)))
-    (arrow1b (pts (xy 278.5 44) (xy 277.91358 45.126503)))
-    (arrow2a (pts (xy 278.5 181) (xy 279.08642 179.873497)))
-    (arrow2b (pts (xy 278.5 181) (xy 277.91358 179.873497)))
-  )
-  (gr_line (start 197 181) (end 197 44) (angle 90) (layer Edge.Cuts) (width 0.1))
-  (gr_line (start 262 181) (end 197 181) (angle 90) (layer Edge.Cuts) (width 0.1))
-  (gr_line (start 262 44) (end 262 181) (angle 90) (layer Edge.Cuts) (width 0.1))
-  (gr_line (start 197 44) (end 262 44) (angle 90) (layer Edge.Cuts) (width 0.1))
+  (gr_line (start 262 181) (end 262 44) (angle 90) (layer Edge.Cuts) (width 0.1))
+  (gr_line (start 197 181) (end 262 181) (angle 90) (layer Edge.Cuts) (width 0.1))
+  (gr_line (start 197 44) (end 197 181) (angle 90) (layer Edge.Cuts) (width 0.1))
+  (gr_line (start 262 44) (end 197 44) (angle 90) (layer Edge.Cuts) (width 0.1))
   (gr_text v1.0 (at 246 179.5) (layer F.Cu)
     (effects (font (size 1.5 1.5) (thickness 0.3)))
@@
     (effects (font (size 1.5 1.5) (thickness 0.3)))
   )
-  (dimension 65 (width 0.3) (layer Cmts.User)
-    (gr_text "65.000 mm" (at 229.5 35.650001) (layer Cmts.User)
-      (effects (font (size 1.5 1.5) (thickness 0.3)))
-    )
-    (feature1 (pts (xy 197 41) (xy 197 34.300001)))
-    (feature2 (pts (xy 262 41) (xy 262 34.300001)))
-    (crossbar (pts (xy 262 37.000001) (xy 197 37.000001)))
-    (arrow1a (pts (xy 197 37.000001) (xy 198.126503 36.413581)))
-    (arrow1b (pts (xy 197 37.000001) (xy 198.126503 37.586421)))
-    (arrow2a (pts (xy 262 37.000001) (xy 260.873497 36.413581)))
-    (arrow2b (pts (xy 262 37.000001) (xy 260.873497 37.586421)))
-  )
   (segment (start 202 72.73) (end 206.77 72.73) (width 0.7) (layer B.Cu) (net 1))
   (segment (start 217.5 64) (end 217.5 61.8) (width 0.7) (layer B.Cu) (net 1))
@@
   (segment (start 241 65.5) (end 242.676 67.176) (width 0.7) (layer F.Cu) (net 42))
   (segment (start 242.676 67.176) (end 245.7296 67.176) (width 0.7) (layer F.Cu) (net 42) (status 20))
+  (segment (start 210.1 140.9) (end 210.1 139.8) (width 0.7) (layer F.Cu) (net 43))
+  (via (at 210.1 139.8) (size 1.2) (layers F.Cu B.Cu) (net 43))
   (segment (start 259.5296 170.326) (end 259.5296 158.5296) (width 0.7) (layer B.Cu) (net 43))
   (segment (start 257 156) (end 252.3 156) (width 0.7) (layer B.Cu) (net 43))
@@
   (segment (start 226.755 157.445) (end 226.755 159.2) (width 0.7) (layer F.Cu) (net 43))
   (segment (start 228.25 155.95) (end 226.755 157.445) (width 0.7) (layer F.Cu) (net 43))
-  (segment (start 210 140.9) (end 210 139) (width 0.7) (layer F.Cu) (net 43))
-  (via (at 210 139) (size 1.2) (layers F.Cu B.Cu) (net 43))
   (segment (start 244.4796 126.956) (end 252.3 126.956) (width 0.7) (layer B.Cu) (net 43))
   (segment (start 252.3 126.956) (end 252.3 126.9) (width 0.7) (layer B.Cu) (net 43))
@@
   (segment (start 204.6 145.5) (end 203.27 145.5) (width 0.7) (layer F.Cu) (net 43))
   (segment (start 209.2 140.9) (end 204.6 145.5) (width 0.7) (layer F.Cu) (net 43))
-  (segment (start 210.2 140.9) (end 210 140.9) (width 0.7) (layer F.Cu) (net 43))
+  (segment (start 210.2 140.9) (end 210.1 140.9) (width 0.7) (layer F.Cu) (net 43))
+  (segment (start 210.1 140.9) (end 210 140.9) (width 0.7) (layer F.Cu) (net 43))
   (segment (start 210 140.9) (end 209.2 140.9) (width 0.7) (layer F.Cu) (net 43))
   (segment (start 210.6 141.3) (end 210.2 140.9) (width 0.7) (layer F.Cu) (net 43))
@@
     (polygon
       (pts
-        (xy 265 185) (xy 195 185) (xy 195 40) (xy 265 40)
+        (xy 262 181) (xy 197 181) (xy 197 44) (xy 262 44)
       )
     )
@@
     (polygon
       (pts
-        (xy 270 190) (xy 190 190) (xy 190 35) (xy 270 35)
+        (xy 262 181) (xy 197 181) (xy 197 44) (xy 262 44)
       )
     )
