File: hardware/sensor_board/sensor_board.kicad_pcb (KiCad board)
At the start: 2 copper layers, 65 x 137 mm, 99 parts, among them IC1 ATMEGA88A-A, J1 RJ45_8P8C_8FACH, K1 pow_sel, P1 UART, P2 Shield, P3 i2c_pow, P4 i2c_chain, P5 12Vin, P6 HOHLBUCHSE, P7 Vccin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

Commit message: for put all together
Parts:
- moved C1 309.1 mm to (514.2, 62.0)
- moved C10 309.1 mm to (546.2, 99.8)
- moved C12 309.1 mm to (546.2, 71.8)
- moved C13 309.1 mm to (546.2, 57.8)
- moved C14 309.1 mm to (546.2, 43.8)
- moved C2 309.1 mm to (522.2, 98.4)
- moved C29 309.1 mm to (535.7, 93.7)
- moved C3 309.1 mm to (523.2, 76.1)
- moved C32 309.1 mm to (535.7, 133.2)
- moved C7 309.1 mm to (546.2, 141.8)
- moved C8 309.1 mm to (546.2, 127.8)
- moved C9 309.1 mm to (546.2, 113.8)
- moved R10 309.1 mm to (539.2, 134.8)
- moved R11 309.1 mm to (539.2, 120.8)
- moved R12 309.1 mm to (539.2, 106.8)
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