File: hardware/temperature_board/temperature_board.sch (KiCad schematic (older format))
At the start: 10 parts

Commit message: modify sensor board schematik
Connections:
- wire segments 34 -> 36
Other:
- moved on the sheet: C?, J?, R?, U?
