File: hardware/temperature_board/temperature_board.sch (KiCad schematic (older format))
At the start: 11 parts

Commit message: begin with pcb
Parts:
- removed U?: ST485, symbol ST485
- added U?: ST485, ~, symbol ST485
- gave numbers to parts that had none: 10
Connections:
- wire segments 38 -> 49
Changed lines of the file:
@@
 $EndDescr
 $Comp
-L VCC #PWR?
+L VCC #PWR01
 U 1 1 532DBFEE
 P 4750 2700
-F 0 "#PWR?" H 4750 2800 30  0001 C CNN
+F 0 "#PWR01" H 4750 2800 30  0001 C CNN
 F 1 "VCC" H 4750 2800 30  0000 C CNN
 F 2 "" H 4750 2700 60  0000 C CNN
@@
 $EndComp
 $Comp
-L TSIC50XF U?
+L TSIC50XF U1
 U 1 1 532DDB20
 P 3250 3900
-F 0 "U?" H 3450 4350 70  0000 C CNN
+F 0 "U1" H 3450 4350 70  0000 C CNN
 F 1 "TSIC50XF" H 3250 3700 70  0000 C CNN
 F 2 "~" H 3250 3900 60  0000 C CNN
@@
 $EndComp
 $Comp
-L ST485 U?
-U 1 1 532DDB2F
-P 6050 3600
-F 0 "U?" H 6500 4200 70  0000 C BNN
-F 1 "ST485" H 6450 3050 70  0000 C CNN
-F 2 "" H 6050 3500 60  0000 C CNN
-F 3 "" H 6050 3500 60  0000 C CNN
-	1    6050 3600
-	1    0    0    -1
-$EndComp
-$Comp
-L R R?
+L R R4
 U 1 1 532DDB70
 P 8000 3600
-F 0 "R?" V 8080 3600 40  0000 C CNN
+F 0 "R4" V 8080 3600 40  0000 C CNN
 F 1 "120" V 8007 3601 40  0000 C CNN
 F 2 "~" V 7930 3600 30  0000 C CNN
@@
 	8000 3250 8000 3350
 $Comp
-L GND #PWR?
+L GND #PWR02
 U 1 1 532DDBFC
 P 6050 5000
-F 0 "#PWR?" H 6050 5000 30  0001 C CNN
+F 0 "#PWR02" H 6050 5000 30  0001 C CNN
 F 1 "GND" H 6050 4930 30  0001 C CNN
 F 2 "" H 6050 5000 60  0000 C CNN
@@
 $EndComp
 $Comp
-L VCC #PWR?
+L VCC #PWR03
 U 1 1 532DDC02
 P 6050 1850
-F 0 "#PWR?" H 6050 1950 30  0001 C CNN
+F 0 "#PWR03" H 6050 1950 30  0001 C CNN
 F 1 "VCC" H 6050 1950 30  0000 C CNN
 F 2 "" H 6050 1850 60  0000 C CNN
@@
 $EndComp
 Wire Wire Line
-	6050 1850 6050 2550
+	6050 1850 6050 2050
+Wire Wire Line
+	6050 2050 6050 2400
+Wire Wire Line
+	6050 2400 6050 2550
 Wire Wire Line
 	6050 4550 6050 5000
 $Comp
-L C C?
+L C C3
 U 1 1 532DDC2C
 P 6500 2400
-F 0 "C?" H 6500 2500 40  0000 L CNN
+F 0 "C3" H 6500 2500 40  0000 L CNN
 F 1 "10uF" H 6506 2315 40  0000 L CNN
 F 2 "~" H 6538 2250 30  0000 C CNN
@@
 $EndComp
 $Comp
-L GND #PWR?
+L GND #PWR04
 U 1 1 532DDC32
 P 6900 2600
-F 0 "#PWR?" H 6900 2600 30  0001 C CNN
+F 0 "#PWR04" H 6900 2600 30  0001 C CNN
 F 1 "GND" H 6900 2530 30  0001 C CNN
 F 2 "" H 6900 2600 60  0000 C CNN
@@
 	6700 2400 6900 2400
 Wire Wire Line
-	6900 2050 6900 2600
-$Comp
-L GND #PWR?
+	6900 2050 6900 2400
+Wire Wire Line
+	6900 2400 6900 2600
+$Comp
+L GND #PWR05
 U 1 1 532DDC5E
 P 3250 5200
-F 0 "#PWR?" H 3250 5200 30  0001 C CNN
+F 0 "#PWR05" H 3250 5200 30  0001 C CNN
 F 1 "GND" H 3250 5130 30  0001 C CNN
 F 2 "" H 3250 5200 60  0000 C CNN
@@
 $EndComp
 $Comp
-L C C?
+L C C1
 U 1 1 532DDC6A
 P 3900 2850
-F 0 "C?" H 3900 2950 40  0000 L CNN
+F 0 "C1" H 3900 2950 40  0000 L CNN
 F 1 "100nF" H 3906 2765 40  0000 L CNN
 F 2 "~" H 3938 2700 30  0000 C CNN
@@
 	3700 2850 3250 2850
 Wire Wire Line
-	3250 2650 3250 3050
-$Comp
-L R R?
+	3250 2650 3250 2850
+Wire Wire Line
+	3250 2850 3250 3050
+$Comp
+L R R1
 U 1 1 532DDC9D
 P 3250 2400
-F 0 "R?" V 3330 2400 40  0000 C CNN
+F 0 "R1" V 3330 2400 40  0000 C CNN
 F 1 "220" V 3257 2401 40  0000 C CNN
 F 2 "~" V 3180 2400 30  0000 C CNN
@@
 $EndComp
 $Comp
-L GND #PWR?
+L GND #PWR06
 U 1 1 532DDCAA
 P 4250 3250
-F 0 "#PWR?" H 4250 3250 30  0001 C CNN
+F 0 "#PWR06" H 4250 3250 30  0001 C CNN
 F 1 "GND" H 4250 3180 30  0001 C CNN
 F 2 "" H 4250 3250 60  0000 C CNN
@@
 Connection ~ 3250 2850
 $Comp
-L VCC #PWR?
+L VCC #PWR07
 U 1 1 532DDCEC
 P 3250 1950
-F 0 "#PWR?" H 3250 2050 30  0001 C CNN
+F 0 "#PWR07" H 3250 2050 30  0001 C CNN
 F 1 "VCC" H 3250 2050 30  0000 C CNN
 F 2 "" H 3250 1950 60  0000 C CNN
@@
 	3900 3900 5150 3900
 Wire Wire Line
-	4750 2700 4750 3700
+	4750 2700 4750 3500
+Wire Wire Line
+	4750 3500 4750 3700
 Wire Wire Line
 	4750 3500 5150 3500
@@
 Connection ~ 4750 3500
 $Comp
-L RJ45 J?
+L RJ45 J1
 U 1 1 532DDDA3
 P 9950 3600
-F 0 "J?" H 10150 4100 60  0000 C CNN
+F 0 "J1" H 10150 4100 60  0000 C CNN
 F 1 "RJ45" H 9800 4100 60  0000 C CNN
 F 2 "~" H 9950 3600 60  0000 C CNN
@@
 $EndComp
 $Comp
-L GND #PWR?
+L GND #PWR08
 U 1 1 532DDE77
 P 9350 4200
-F 0 "#PWR?" H 9350 4200 30  0001 C CNN
+F 0 "#PWR08" H 9350 4200 30  0001 C CNN
 F 1 "GND" H 9350 4130 30  0001 C CNN
 F 2 "" H 9350 4200 60  0000 C CNN
@@
 	9350 3950 9500 3950
 $Comp
-L VCC #PWR?
+L VCC #PWR09
 U 1 1 532DE001
 P 9350 3500
-F 0 "#PWR?" H 9350 3600 30  0001 C CNN
+F 0 "#PWR09" H 9350 3600 30  0001 C CNN
 F 1 "VCC" H 9350 3600 30  0000 C CNN
 F 2 "" H 9350 3500 60  0000 C CNN
@@
 Connection ~ 8000 3250
 $Comp
-L C C?
+L C C4
 U 1 1 534839D5
 P 8000 4150
-F 0 "C?" H 8000 4250 40  0000 L CNN
+F 0 "C4" H 8000 4250 40  0000 L CNN
 F 1 "100nF" H 8006 4065 40  0000 L CNN
 F 2 "~" H 8038 4000 30  0000 C CNN
@@
 	8000 3850 8000 3950
 Wire Wire Line
-	7050 4350 8500 4350
+	7050 4350 7350 4350
+Wire Wire Line
+	7350 4350 8000 4350
+Wire Wire Line
+	8000 4350 8500 4350
 Connection ~ 8000 4350
 $Comp
-L R R?
+L R R2
 U 1 1 53483A7B
 P 7350 3750
-F 0 "R?" V 7430 3750 40  0000 C CNN
+F 0 "R2" V 7430 3750 40  0000 C CNN
 F 1 "22k" V 7357 3751 40  0000 C CNN
 F 2 "~" V 7280 3750 30  0000 C CNN
@@
 $EndComp
 $Comp
-L R R?
+L R R3
 U 1 1 53483A81
 P 7600 3750
-F 0 "R?" V 7680 3750 40  0000 C CNN
+F 0 "R3" V 7680 3750 40  0000 C CNN
 F 1 "22k" V 7607 3751 40  0000 C CNN
 F 2 "~" V 7530 3750 30  0000 C CNN
@@
 $EndComp
 $Comp
-L GND #PWR?
+L GND #PWR010
 U 1 1 53483B09
 P 7600 4200
-F 0 "#PWR?" H 7600 4200 30  0001 C CNN
+F 0 "#PWR010" H 7600 4200 30  0001 C CNN
 F 1 "GND" H 7600 4130 30  0001 C CNN
 F 2 "" H 7600 4200 60  0000 C CNN
@@
 $EndComp
 $Comp
-L VCC #PWR?
+L VCC #PWR011
 U 1 1 53483B0F
 P 7350 3400
-F 0 "#PWR?" H 7350 3500 30  0001 C CNN
+F 0 "#PWR011" H 7350 3500 30  0001 C CNN
 F 1 "VCC" H 7350 3500 30  0000 C CNN
 F 2 "" H 7350 3400 60  0000 C CNN
@@
 	7600 4000 7600 4200
 $Comp
-L GND #PWR?
+L GND #PWR012
 U 1 1 534937C6
 P 10300 4300
-F 0 "#PWR?" H 10300 4300 30  0001 C CNN
+F 0 "#PWR012" H 10300 4300 30  0001 C CNN
 F 1 "GND" H 10300 4230 30  0001 C CNN
 F 2 "" H 10300 4300 60  0000 C CNN
@@
 	10300 4150 10300 4300
 Wire Wire Line
-	9350 3500 9350 3650
+	9350 3500 9350 3550
+Wire Wire Line
+	9350 3550 9350 3650
 Wire Wire Line
 	9350 3550 9500 3550
@@
 Connection ~ 9350 3550
 Wire Wire Line
-	9350 3850 9350 4200
+	9350 3850 9350 3950
+Wire Wire Line
+	9350 3950 9350 4200
 Wire Wire Line
 	9500 3850 9350 3850
@@
 	9350 3350 9500 3350
 Wire Wire Line
-	7050 3250 8500 3250
-$Comp
-L C C?
+	7050 3250 7600 3250
+Wire Wire Line
+	7600 3250 8000 3250
+Wire Wire Line
+	8000 3250 8500 3250
+$Comp
+L C C2
 U 1 1 535FF48E
 P 6500 2050
-F 0 "C?" H 6500 2150 40  0000 L CNN
+F 0 "C2" H 6500 2150 40  0000 L CNN
 F 1 "100nF" H 6506 1965 40  0000 L CNN
 F 2 "~" H 6538 1900 30  0000 C CNN
@@
 	6300 2050 6050 2050
 Connection ~ 6050 2050
+$Comp
+L ST485 U?
+U 1 1 5360054D
+P 6050 3600
+F 0 "U?" H 6500 4200 70  0000 C BNN
+F 1 "ST485" H 6450 3050 70  0000 C CNN
+F 2 "~" H 6050 3500 60  0000 C CNN
+F 3 "~" H 6050 3500 60  0000 C CNN
+	1    6050 3600
+	1    0    0    -1
+$EndComp
 $EndSCHEMATC

Commit message: add netlist and pcb
Parts:
- gave numbers to parts that had none: 1
Connections:
- wire segments 49 -> 38
Changed lines of the file:
@@
 $EndComp
 Wire Wire Line
-	6050 1850 6050 2050
-Wire Wire Line
-	6050 2050 6050 2400
-Wire Wire Line
-	6050 2400 6050 2550
+	6050 1850 6050 2550
 Wire Wire Line
 	6050 4550 6050 5000
@@
 	6700 2400 6900 2400
 Wire Wire Line
-	6900 2050 6900 2400
-Wire Wire Line
-	6900 2400 6900 2600
+	6900 2050 6900 2600
 $Comp
 L GND #PWR05
@@
 	3700 2850 3250 2850
 Wire Wire Line
-	3250 2650 3250 2850
-Wire Wire Line
-	3250 2850 3250 3050
+	3250 2650 3250 3050
 $Comp
 L R R1
@@
 	3900 3900 5150 3900
 Wire Wire Line
-	4750 2700 4750 3500
-Wire Wire Line
-	4750 3500 4750 3700
+	4750 2700 4750 3700
 Wire Wire Line
 	4750 3500 5150 3500
@@
 	8000 3850 8000 3950
 Wire Wire Line
-	7050 4350 7350 4350
-Wire Wire Line
-	7350 4350 8000 4350
-Wire Wire Line
-	8000 4350 8500 4350
+	7050 4350 8500 4350
 Connection ~ 8000 4350
 $Comp
@@
 	10300 4150 10300 4300
 Wire Wire Line
-	9350 3500 9350 3550
-Wire Wire Line
-	9350 3550 9350 3650
+	9350 3500 9350 3650
 Wire Wire Line
 	9350 3550 9500 3550
@@
 Connection ~ 9350 3550
 Wire Wire Line
-	9350 3850 9350 3950
-Wire Wire Line
-	9350 3950 9350 4200
+	9350 3850 9350 4200
 Wire Wire Line
 	9500 3850 9350 3850
@@
 	9350 3350 9500 3350
 Wire Wire Line
-	7050 3250 7600 3250
-Wire Wire Line
-	7600 3250 8000 3250
-Wire Wire Line
-	8000 3250 8500 3250
+	7050 3250 8500 3250
 $Comp
 L C C2
@@
 Connection ~ 6050 2050
 $Comp
-L ST485 U?
+L ST485 U2
 U 1 1 5360054D
 P 6050 3600
-F 0 "U?" H 6500 4200 70  0000 C BNN
+F 0 "U2" H 6500 4200 70  0000 C BNN
 F 1 "ST485" H 6450 3050 70  0000 C CNN
 F 2 "~" H 6050 3500 60  0000 C CNN

Commit message: many images :)
Connections:
- wire segments 38 -> 49
- no-connect marks 0 -> 1
Other:
- moved on the sheet: J1
Changed lines of the file:
@@
 Sheet 1 1
 Title ""
-Date "29 apr 2014"
+Date "21 jun 2014"
 Rev ""
 Comp ""
@@
 $EndComp
 Wire Wire Line
-	6050 1850 6050 2550
+	6050 1850 6050 2050
+Wire Wire Line
+	6050 2050 6050 2400
+Wire Wire Line
+	6050 2400 6050 2550
 Wire Wire Line
 	6050 4550 6050 5000
@@
 	6700 2400 6900 2400
 Wire Wire Line
-	6900 2050 6900 2600
+	6900 2050 6900 2400
+Wire Wire Line
+	6900 2400 6900 2600
 $Comp
 L GND #PWR05
 U 1 1 532DDC5E
-P 3250 5200
-F 0 "#PWR05" H 3250 5200 30  0001 C CNN
-F 1 "GND" H 3250 5130 30  0001 C CNN
-F 2 "" H 3250 5200 60  0000 C CNN
-F 3 "" H 3250 5200 60  0000 C CNN
-	1    3250 5200
+P 3250 5000
+F 0 "#PWR05" H 3250 5000 30  0001 C CNN
+F 1 "GND" H 3250 4930 30  0001 C CNN
+F 2 "" H 3250 5000 60  0000 C CNN
+F 3 "" H 3250 5000 60  0000 C CNN
+	1    3250 5000
 	1    0    0    -1
 $EndComp
@@
 $EndComp
 Wire Wire Line
-	3250 5200 3250 4750
-Wire Wire Line
 	3700 2850 3250 2850
 Wire Wire Line
-	3250 2650 3250 3050
+	3250 2650 3250 2850
+Wire Wire Line
+	3250 2850 3250 3050
 $Comp
 L R R1
@@
 L VCC #PWR07
 U 1 1 532DDCEC
-P 3250 1950
-F 0 "#PWR07" H 3250 2050 30  0001 C CNN
-F 1 "VCC" H 3250 2050 30  0000 C CNN
-F 2 "" H 3250 1950 60  0000 C CNN
-F 3 "" H 3250 1950 60  0000 C CNN
-	1    3250 1950
-	1    0    0    -1
-$EndComp
-Wire Wire Line
-	3250 1950 3250 2150
+P 3250 1850
+F 0 "#PWR07" H 3250 1950 30  0001 C CNN
+F 1 "VCC" H 3250 1950 30  0000 C CNN
+F 2 "" H 3250 1850 60  0000 C CNN
+F 3 "" H 3250 1850 60  0000 C CNN
+	1    3250 1850
+	1    0    0    -1
+$EndComp
+Wire Wire Line
+	3250 1850 3250 2150
 Wire Wire Line
 	3900 3900 5150 3900
 Wire Wire Line
-	4750 2700 4750 3700
+	4750 2700 4750 3500
+Wire Wire Line
+	4750 3500 4750 3700
 Wire Wire Line
 	4750 3500 5150 3500
@@
 L RJ45 J1
 U 1 1 532DDDA3
-P 9950 3600
-F 0 "J1" H 10150 4100 60  0000 C CNN
-F 1 "RJ45" H 9800 4100 60  0000 C CNN
-F 2 "~" H 9950 3600 60  0000 C CNN
-F 3 "~" H 9950 3600 60  0000 C CNN
-	1    9950 3600
+P 9450 3700
+F 0 "J1" H 9650 4200 60  0000 C CNN
+F 1 "RJ45" H 9300 4200 60  0000 C CNN
+F 2 "~" H 9450 3700 60  0000 C CNN
+F 3 "~" H 9450 3700 60  0000 C CNN
+	1    9450 3700
 	0    1    1    0
 $EndComp
@@
 L GND #PWR08
 U 1 1 532DDE77
-P 9350 4200
-F 0 "#PWR08" H 9350 4200 30  0001 C CNN
-F 1 "GND" H 9350 4130 30  0001 C CNN
-F 2 "" H 9350 4200 60  0000 C CNN
-F 3 "" H 9350 4200 60  0000 C CNN
-	1    9350 4200
-	1    0    0    -1
-$EndComp
-Wire Wire Line
-	9350 3950 9500 3950
+P 8850 4300
+F 0 "#PWR08" H 8850 4300 30  0001 C CNN
+F 1 "GND" H 8850 4230 30  0001 C CNN
+F 2 "" H 8850 4300 60  0000 C CNN
+F 3 "" H 8850 4300 60  0000 C CNN
+	1    8850 4300
+	1    0    0    -1
+$EndComp
+Wire Wire Line
+	8850 4050 9000 4050
 $Comp
 L VCC #PWR09
 U 1 1 532DE001
-P 9350 3500
-F 0 "#PWR09" H 9350 3600 30  0001 C CNN
-F 1 "VCC" H 9350 3600 30  0000 C CNN
-F 2 "" H 9350 3500 60  0000 C CNN
-F 3 "" H 9350 3500 60  0000 C CNN
-	1    9350 3500
+P 8850 3600
+F 0 "#PWR09" H 8850 3700 30  0001 C CNN
+F 1 "VCC" H 8850 3700 30  0000 C CNN
+F 2 "" H 8850 3600 60  0000 C CNN
+F 3 "" H 8850 3600 60  0000 C CNN
+	1    8850 3600
 	1    0    0    -1
 $EndComp
@@
 	8000 3850 8000 3950
 Wire Wire Line
-	7050 4350 8500 4350
+	7050 4350 7350 4350
+Wire Wire Line
+	7350 4350 8000 4350
+Wire Wire Line
+	8000 4350 8500 4350
 Connection ~ 8000 4350
 $Comp
@@
 L GND #PWR012
 U 1 1 534937C6
-P 10300 4300
-F 0 "#PWR012" H 10300 4300 30  0001 C CNN
-F 1 "GND" H 10300 4230 30  0001 C CNN
-F 2 "" H 10300 4300 60  0000 C CNN
-F 3 "" H 10300 4300 60  0000 C CNN
-	1    10300 4300
-	1    0    0    -1
-$EndComp
-Wire Wire Line
-	10300 4150 10300 4300
-Wire Wire Line
-	9350 3500 9350 3650
-Wire Wire Line
-	9350 3550 9500 3550
-Wire Wire Line
-	9350 3650 9500 3650
-Connection ~ 9350 3550
-Wire Wire Line
-	9350 3850 9350 4200
-Wire Wire Line
-	9500 3850 9350 3850
-Connection ~ 9350 3950
+P 9800 4400
+F 0 "#PWR012" H 9800 4400 30  0001 C CNN
+F 1 "GND" H 9800 4330 30  0001 C CNN
+F 2 "" H 9800 4400 60  0000 C CNN
+F 3 "" H 9800 4400 60  0000 C CNN
+	1    9800 4400
+	1    0    0    -1
+$EndComp
+Wire Wire Line
+	9800 4250 9800 4400
+Wire Wire Line
+	8850 3600 8850 3650
+Wire Wire Line
+	8850 3650 8850 3750
+Wire Wire Line
+	8850 3650 9000 3650
+Wire Wire Line
+	8850 3750 9000 3750
+Connection ~ 8850 3650
+Wire Wire Line
+	8850 3950 8850 4050
+Wire Wire Line
+	8850 4050 8850 4300
+Wire Wire Line
+	9000 3950 8850 3950
+Connection ~ 8850 4050
 Wire Wire Line
 	7350 3400 7350 3500
@@
 	7600 3500 7600 3250
 Connection ~ 7600 3250
-Text Label 9350 3250 0    60   ~ 0
+Text Label 8850 3350 0    60   ~ 0
 za
-Text Label 9350 3350 0    60   ~ 0
+Text Label 8850 3450 0    60   ~ 0
 zb
 Text Label 8500 4350 0    60   ~ 0
@@
 zb
 Wire Wire Line
-	9350 3250 9500 3250
-Wire Wire Line
-	9350 3350 9500 3350
-Wire Wire Line
-	7050 3250 8500 3250
+	8850 3350 9000 3350
+Wire Wire Line
+	8850 3450 9000 3450
+Wire Wire Line
+	7050 3250 7600 3250
+Wire Wire Line
+	7600 3250 8000 3250
+Wire Wire Line
+	8000 3250 8500 3250
 $Comp
 L C C2
@@
 	1    0    0    -1
 $EndComp
+Wire Wire Line
+	3250 4750 3250 5000
+NoConn ~ 5150 3300
 $EndSCHEMATC

Commit message: report schematic images
Connections:
- wire segments 49 -> 38
Other:
- moved on the sheet: C1, C2, C3, C4, J1, R1, R2, R3, R4, U2
