File: hardware/temperature_board/temperature_board-append.kicad_pcb (KiCad board)
At the start: 2 copper layers, 502 x 375 mm, 740 parts, among them IC1 ATMEGA88-A, IC1 ATMEGA88A-A, J1 RJ45, J1 RJ45_8P8C_8FACH, K1 CONN_3, K1 pow_sel, K2 CONN_3, P1 CONN_4, P1 ISP, P1 UART, P2 CONN_4, P2 Shield, P2 UART, P2 so8, P3 CONN_4, P3 i2c_pow, P4 i2c_chain, P5 12Vin, P6 HOHLBUCHSE, P7 Vccin, P8 ISP, P9 5Vin, SW1 SW1, SW1 SW_RESET, SW2 SCHALTER_2POL, SW3 SW_RESET, U1 LM7805, U1 ST485, U1 TSIC50XF, U2 HYT271, U2 ST485, U3 ST485, U4 ST485, U5 ST485, U6 ST485, U7 ST485, U8 ST485, U9 ST485, X1 20MHz, m3_loch VAL**

Commit message: finished
Parts:
- removed the C1 at (520.0, 97.9)
- removed the C1 at (489.0, 142.1)
- removed the C2 at (505.0, 85.0)
- removed the C2 at (504.0, 155.0)
- removed the C3 at (518.0, 81.8)
- removed the C3 at (491.0, 158.2)
- removed the C4 at (505.0, 82.0)
- removed the C4 at (504.0, 158.0)
- removed the C5 at (511.5, 76.5)
- removed the C5 at (497.5, 163.5)
- removed the C6 at (519.5, 114.5)
- removed the C6 at (489.5, 125.5)
- removed the D1 at (506.0, 104.6)
- removed the D1 at (503.0, 135.4)
- removed the D2 at (503.6, 104.6)
- removed the D2 at (505.4, 135.4)
- removed the IC1 at (514.0, 103.0)
- removed the IC1 at (495.0, 137.0)
- removed the J1 at (512.0, 64.0)
- removed the J1 at (497.0, 176.0)
- removed the K1 at (317.5, 390.9)
- removed the K2 at (312.4, 390.9)
- removed the P1 at (512.0, 92.0)
- removed the P1 at (497.0, 148.0)
- removed the P1 at (310.7, 358.3)
- removed the P1 at (373.6, 273.7)
- removed the P2 at (517.8, 112.4)
- removed the P2 at (491.2, 127.6)
- removed the P2 at (310.7, 353.9)
- removed the P2 at (368.5, 273.7)
- removed the P3 at (310.7, 345.6)
- removed the R1 at (506.0, 100.0)
- removed the R1 at (503.0, 140.0)
- removed the R2 at (503.6, 100.0)
- removed the R2 at (505.4, 140.0)
- removed the R3 at (518.0, 85.3)
- removed the R3 at (491.0, 154.7)
- removed the R4 at (518.0, 78.8)
- removed the R4 at (491.0, 161.2)
- removed the R5 at (505.0, 79.0)
- removed the R5 at (504.0, 161.0)
- removed the R6 at (507.5, 76.5)
- removed the R6 at (501.5, 163.5)
- removed the R7 at (511.4, 119.2)
- removed the R7 at (497.6, 120.8)
- removed the R8 at (515.2, 119.2)
- removed the R8 at (493.8, 120.8)
- removed the SW1 at (506.0, 70.5)
- removed the SW1 at (503.0, 169.5)
- removed the U1 at (512.0, 81.0)
- removed the U1 at (497.0, 159.0)
- removed the U2 at (512.0, 147.5)
- removed the U2 at (497.0, 92.5)
- removed the m3_loch at (507.0, 113.0)
- removed the m3_loch at (517.0, 71.5)
- removed the m3_loch at (502.0, 127.0)
- removed the m3_loch at (492.0, 168.5)
Routing:
- net VCC: track 4185.5 -> 3787.2 mm, vias 89 -> 81
- net GND: track 6154.2 -> 5785.4 mm, vias 81 -> 71
- net /RESET: track 767.0 -> 655.4 mm, vias 22 -> 18
- net /SDA: track 583.6 -> 498.6 mm
- net /SCL: track 605.1 -> 520.7 mm
- net /za: track 619.2 -> 560.8 mm, vias 8 -> 6
- net /zb: track 620.3 -> 565.0 mm
- net /DI: track 148.1 -> 111.1 mm
- net /MOSI: track 243.1 -> 219.5 mm, vias 14 -> 12
- net N-000002: track 100.2 -> 78.2 mm
- net /SCK: track 120.9 -> 99.6 mm
- net /RX: track 219.6 -> 199.5 mm
- net /MISO: track 104.0 -> 84.6 mm
- net N-000001: track 80.6 -> 63.6 mm
- net N-000003: track 109.6 -> 93.2 mm
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Other:
- board size 502 x 375 mm -> 200.1 x 330 mm

Commit message: 3 humidity boards but just 19 temperature
Parts:
- removed the C1 at (68.9, 82.0)
- removed the C1 at (68.9, 22.0)
- removed the C1 at (113.1, 53.0)
- removed the C1 at (113.1, 83.0)
- removed the C1 at (68.9, 52.0)
- removed the C2 at (56.0, 97.0)
- removed the C2 at (56.0, 37.0)
- removed the C2 at (126.0, 38.0)
- removed the C2 at (126.0, 68.0)
- removed the C2 at (56.0, 67.0)
- removed the C3 at (52.8, 84.0)
- removed the C3 at (52.8, 24.0)
- removed the C3 at (129.2, 51.0)
- removed the C3 at (129.2, 81.0)
- removed the C3 at (52.8, 54.0)
- removed the C4 at (53.0, 97.0)
- removed the C4 at (53.0, 37.0)
- removed the C4 at (129.0, 38.0)
- removed the C4 at (129.0, 68.0)
- removed the C4 at (53.0, 67.0)
- removed the C5 at (47.5, 90.5)
- removed the C5 at (47.5, 30.5)
- removed the C5 at (134.5, 44.5)
- removed the C5 at (134.5, 74.5)
- removed the C5 at (47.5, 60.5)
- removed the C6 at (85.5, 82.5)
- removed the C6 at (85.5, 22.5)
- removed the C6 at (96.5, 52.5)
- removed the C6 at (96.5, 82.5)
- removed the C6 at (85.5, 52.5)
- removed the D1 at (75.6, 96.0)
- removed the D1 at (75.6, 36.0)
- removed the D1 at (106.4, 39.0)
- removed the D1 at (106.4, 69.0)
- removed the D1 at (75.6, 66.0)
- removed the D2 at (75.6, 98.4)
- removed the D2 at (75.6, 38.4)
- removed the D2 at (106.4, 36.6)
- removed the D2 at (106.4, 66.6)
- removed the D2 at (75.6, 68.4)
- removed the IC1 at (74.0, 88.0)
- removed the IC1 at (74.0, 28.0)
- removed the IC1 at (108.0, 47.0)
- removed the IC1 at (108.0, 77.0)
- removed the IC1 at (74.0, 58.0)
- removed the J1 at (35.0, 90.0)
- removed the J1 at (35.0, 30.0)
- removed the J1 at (147.0, 45.0)
- removed the J1 at (147.0, 75.0)
- removed the J1 at (35.0, 60.0)
- removed the K1 at (28.5, 105.9)
- removed K2: CONN_3, Tsic_TO92
- removed the P1 at (63.0, 90.0)
- removed the P1 at (63.0, 30.0)
- removed the P1 at (119.0, 45.0)
- removed the P1 at (119.0, 75.0)
- removed the P1 at (63.0, 60.0)
- removed the P1 at (173.3, 25.3)
- removed the P1 at (23.4, 117.3)
- removed the P1 at (155.3, 25.3)
- removed the P1 at (137.3, 25.3)
- removed the P1 at (46.3, 108.3)
- removed the P1 at (52.4, 107.3)
- removed the P2 at (83.4, 84.2)
- removed the P2 at (83.4, 24.2)
- removed the P2 at (98.6, 50.8)
- removed the P2 at (98.6, 80.8)
- removed the P2 at (83.4, 54.2)
- removed the P2 at (168.9, 25.3)
- removed the P2 at (28.5, 117.3)
- removed the P2 at (150.9, 25.3)
- removed the P2 at (132.9, 25.3)
- removed the P2 at (41.9, 108.3)
- removed the P2 at (57.5, 107.3)
- removed the P3 at (142.6, 25.3)
- removed the P3 at (124.6, 25.3)
- removed the P3 at (33.6, 108.3)
- removed the P3 at (160.6, 25.3)
- removed the R1 at (71.0, 96.0)
- removed the R1 at (71.0, 36.0)
- removed the R1 at (111.0, 39.0)
- removed the R1 at (111.0, 69.0)
- removed the R1 at (71.0, 66.0)
- removed the R2 at (71.0, 98.4)
- removed the R2 at (71.0, 38.4)
- removed the R2 at (111.0, 36.6)
- removed the R2 at (111.0, 66.6)
- removed the R2 at (71.0, 68.4)
- removed the R3 at (56.3, 84.0)
- removed the R3 at (56.3, 24.0)
- removed the R3 at (125.7, 51.0)
- removed the R3 at (125.7, 81.0)
- removed the R3 at (56.3, 54.0)
- removed the R4 at (49.8, 84.0)
- removed the R4 at (49.8, 24.0)
- removed the R4 at (132.2, 51.0)
- removed the R4 at (132.2, 81.0)
- removed the R4 at (49.8, 54.0)
- removed the R5 at (50.0, 97.0)
- removed the R5 at (50.0, 37.0)
- removed the R5 at (132.0, 38.0)
- removed the R5 at (132.0, 68.0)
- removed the R5 at (50.0, 67.0)
- removed the R6 at (47.5, 94.5)
- removed the R6 at (47.5, 34.5)
- removed the R6 at (134.5, 40.5)
- removed the R6 at (134.5, 70.5)
- removed the R6 at (47.5, 64.5)
- removed the R7 at (90.2, 90.6)
- removed the R7 at (90.2, 30.6)
- removed the R7 at (91.8, 44.4)
- removed the R7 at (91.8, 74.4)
- removed the R7 at (90.2, 60.6)
- removed the R8 at (90.2, 86.8)
- removed the R8 at (90.2, 26.8)
- removed the R8 at (91.8, 48.2)
- removed the R8 at (91.8, 78.2)
- removed the R8 at (90.2, 56.8)
- removed the SW1 at (41.5, 96.0)
- removed the SW1 at (41.5, 36.0)
- removed the SW1 at (140.5, 39.0)
- removed the SW1 at (140.5, 69.0)
- removed the SW1 at (41.5, 66.0)
- removed the U1 at (52.0, 90.0)
- removed the U1 at (52.0, 30.0)
- removed the U1 at (130.0, 45.0)
- removed the U1 at (130.0, 75.0)
- removed the U1 at (52.0, 60.0)
- removed the U2 at (118.5, 90.0)
- removed the U2 at (118.5, 30.0)
- removed the U2 at (63.5, 45.0)
- removed the U2 at (63.5, 75.0)
- removed the U2 at (118.5, 60.0)
- removed the m3_loch at (84.0, 95.0)
- removed the m3_loch at (84.0, 65.0)
- removed the m3_loch at (42.5, 85.0)
- removed the m3_loch at (84.0, 35.0)
- removed the m3_loch at (42.5, 25.0)
- removed the m3_loch at (98.0, 40.0)
- removed the m3_loch at (139.5, 50.0)
- removed the m3_loch at (139.5, 80.0)
- removed the m3_loch at (98.0, 70.0)
- removed the m3_loch at (42.5, 55.0)
- added C1: 100nF, SM0603_big, F.Cu at (61.5, 97.8)
- added C1: 100nF, SM0603_big, F.Cu at (440.5, 209.8)
- added C1: 100nF, SM0603_big, F.Cu at (61.5, 67.8)
- added C1: 100nF, SM0603_big, F.Cu at (388.5, 66.8)
- added C1: 100nF, SM0603_big, F.Cu at (72.5, 97.2)
- added C1: 100nF, SM0603_big, F.Cu at (113.1, 68.0)
- added C1: 100nF, SM0603_big, F.Cu at (399.5, 96.2)
- added C1: 100nF, SM0603_big, F.Cu at (364.5, 370.2)
- added C1: 100nF, SM0603_big, F.Cu at (113.1, 38.0)
- added C1: 100nF, SM0603_big, F.Cu at (68.9, 37.0)
- added C2: 100nF, SM0603_big, F.Cu at (52.8, 112.2)
- added C2: 100nF, SM0603_big, F.Cu at (431.8, 224.2)
- added C2: 100nF, SM0603_big, F.Cu at (52.8, 82.2)
- added C2: 100nF, SM0603_big, F.Cu at (379.8, 81.2)
- added C2: 100nF, SM0603_big, F.Cu at (81.2, 82.8)
- added C2: 10uF, SM0805_big, F.Cu at (126.0, 53.0)
- added C2: 100nF, SM0603_big, F.Cu at (408.2, 81.8)
- added C2: 100nF, SM0603_big, F.Cu at (373.2, 355.8)
- added C2: 10uF, SM0805_big, F.Cu at (126.0, 23.0)
- added C2: 10uF, SM0805_big, F.Cu at (56.0, 52.0)
- added C3: 10uF, SM0805_big, F.Cu at (49.2, 112.2)
- added C3: 10uF, SM0805_big, F.Cu at (428.2, 224.2)
- added C3: 10uF, SM0805_big, F.Cu at (49.2, 82.2)
- added C3: 10uF, SM0805_big, F.Cu at (376.2, 81.2)
- added C3: 10uF, SM0805_big, F.Cu at (84.8, 82.8)
- added C3: 100nF, SM0603_big, F.Cu at (129.2, 66.0)
- added C3: 10uF, SM0805_big, F.Cu at (411.8, 81.8)
- added C3: 10uF, SM0805_big, F.Cu at (376.8, 355.8)
- added C3: 100nF, SM0603_big, F.Cu at (129.2, 36.0)
- added C3: 100nF, SM0603_big, F.Cu at (52.8, 39.0)
- added C4: 100nF, SM0603_big, F.Cu at (42.0, 106.8)
- added C4: 100nF, SM0603_big, F.Cu at (421.0, 218.8)
- added C4: 100nF, SM0603_big, F.Cu at (42.0, 76.8)
- added C4: 100nF, SM0603_big, F.Cu at (369.0, 75.8)
- added C4: 100nF, SM0603_big, F.Cu at (92.0, 88.2)
- added C4: 10uF, SM0805_big, F.Cu at (129.0, 53.0)
- added C4: 100nF, SM0603_big, F.Cu at (419.0, 87.2)
- added C4: 100nF, SM0603_big, F.Cu at (384.0, 361.2)
- added C4: 10uF, SM0805_big, F.Cu at (129.0, 23.0)
- added C4: 10uF, SM0805_big, F.Cu at (53.0, 52.0)
- added C5: 100nF, SM0603_big, F.Cu at (134.5, 59.5)
- added C5: 100nF, SM0603_big, F.Cu at (134.5, 29.5)
- added C5: 100nF, SM0603_big, F.Cu at (47.5, 45.5)
- added C6: 100nF, SM0603_big, F.Cu at (96.5, 67.5)
- added C6: 100nF, SM0603_big, F.Cu at (96.5, 37.5)
- added C6: 100nF, SM0603_big, F.Cu at (85.5, 37.5)
- added D1: LED, SM0603_big, F.Cu at (106.4, 54.0)
- added D1: LED, SM0603_big, F.Cu at (106.4, 24.0)
- added D1: LED, SM0603_big, F.Cu at (75.6, 51.0)
- added D2: LED, SM0603_big, F.Cu at (106.4, 51.6)
- added D2: LED, SM0603_big, F.Cu at (106.4, 21.6)
- added D2: LED, SM0603_big, F.Cu at (75.6, 53.4)
- added IC1: ATMEGA88-A, TQFP32, F.Cu at (108.0, 62.0)
- added IC1: ATMEGA88-A, TQFP32, F.Cu at (108.0, 32.0)
- added IC1: ATMEGA88-A, TQFP32, F.Cu at (74.0, 43.0)
- added J1: RJ45, RJ45_8P8_simple, F.Cu at (36.0, 105.0)
- added J1: RJ45, RJ45_8P8_simple, F.Cu at (415.0, 217.0)
- added J1: RJ45, RJ45_8P8_simple, F.Cu at (36.0, 75.0)
- added J1: RJ45, RJ45_8P8_simple, F.Cu at (363.0, 74.0)
- added J1: RJ45, RJ45_8P8_simple, F.Cu at (98.0, 90.0)
- added J1: RJ45, RJ45_8P8_simple, F.Cu at (147.0, 60.0)
- added J1: RJ45, RJ45_8P8_simple, F.Cu at (425.0, 89.0)
- added J1: RJ45, RJ45_8P8_simple, F.Cu at (390.0, 363.0)
- added J1: RJ45, RJ45_8P8_simple, F.Cu at (147.0, 30.0)
- added J1: RJ45, RJ45_8P8_simple, F.Cu at (35.0, 45.0)
- added P1: ISP, wannenstecker_2x5_rm254, F.Cu at (119.0, 60.0)
- added P1: ISP, wannenstecker_2x5_rm254, F.Cu at (119.0, 30.0)
- added P1: ISP, wannenstecker_2x5_rm254, F.Cu at (63.0, 45.0)
- added P2: UART, Stiftleiste_4x1, F.Cu at (98.6, 65.8)
- added P2: UART, Stiftleiste_4x1, F.Cu at (98.6, 35.8)
- added P2: UART, Stiftleiste_4x1, F.Cu at (83.4, 39.2)
- added R1: 220, SM0603_big, F.Cu at (57.5, 97.8)
- added R1: 220, SM0603_big, F.Cu at (436.5, 209.8)
- added R1: 220, SM0603_big, F.Cu at (57.5, 67.8)
- added R1: 220, SM0603_big, F.Cu at (384.5, 66.8)
- added R1: 220, SM0603_big, F.Cu at (76.5, 97.2)
- added R1: 150, SM0805_big, F.Cu at (111.0, 54.0)
- added R1: 220, SM0603_big, F.Cu at (403.5, 96.2)
- added R1: 220, SM0603_big, F.Cu at (368.5, 370.2)
- added R1: 150, SM0805_big, F.Cu at (111.0, 24.0)
- added R1: 150, SM0805_big, F.Cu at (71.0, 51.0)
- added R2: 22k, SM0603_big, F.Cu at (45.8, 107.5)
- added R2: 22k, SM0603_big, F.Cu at (424.8, 219.5)
- added R2: 22k, SM0603_big, F.Cu at (45.8, 77.5)
- added R2: 22k, SM0603_big, F.Cu at (372.8, 76.5)
- added R2: 22k, SM0603_big, F.Cu at (88.2, 87.5)
- added R2: 150, SM0805_big, F.Cu at (111.0, 51.6)
- added R2: 22k, SM0603_big, F.Cu at (415.2, 86.5)
- added R2: 22k, SM0603_big, F.Cu at (380.2, 360.5)
- added R2: 150, SM0805_big, F.Cu at (111.0, 21.6)
- added R2: 150, SM0805_big, F.Cu at (71.0, 53.4)
- added R3: 22k, SM0603_big, F.Cu at (45.8, 112.5)
- added R3: 22k, SM0603_big, F.Cu at (424.8, 224.5)
- added R3: 22k, SM0603_big, F.Cu at (45.8, 82.5)
- added R3: 22k, SM0603_big, F.Cu at (372.8, 81.5)
- added R3: 22k, SM0603_big, F.Cu at (88.2, 82.5)
- added R3: 10k, SM0603_big, F.Cu at (125.7, 66.0)
- added R3: 22k, SM0603_big, F.Cu at (415.2, 81.5)
- added R3: 22k, SM0603_big, F.Cu at (380.2, 355.5)
- added R3: 10k, SM0603_big, F.Cu at (125.7, 36.0)
- added R3: 10k, SM0603_big, F.Cu at (56.3, 39.0)
- added R4: 120, SM0603_big, F.Cu at (42.0, 110.8)
- added R4: 120, SM0603_big, F.Cu at (421.0, 222.8)
- added R4: 120, SM0603_big, F.Cu at (42.0, 80.8)
- added R4: 120, SM0603_big, F.Cu at (369.0, 79.8)
- added R4: 120, SM0603_big, F.Cu at (92.0, 84.2)
- added R4: 22k, SM0603_big, F.Cu at (132.2, 66.0)
- added R4: 120, SM0603_big, F.Cu at (419.0, 83.2)
- added R4: 120, SM0603_big, F.Cu at (384.0, 357.2)
- added R4: 22k, SM0603_big, F.Cu at (132.2, 36.0)
- added R4: 22k, SM0603_big, F.Cu at (49.8, 39.0)
- added R5: 22k, SM0603_big, F.Cu at (132.0, 53.0)
- added R5: 22k, SM0603_big, F.Cu at (132.0, 23.0)
- added R5: 22k, SM0603_big, F.Cu at (50.0, 52.0)
- added R6: 120, SM0603_big, F.Cu at (134.5, 55.5)
- added R6: 120, SM0603_big, F.Cu at (134.5, 25.5)
- added R6: 120, SM0603_big, F.Cu at (47.5, 49.5)
- added R7: 2k2, SM0603_big, F.Cu at (91.8, 59.4)
- added R7: 2k2, SM0603_big, F.Cu at (91.8, 29.4)
- added R7: 2k2, SM0603_big, F.Cu at (90.2, 45.6)
- added R8: 2k2, SM0603_big, F.Cu at (91.8, 63.2)
- added R8: 2k2, SM0603_big, F.Cu at (91.8, 33.2)
- added R8: 2k2, SM0603_big, F.Cu at (90.2, 41.8)
- added SW1: SW_RESET, Taster_6mm, F.Cu at (140.5, 54.0)
- added SW1: SW_RESET, Taster_6mm, F.Cu at (140.5, 24.0)
- added SW1: SW_RESET, Taster_6mm, F.Cu at (41.5, 51.0)
- added U1: TSIC50XF, Tsic_TO92, F.Cu at (92.5, 105.0)
- added U1: TSIC50XF, Tsic_TO92, F.Cu at (471.5, 217.0)
- added U1: TSIC50XF, Tsic_TO92, F.Cu at (92.5, 75.0)
- added U1: TSIC50XF, Tsic_TO92, F.Cu at (419.5, 74.0)
- added U1: TSIC50XF, Tsic_TO92, F.Cu at (41.5, 90.0)
- added U1: ST485, st485, F.Cu at (130.0, 60.0)
- added U1: TSIC50XF, Tsic_TO92, F.Cu at (368.5, 89.0)
- added U1: TSIC50XF, Tsic_TO92, F.Cu at (333.5, 363.0)
- added U1: ST485, st485, F.Cu at (130.0, 30.0)
- added U1: ST485, st485, F.Cu at (52.0, 45.0)
- added U2: ST485, st485, F.Cu at (51.8, 105.0)
- added U2: ST485, st485, F.Cu at (430.8, 217.0)
- added U2: ST485, st485, F.Cu at (51.8, 75.0)
- added U2: ST485, st485, F.Cu at (378.8, 74.0)
- added U2: ST485, st485, F.Cu at (82.2, 90.0)
- added U2: HYT271, HYT271, F.Cu at (63.5, 60.0)
- added U2: ST485, st485, F.Cu at (409.2, 89.0)
- added U2: ST485, st485, F.Cu at (374.2, 363.0)
- added U2: HYT271, HYT271, F.Cu at (63.5, 30.0)
- added U2: HYT271, HYT271, F.Cu at (118.5, 45.0)
- added m3_loch: VAL**, m3_loch, F.Cu at (60.2, 110.0)
- added m3_loch: VAL**, m3_loch, F.Cu at (139.5, 65.0)
- added m3_loch: VAL**, m3_loch, F.Cu at (416.8, 94.0)
- added m3_loch: VAL**, m3_loch, F.Cu at (400.8, 84.0)
- added m3_loch: VAL**, m3_loch, F.Cu at (365.8, 358.0)
- added m3_loch: VAL**, m3_loch, F.Cu at (381.8, 368.0)
- added m3_loch: VAL**, m3_loch, F.Cu at (98.0, 25.0)
- added m3_loch: VAL**, m3_loch, F.Cu at (139.5, 35.0)
- added m3_loch: VAL**, m3_loch, F.Cu at (84.0, 50.0)
- added m3_loch: VAL**, m3_loch, F.Cu at (42.5, 40.0)
- added m3_loch: VAL**, m3_loch, F.Cu at (44.2, 100.0)
- added m3_loch: VAL**, m3_loch, F.Cu at (423.2, 212.0)
- added m3_loch: VAL**, m3_loch, F.Cu at (439.2, 222.0)
- added m3_loch: VAL**, m3_loch, F.Cu at (60.2, 80.0)
- added m3_loch: VAL**, m3_loch, F.Cu at (44.2, 70.0)
- added m3_loch: VAL**, m3_loch, F.Cu at (371.2, 69.0)
- added m3_loch: VAL**, m3_loch, F.Cu at (387.2, 79.0)
- added m3_loch: VAL**, m3_loch, F.Cu at (73.8, 85.0)
- added m3_loch: VAL**, m3_loch, F.Cu at (89.8, 95.0)
- added m3_loch: VAL**, m3_loch, F.Cu at (98.0, 55.0)
- moved C1 459.0 mm to (498.1, 363.0)
- moved C2 459.0 mm to (511.0, 348.0)
- moved C3 459.0 mm to (514.2, 361.0)
- moved C4 459.0 mm to (514.0, 348.0)
- moved C5 459.0 mm to (519.5, 354.5)
- moved C6 459.0 mm to (481.5, 362.5)
- moved D1 459.0 mm to (491.4, 349.0)
- moved D2 459.0 mm to (491.4, 346.6)
- moved IC1 459.0 mm to (493.0, 357.0)
- moved J1 459.0 mm to (532.0, 355.0)
- moved P1 459.0 mm to (504.0, 355.0)
- moved P2 459.0 mm to (483.6, 360.8)
- moved R1 459.0 mm to (496.0, 349.0)
- moved R2 459.0 mm to (496.0, 346.6)
- moved R3 459.0 mm to (510.7, 361.0)
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Routing:
- net GND: track 5785.4 -> 6304.5 mm, vias 71 -> 75
- net N-000007: track 753.3 -> 1058.4 mm
- net N-0000010: track 632.0 -> 908.5 mm
- net /zb: track 565.0 -> 684.1 mm
- net /RESET: track 655.4 -> 543.9 mm, vias 18 -> 14
- net /za: track 560.8 -> 671.3 mm, vias 6 -> 4
- net /SDA: track 498.6 -> 413.6 mm
- net /SCL: track 520.7 -> 436.3 mm
- net N-000002: track 78.2 -> 37.5 mm
- net /DI: track 111.1 -> 74.1 mm
- net N-000001: track 63.6 -> 30.0 mm
- net N-000004: track 60.3 -> 30.0 mm
- net /MOSI: track 219.5 -> 196.0 mm, vias 12 -> 10
- net /SCK: track 99.6 -> 78.3 mm
- net /RX: track 199.5 -> 179.3 mm
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Other:
- board size 200.1 x 330 mm -> 527 x 353 mm
- board text added: "v1.1"
- board text removed: "SO8"
- board text removed: "V1.1"
