File: hardware/humidity/humidity_board.sch (KiCad schematic (older format))
At the start: 18 parts

Commit message: comments in schematics
Other:
- note added: "100nF FOR DE NOISING"
- note added: "A=1\nB=2"
- note added: "DO WE NEED UART INTERFACE\nFOR DEBUGGING???"
- note added: "DO WE REALLY NEED 2 LEDS?\nI WOULD PREFER UART"
- note added: "NO RC FILTER\n(not in datasheet of hyt)"
- note added: "PERHAPS ONE ADDITIONAL 10uF CAPACITOR\nFOR PEAK CURRENT CONSUMPTION SOMPENSATION"
- note added: "a/b SHOULD BE SWAPPED\n(EASISER ROUTING)\n+ COMPATIBILITY WITH COLLECTOR BOARD"
Changed lines of the file:
@@
 Sheet 1 1
 Title ""
-Date "12 apr 2014"
+Date "28 apr 2014"
 Rev ""
 Comp ""
@@
 Wire Wire Line
 	9700 3450 9700 3600
+Text Notes 6300 4750 0    60   ~ 0
+NO RC FILTER\n(not in datasheet of hyt)
+Text Notes 3550 3100 0    60   ~ 0
+DO WE NEED UART INTERFACE\nFOR DEBUGGING???
+Text Notes 6650 1050 0    60   ~ 0
+PERHAPS ONE ADDITIONAL 10uF CAPACITOR\nFOR PEAK CURRENT CONSUMPTION SOMPENSATION
+Text Notes 850  1150 0    60   ~ 0
+100nF FOR DE NOISING
+Text Notes 750  7450 0    60   ~ 0
+DO WE REALLY NEED 2 LEDS?\nI WOULD PREFER UART
+Text Notes 8750 2300 0    60   ~ 0
+a/b SHOULD BE SWAPPED\n(EASISER ROUTING)\n+ COMPATIBILITY WITH COLLECTOR BOARD
+Text Notes 9950 2600 0    60   ~ 0
+A=1\nB=2
 $EndSCHEMATC
