File: hardware/humidity/humidity_board.sch (KiCad schematic (older format))
At the start: 21 parts

Commit message: modify again
Connections:
- net VCC: now also R?.1
- net zb: now also U?.7 (B); no longer R?.1, R?.1
Other:
- moved on the sheet: C?, R?
Changed lines of the file:
@@
 L R R?
 U 1 1 532DDB70
-P 8250 2650
-F 0 "R?" V 8330 2650 40  0000 C CNN
-F 1 "120" V 8257 2651 40  0000 C CNN
-F 2 "~" V 8180 2650 30  0000 C CNN
-F 3 "~" H 8250 2650 30  0000 C CNN
-	1    8250 2650
+P 8250 2750
+F 0 "R?" V 8330 2750 40  0000 C CNN
+F 1 "120" V 8257 2751 40  0000 C CNN
+F 2 "~" V 8180 2750 30  0000 C CNN
+F 3 "~" H 8250 2750 30  0000 C CNN
+	1    8250 2750
 	1    0    0    -1
 $EndComp
@@
 L C C?
 U 1 1 534938E9
-P 8250 3250
-F 0 "C?" H 8250 3350 40  0000 L CNN
-F 1 "100nF" H 8256 3165 40  0000 L CNN
-F 2 "~" H 8288 3100 30  0000 C CNN
-F 3 "~" H 8250 3250 60  0000 C CNN
-	1    8250 3250
+P 8250 3300
+F 0 "C?" H 8250 3400 40  0000 L CNN
+F 1 "100nF" H 8256 3215 40  0000 L CNN
+F 2 "~" H 8288 3150 30  0000 C CNN
+F 3 "~" H 8250 3300 60  0000 C CNN
+	1    8250 3300
 	-1   0    0    1
 $EndComp
@@
 L R R?
 U 1 1 535D7B1E
-P 7400 2900
-F 0 "R?" V 7480 2900 40  0000 C CNN
-F 1 "22k" V 7407 2901 40  0000 C CNN
-F 2 "~" V 7330 2900 30  0000 C CNN
-F 3 "~" H 7400 2900 30  0000 C CNN
-	1    7400 2900
+P 7400 3000
+F 0 "R?" V 7480 3000 40  0000 C CNN
+F 1 "22k" V 7407 3001 40  0000 C CNN
+F 2 "~" V 7330 3000 30  0000 C CNN
+F 3 "~" H 7400 3000 30  0000 C CNN
+	1    7400 3000
 	1    0    0    -1
 $EndComp
@@
 L R R?
 U 1 1 535D7B2D
-P 7650 2900
-F 0 "R?" V 7730 2900 40  0000 C CNN
-F 1 "22k" V 7657 2901 40  0000 C CNN
-F 2 "~" V 7580 2900 30  0000 C CNN
-F 3 "~" H 7650 2900 30  0000 C CNN
-	1    7650 2900
-	1    0    0    -1
-$EndComp
-$Comp
-L VCC #PWR?
-U 1 1 535D7B5F
-P 7400 2500
-F 0 "#PWR?" H 7400 2600 30  0001 C CNN
-F 1 "VCC" H 7400 2600 30  0000 C CNN
-F 2 "" H 7400 2500 60  0000 C CNN
-F 3 "" H 7400 2500 60  0000 C CNN
-	1    7400 2500
+P 7650 3000
+F 0 "R?" V 7730 3000 40  0000 C CNN
+F 1 "22k" V 7657 3001 40  0000 C CNN
+F 2 "~" V 7580 3000 30  0000 C CNN
+F 3 "~" H 7650 3000 30  0000 C CNN
+	1    7650 3000
 	1    0    0    -1
 $EndComp
@@
 L GND #PWR?
 U 1 1 535D7B6F
-P 7650 3350
-F 0 "#PWR?" H 7650 3350 30  0001 C CNN
-F 1 "GND" H 7650 3280 30  0001 C CNN
-F 2 "" H 7650 3350 60  0000 C CNN
-F 3 "" H 7650 3350 60  0000 C CNN
-	1    7650 3350
+P 7650 3400
+F 0 "#PWR?" H 7650 3400 30  0001 C CNN
+F 1 "GND" H 7650 3330 30  0001 C CNN
+F 2 "" H 7650 3400 60  0000 C CNN
+F 3 "" H 7650 3400 60  0000 C CNN
+	1    7650 3400
 	1    0    0    -1
 $EndComp
@@
 Text Label 8650 3550 0    60   ~ 0
 za
-Text Label 8650 2300 0    60   ~ 0
+Text Label 8650 2500 0    60   ~ 0
 zb
 Text Label 9650 2550 0    60   ~ 0
@@
 	1    0    0    -1
 $EndComp
-Text Label 4550 5300 0    60   ~ 0
+Text Label 4650 5300 2    60   ~ 0
 RX
-Text Label 4550 5400 0    60   ~ 0
+Text Label 4650 5400 2    60   ~ 0
 TX
 Wire Wire Line
-	7100 2500 7200 2500
+	7100 2500 7650 2500
+Wire Wire Line
+	7650 2500 8650 2500
 Wire Wire Line
 	7100 2800 7200 2800
@@
 	7200 2800 7200 3550
 Wire Wire Line
-	7400 2300 7400 2650
-Wire Wire Line
-	8250 2300 8250 2400
-Wire Wire Line
-	6200 850  6200 1600
+	6200 850  6200 1150
+Wire Wire Line
+	6200 1150 6200 1450
+Wire Wire Line
+	6200 1450 6200 1600
 Wire Wire Line
 	6200 3600 6200 4050
@@
 	6850 1450 7050 1450
 Wire Wire Line
-	7050 1150 7050 1650
+	7050 1150 7050 1450
+Wire Wire Line
+	7050 1450 7050 1650
 Wire Wire Line
 	9300 4600 9100 4600
@@
 Connection ~ 9100 4600
 Wire Wire Line
-	4900 1750 4900 2750
+	4900 1750 4900 2550
+Wire Wire Line
+	4900 2550 4900 2750
 Wire Wire Line
 	4900 2550 5300 2550
@@
 	9750 3250 9650 3250
 Wire Wire Line
-	9650 3150 9650 3500
-Connection ~ 8250 2300
-Wire Wire Line
-	9100 4300 9100 4700
+	9650 3150 9650 3250
+Wire Wire Line
+	9650 3250 9650 3500
+Wire Wire Line
+	9100 4300 9100 4600
+Wire Wire Line
+	9100 4600 9100 4700
 Wire Wire Line
 	9100 6650 9100 6400
@@
 	1600 3550 1400 3550
 Wire Wire Line
-	1400 3550 1400 4050
+	1400 3550 1400 3650
+Wire Wire Line
+	1400 3650 1400 3750
+Wire Wire Line
+	1400 3750 1400 4050
 Wire Wire Line
 	1600 3650 1400 3650
@@
 Connection ~ 1400 3750
 Wire Wire Line
-	1450 700  1450 1750
+	1450 700  1450 900
+Wire Wire Line
+	1450 900  1450 1200
+Wire Wire Line
+	1450 1200 1450 1450
+Wire Wire Line
+	1450 1450 1450 1550
+Wire Wire Line
+	1450 1550 1450 1750
 Wire Wire Line
 	1450 1450 1600 1450
@@
 	2950 5150 2800 5150
 Wire Wire Line
-	3000 5350 3000 5800
+	3000 5350 3000 5450
+Wire Wire Line
+	3000 5450 3000 5550
+Wire Wire Line
+	3000 5550 3000 5800
 Wire Wire Line
 	3000 5350 2800 5350
@@
 	2350 6950 2100 6950
 Wire Wire Line
-	7200 3550 8650 3550
-Wire Wire Line
-	8250 3450 8250 3550
+	7200 3550 7400 3550
+Wire Wire Line
+	7400 3550 8250 3550
+Wire Wire Line
+	8250 3550 8650 3550
+Wire Wire Line
+	8250 3500 8250 3550
 Connection ~ 8250 3550
 Wire Wire Line
-	8250 2900 8250 3050
+	8250 3000 8250 3100
 Wire Wire Line
 	10550 3450 10550 3600
 Wire Wire Line
-	7650 3150 7650 3350
-Wire Wire Line
-	7650 2650 7650 2300
-Connection ~ 7650 2300
-Wire Wire Line
-	7400 3150 7400 3550
+	7650 3250 7650 3400
+Wire Wire Line
+	7400 3250 7400 3550
 Connection ~ 7400 3550
 Wire Wire Line
-	9650 2800 9650 2950
+	9650 2800 9650 2850
+Wire Wire Line
+	9650 2850 9650 2950
 Wire Wire Line
 	9650 2850 9750 2850
@@
 Connection ~ 9650 3250
 Wire Wire Line
-	7400 2300 8650 2300
-Wire Wire Line
 	6850 1150 7050 1150
 Connection ~ 7050 1450
@@
 Connection ~ 1450 1200
 Wire Wire Line
-	850  900  850  1950
+	850  900  850  1200
+Wire Wire Line
+	850  1200 850  1950
 Connection ~ 850  1200
 Wire Wire Line
@@
 	6700 6000 6700 6350
 Wire Wire Line
-	6000 6350 6900 6350
+	6000 6350 6700 6350
+Wire Wire Line
+	6700 6350 6900 6350
 Wire Wire Line
 	7500 6350 7800 6350
@@
 Wire Wire Line
 	3800 3150 3500 3150
+$Comp
+L VCC #PWR?
+U 1 1 536003C2
+P 7400 2650
+F 0 "#PWR?" H 7400 2750 30  0001 C CNN
+F 1 "VCC" H 7400 2750 30  0000 C CNN
+F 2 "" H 7400 2650 60  0000 C CNN
+F 3 "" H 7400 2650 60  0000 C CNN
+	1    7400 2650
+	1    0    0    -1
+$EndComp
+Wire Wire Line
+	7400 2650 7400 2750
+Wire Wire Line
+	7650 2750 7650 2500
+Connection ~ 7650 2500
 $EndSCHEMATC

Commit message: again
Connections:
- net za: now also J?.1
- net zb: now also J?.2
Changed lines of the file:
@@
 TX
 Wire Wire Line
-	7100 2500 7650 2500
-Wire Wire Line
-	7650 2500 8650 2500
+	7100 2500 8650 2500
 Wire Wire Line
 	7100 2800 7200 2800
@@
 	7200 2800 7200 3550
 Wire Wire Line
-	6200 850  6200 1150
-Wire Wire Line
-	6200 1150 6200 1450
-Wire Wire Line
-	6200 1450 6200 1600
+	6200 850  6200 1600
 Wire Wire Line
 	6200 3600 6200 4050
@@
 	6850 1450 7050 1450
 Wire Wire Line
-	7050 1150 7050 1450
-Wire Wire Line
-	7050 1450 7050 1650
+	7050 1150 7050 1650
 Wire Wire Line
 	9300 4600 9100 4600
@@
 Connection ~ 9100 4600
 Wire Wire Line
-	4900 1750 4900 2550
-Wire Wire Line
-	4900 2550 4900 2750
+	4900 1750 4900 2750
 Wire Wire Line
 	4900 2550 5300 2550
@@
 	9750 3250 9650 3250
 Wire Wire Line
-	9650 3150 9650 3250
-Wire Wire Line
-	9650 3250 9650 3500
-Wire Wire Line
-	9100 4300 9100 4600
-Wire Wire Line
-	9100 4600 9100 4700
+	9650 3150 9650 3500
+Wire Wire Line
+	9100 4300 9100 4700
 Wire Wire Line
 	9100 6650 9100 6400
@@
 	1600 3550 1400 3550
 Wire Wire Line
-	1400 3550 1400 3650
-Wire Wire Line
-	1400 3650 1400 3750
-Wire Wire Line
-	1400 3750 1400 4050
+	1400 3550 1400 4050
 Wire Wire Line
 	1600 3650 1400 3650
@@
 Connection ~ 1400 3750
 Wire Wire Line
-	1450 700  1450 900
-Wire Wire Line
-	1450 900  1450 1200
-Wire Wire Line
-	1450 1200 1450 1450
-Wire Wire Line
-	1450 1450 1450 1550
-Wire Wire Line
-	1450 1550 1450 1750
+	1450 700  1450 1750
 Wire Wire Line
 	1450 1450 1600 1450
@@
 	2950 5150 2800 5150
 Wire Wire Line
-	3000 5350 3000 5450
-Wire Wire Line
-	3000 5450 3000 5550
-Wire Wire Line
-	3000 5550 3000 5800
+	3000 5350 3000 5800
 Wire Wire Line
 	3000 5350 2800 5350
@@
 	2350 6950 2100 6950
 Wire Wire Line
-	7200 3550 7400 3550
-Wire Wire Line
-	7400 3550 8250 3550
-Wire Wire Line
-	8250 3550 8650 3550
+	7200 3550 8650 3550
 Wire Wire Line
 	8250 3500 8250 3550
@@
 Connection ~ 7400 3550
 Wire Wire Line
-	9650 2800 9650 2850
-Wire Wire Line
-	9650 2850 9650 2950
+	9650 2800 9650 2950
 Wire Wire Line
 	9650 2850 9750 2850
@@
 Connection ~ 1450 1200
 Wire Wire Line
-	850  900  850  1200
-Wire Wire Line
-	850  1200 850  1950
+	850  900  850  1950
 Connection ~ 850  1200
 Wire Wire Line
@@
 	6700 6000 6700 6350
 Wire Wire Line
-	6000 6350 6700 6350
-Wire Wire Line
-	6700 6350 6900 6350
+	6000 6350 6900 6350
 Wire Wire Line
 	7500 6350 7800 6350
@@
 	7650 2750 7650 2500
 Connection ~ 7650 2500
+Wire Wire Line
+	9750 2550 9650 2550
+Wire Wire Line
+	9750 2650 9650 2650
 $EndSCHEMATC

Commit message: begin with pcb
Parts:
- removed U?: ST485, symbol ST485
- added U?: ST485, ~, symbol ST485
- SW1: renamed from SW?; value SW_PUSH -> SW_RESET
- gave numbers to parts that had none: 19
Connections:
- net DI: now also U?.4 (DI)
- net GND: now also U?.5 (GND)
- net VCC: now also U?.2 (nRE), U?.3 (DE), U?.8 (VCC)
- net za: now also U?.6 (A)
- net zb: now also U?.7 (B)

Commit message: add netlist and pcb
Parts:
- gave numbers to parts that had none: 1
Changed lines of the file:
@@
 $EndDescr
 $Comp
-L VCC #PWR01
+L VCC #PWR10
 U 1 1 532DBFEE
 P 4900 1750
-F 0 "#PWR01" H 4900 1850 30  0001 C CNN
+F 0 "#PWR10" H 4900 1850 30  0001 C CNN
 F 1 "VCC" H 4900 1850 30  0000 C CNN
 F 2 "" H 4900 1750 60  0000 C CNN
@@
 $EndComp
 $Comp
-L GND #PWR02
+L GND #PWR12
 U 1 1 532DDBFC
 P 6200 4050
-F 0 "#PWR02" H 6200 4050 30  0001 C CNN
+F 0 "#PWR12" H 6200 4050 30  0001 C CNN
 F 1 "GND" H 6200 3980 30  0001 C CNN
 F 2 "" H 6200 4050 60  0000 C CNN
@@
 $EndComp
 $Comp
-L VCC #PWR03
+L VCC #PWR11
 U 1 1 532DDC02
 P 6200 850
-F 0 "#PWR03" H 6200 950 30  0001 C CNN
+F 0 "#PWR11" H 6200 950 30  0001 C CNN
 F 1 "VCC" H 6200 950 30  0000 C CNN
 F 2 "" H 6200 850 60  0000 C CNN
@@
 $EndComp
 $Comp
-L GND #PWR04
+L GND #PWR14
 U 1 1 532DDC32
 P 7050 1650
-F 0 "#PWR04" H 7050 1650 30  0001 C CNN
+F 0 "#PWR14" H 7050 1650 30  0001 C CNN
 F 1 "GND" H 7050 1580 30  0001 C CNN
 F 2 "" H 7050 1650 60  0000 C CNN
@@
 $EndComp
 $Comp
-L GND #PWR05
+L GND #PWR19
 U 1 1 532DDC5E
 P 9100 6650
-F 0 "#PWR05" H 9100 6650 30  0001 C CNN
+F 0 "#PWR19" H 9100 6650 30  0001 C CNN
 F 1 "GND" H 9100 6580 30  0001 C CNN
 F 2 "" H 9100 6650 60  0000 C CNN
@@
 $EndComp
 $Comp
-L GND #PWR06
+L GND #PWR22
 U 1 1 532DDCAA
 P 10000 5000
-F 0 "#PWR06" H 10000 5000 30  0001 C CNN
+F 0 "#PWR22" H 10000 5000 30  0001 C CNN
 F 1 "GND" H 10000 4930 30  0001 C CNN
 F 2 "" H 10000 5000 60  0000 C CNN
@@
 $EndComp
 $Comp
-L VCC #PWR07
+L VCC #PWR18
 U 1 1 532DDCEC
 P 9100 4300
-F 0 "#PWR07" H 9100 4400 30  0001 C CNN
+F 0 "#PWR18" H 9100 4400 30  0001 C CNN
 F 1 "VCC" H 9100 4400 30  0000 C CNN
 F 2 "" H 9100 4300 60  0000 C CNN
@@
 $EndComp
 $Comp
-L GND #PWR08
+L GND #PWR21
 U 1 1 532DDE77
 P 9650 3500
-F 0 "#PWR08" H 9650 3500 30  0001 C CNN
+F 0 "#PWR21" H 9650 3500 30  0001 C CNN
 F 1 "GND" H 9650 3430 30  0001 C CNN
 F 2 "" H 9650 3500 60  0000 C CNN
@@
 $EndComp
 $Comp
-L GND #PWR09
+L GND #PWR2
 U 1 1 5330251C
 P 1400 4050
-F 0 "#PWR09" H 1400 4050 30  0001 C CNN
+F 0 "#PWR2" H 1400 4050 30  0001 C CNN
 F 1 "GND" H 1400 3980 30  0001 C CNN
 F 2 "" H 1400 4050 60  0000 C CNN
@@
 $EndComp
 $Comp
-L VCC #PWR010
+L VCC #PWR3
 U 1 1 53302620
 P 1450 700
-F 0 "#PWR010" H 1450 800 30  0001 C CNN
+F 0 "#PWR3" H 1450 800 30  0001 C CNN
 F 1 "VCC" H 1450 800 30  0000 C CNN
 F 2 "" H 1450 700 60  0000 C CNN
@@
 MISO
 $Comp
-L GND #PWR011
+L GND #PWR5
 U 1 1 53302A98
 P 3000 5800
-F 0 "#PWR011" H 3000 5800 30  0001 C CNN
+F 0 "#PWR5" H 3000 5800 30  0001 C CNN
 F 1 "GND" H 3000 5730 30  0001 C CNN
 F 2 "" H 3000 5800 60  0000 C CNN
@@
 $EndComp
 $Comp
-L VCC #PWR012
+L VCC #PWR4
 U 1 1 53302A9E
 P 2950 4900
-F 0 "#PWR012" H 2950 5000 30  0001 C CNN
+F 0 "#PWR4" H 2950 5000 30  0001 C CNN
 F 1 "VCC" H 2950 5000 30  0000 C CNN
 F 2 "" H 2950 4900 60  0000 C CNN
@@
 LED2
 $Comp
-L VCC #PWR013
+L VCC #PWR6
 U 1 1 5330344D
 P 3000 6200
-F 0 "#PWR013" H 3000 6300 30  0001 C CNN
+F 0 "#PWR6" H 3000 6300 30  0001 C CNN
 F 1 "VCC" H 3000 6300 30  0000 C CNN
 F 2 "" H 3000 6200 60  0000 C CNN
@@
 $EndComp
 $Comp
-L VCC #PWR014
+L VCC #PWR7
 U 1 1 53303543
 P 3000 6700
-F 0 "#PWR014" H 3000 6800 30  0001 C CNN
+F 0 "#PWR7" H 3000 6800 30  0001 C CNN
 F 1 "VCC" H 3000 6800 30  0000 C CNN
 F 2 "" H 3000 6700 60  0000 C CNN
@@
 $EndComp
 $Comp
-L VCC #PWR015
+L VCC #PWR20
 U 1 1 53493890
 P 9650 2800
-F 0 "#PWR015" H 9650 2900 30  0001 C CNN
+F 0 "#PWR20" H 9650 2900 30  0001 C CNN
 F 1 "VCC" H 9650 2900 30  0000 C CNN
 F 2 "" H 9650 2800 60  0000 C CNN
@@
 $EndComp
 $Comp
-L GND #PWR016
+L GND #PWR23
 U 1 1 53493BBC
 P 10550 3600
-F 0 "#PWR016" H 10550 3600 30  0001 C CNN
+F 0 "#PWR23" H 10550 3600 30  0001 C CNN
 F 1 "GND" H 10550 3530 30  0001 C CNN
 F 2 "" H 10550 3600 60  0000 C CNN
@@
 $EndComp
 $Comp
-L GND #PWR017
+L GND #PWR16
 U 1 1 535D7B6F
 P 7650 3400
-F 0 "#PWR017" H 7650 3400 30  0001 C CNN
+F 0 "#PWR16" H 7650 3400 30  0001 C CNN
 F 1 "GND" H 7650 3330 30  0001 C CNN
 F 2 "" H 7650 3400 60  0000 C CNN
@@
 $EndComp
 $Comp
-L GND #PWR018
+L GND #PWR1
 U 1 1 535FF6E8
 P 850 1950
-F 0 "#PWR018" H 850 1950 30  0001 C CNN
+F 0 "#PWR1" H 850 1950 30  0001 C CNN
 F 1 "GND" H 850 1880 30  0001 C CNN
 F 2 "" H 850 1950 60  0000 C CNN
@@
 RESET
 $Comp
-L VCC #PWR019
+L VCC #PWR13
 U 1 1 535FFA29
 P 6700 5100
-F 0 "#PWR019" H 6700 5200 30  0001 C CNN
+F 0 "#PWR13" H 6700 5200 30  0001 C CNN
 F 1 "VCC" H 6700 5200 30  0000 C CNN
 F 2 "" H 6700 5100 60  0000 C CNN
@@
 $EndComp
 $Comp
-L GND #PWR020
+L GND #PWR17
 U 1 1 535FFA2F
 P 7800 6800
-F 0 "#PWR020" H 7800 6800 30  0001 C CNN
+F 0 "#PWR17" H 7800 6800 30  0001 C CNN
 F 1 "GND" H 7800 6730 30  0001 C CNN
 F 2 "" H 7800 6800 60  0000 C CNN
@@
 $EndComp
 $Comp
-L VCC #PWR021
+L VCC #PWR8
 U 1 1 535FFDF2
 P 4650 4850
-F 0 "#PWR021" H 4650 4950 30  0001 C CNN
+F 0 "#PWR8" H 4650 4950 30  0001 C CNN
 F 1 "VCC" H 4650 4950 30  0000 C CNN
 F 2 "" H 4650 4850 60  0000 C CNN
@@
 $EndComp
 $Comp
-L GND #PWR022
+L GND #PWR9
 U 1 1 535FFDF8
 P 4650 5850
-F 0 "#PWR022" H 4650 5850 30  0001 C CNN
+F 0 "#PWR9" H 4650 5850 30  0001 C CNN
 F 1 "GND" H 4650 5780 30  0001 C CNN
 F 2 "" H 4650 5850 60  0000 C CNN
@@
 TX
 Wire Wire Line
-	7100 2500 7650 2500
-Wire Wire Line
-	7650 2500 8650 2500
+	7100 2500 8650 2500
 Wire Wire Line
 	7100 2800 7200 2800
@@
 	7200 2800 7200 3550
 Wire Wire Line
-	6200 850  6200 1150
-Wire Wire Line
-	6200 1150 6200 1450
-Wire Wire Line
-	6200 1450 6200 1600
+	6200 850  6200 1600
 Wire Wire Line
 	6200 3600 6200 4050
@@
 	6850 1450 7050 1450
 Wire Wire Line
-	7050 1150 7050 1450
-Wire Wire Line
-	7050 1450 7050 1650
+	7050 1150 7050 1650
 Wire Wire Line
 	9300 4600 9100 4600
@@
 Connection ~ 9100 4600
 Wire Wire Line
-	4900 1750 4900 2550
-Wire Wire Line
-	4900 2550 4900 2750
+	4900 1750 4900 2750
 Wire Wire Line
 	4900 2550 5300 2550
@@
 	9750 3250 9650 3250
 Wire Wire Line
-	9650 3150 9650 3250
-Wire Wire Line
-	9650 3250 9650 3500
-Wire Wire Line
-	9100 4300 9100 4600
-Wire Wire Line
-	9100 4600 9100 4700
+	9650 3150 9650 3500
+Wire Wire Line
+	9100 4300 9100 4700
 Wire Wire Line
 	9100 6650 9100 6400
@@
 	1600 3550 1400 3550
 Wire Wire Line
-	1400 3550 1400 3650
-Wire Wire Line
-	1400 3650 1400 3750
-Wire Wire Line
-	1400 3750 1400 4050
+	1400 3550 1400 4050
 Wire Wire Line
 	1600 3650 1400 3650
@@
 Connection ~ 1400 3750
 Wire Wire Line
-	1450 700  1450 900
-Wire Wire Line
-	1450 900  1450 1200
-Wire Wire Line
-	1450 1200 1450 1450
-Wire Wire Line
-	1450 1450 1450 1550
-Wire Wire Line
-	1450 1550 1450 1750
+	1450 700  1450 1750
 Wire Wire Line
 	1450 1450 1600 1450
@@
 	2950 5150 2800 5150
 Wire Wire Line
-	3000 5350 3000 5450
-Wire Wire Line
-	3000 5450 3000 5550
-Wire Wire Line
-	3000 5550 3000 5800
+	3000 5350 3000 5800
 Wire Wire Line
 	3000 5350 2800 5350
@@
 	2350 6950 2100 6950
 Wire Wire Line
-	7200 3550 7400 3550
-Wire Wire Line
-	7400 3550 8250 3550
-Wire Wire Line
-	8250 3550 8650 3550
+	7200 3550 8650 3550
 Wire Wire Line
 	8250 3500 8250 3550
@@
 Connection ~ 7400 3550
 Wire Wire Line
-	9650 2800 9650 2850
-Wire Wire Line
-	9650 2850 9650 2950
+	9650 2800 9650 2950
 Wire Wire Line
 	9650 2850 9750 2850
@@
 Connection ~ 1450 1200
 Wire Wire Line
-	850  900  850  1200
-Wire Wire Line
-	850  1200 850  1950
+	850  900  850  1950
 Connection ~ 850  1200
 Wire Wire Line
@@
 	6700 6000 6700 6350
 Wire Wire Line
-	6000 6350 6700 6350
-Wire Wire Line
-	6700 6350 6900 6350
+	6000 6350 6900 6350
 Wire Wire Line
 	7500 6350 7800 6350
@@
 	3800 3150 3500 3150
 $Comp
-L VCC #PWR023
+L VCC #PWR15
 U 1 1 536003C2
 P 7400 2650
-F 0 "#PWR023" H 7400 2750 30  0001 C CNN
+F 0 "#PWR15" H 7400 2750 30  0001 C CNN
 F 1 "VCC" H 7400 2750 30  0000 C CNN
 F 2 "" H 7400 2650 60  0000 C CNN
@@
 	9750 2650 9650 2650
 $Comp
-L ST485 U?
+L ST485 U1
 U 1 1 53600A20
 P 6200 2650
-F 0 "U?" H 6650 3250 70  0000 C BNN
+F 0 "U1" H 6650 3250 70  0000 C BNN
 F 1 "ST485" H 6600 2100 70  0000 C CNN
 F 2 "~" H 6200 2550 60  0000 C CNN

Commit message: humidity pcb finished
Connections:
- net zb: now also R6.1
Changed lines of the file:
@@
 Sheet 1 1
 Title ""
-Date "29 apr 2014"
+Date "1 may 2014"
 Rev ""
 Comp ""
@@
 TX
 Wire Wire Line
-	7100 2500 8650 2500
+	7100 2500 7650 2500
+Wire Wire Line
+	7650 2500 8250 2500
+Wire Wire Line
+	8250 2500 8650 2500
 Wire Wire Line
 	7100 2800 7200 2800
@@
 	7200 2800 7200 3550
 Wire Wire Line
-	6200 850  6200 1600
+	6200 850  6200 1150
+Wire Wire Line
+	6200 1150 6200 1450
+Wire Wire Line
+	6200 1450 6200 1600
 Wire Wire Line
 	6200 3600 6200 4050
@@
 	6850 1450 7050 1450
 Wire Wire Line
-	7050 1150 7050 1650
+	7050 1150 7050 1450
+Wire Wire Line
+	7050 1450 7050 1650
 Wire Wire Line
 	9300 4600 9100 4600
@@
 Connection ~ 9100 4600
 Wire Wire Line
-	4900 1750 4900 2750
+	4900 1750 4900 2550
+Wire Wire Line
+	4900 2550 4900 2750
 Wire Wire Line
 	4900 2550 5300 2550
@@
 	9750 3250 9650 3250
 Wire Wire Line
-	9650 3150 9650 3500
-Wire Wire Line
-	9100 4300 9100 4700
+	9650 3150 9650 3250
+Wire Wire Line
+	9650 3250 9650 3500
+Wire Wire Line
+	9100 4300 9100 4600
+Wire Wire Line
+	9100 4600 9100 4700
 Wire Wire Line
 	9100 6650 9100 6400
@@
 	1600 3550 1400 3550
 Wire Wire Line
-	1400 3550 1400 4050
+	1400 3550 1400 3650
+Wire Wire Line
+	1400 3650 1400 3750
+Wire Wire Line
+	1400 3750 1400 4050
 Wire Wire Line
 	1600 3650 1400 3650
@@
 Connection ~ 1400 3750
 Wire Wire Line
-	1450 700  1450 1750
+	1450 700  1450 900
+Wire Wire Line
+	1450 900  1450 1200
+Wire Wire Line
+	1450 1200 1450 1450
+Wire Wire Line
+	1450 1450 1450 1550
+Wire Wire Line
+	1450 1550 1450 1750
 Wire Wire Line
 	1450 1450 1600 1450
@@
 	2950 5150 2800 5150
 Wire Wire Line
-	3000 5350 3000 5800
+	3000 5350 3000 5450
+Wire Wire Line
+	3000 5450 3000 5550
+Wire Wire Line
+	3000 5550 3000 5800
 Wire Wire Line
 	3000 5350 2800 5350
@@
 	2350 6950 2100 6950
 Wire Wire Line
-	7200 3550 8650 3550
+	7200 3550 7400 3550
+Wire Wire Line
+	7400 3550 8250 3550
+Wire Wire Line
+	8250 3550 8650 3550
 Wire Wire Line
 	8250 3500 8250 3550
@@
 Connection ~ 7400 3550
 Wire Wire Line
-	9650 2800 9650 2950
+	9650 2800 9650 2850
+Wire Wire Line
+	9650 2850 9650 2950
 Wire Wire Line
 	9650 2850 9750 2850
@@
 Connection ~ 1450 1200
 Wire Wire Line
-	850  900  850  1950
+	850  900  850  1200
+Wire Wire Line
+	850  1200 850  1950
 Connection ~ 850  1200
 Wire Wire Line
@@
 	6700 6000 6700 6350
 Wire Wire Line
-	6000 6350 6900 6350
+	6000 6350 6700 6350
+Wire Wire Line
+	6700 6350 6900 6350
 Wire Wire Line
 	7500 6350 7800 6350
@@
 	1    0    0    -1
 $EndComp
+Connection ~ 8250 2500
 $EndSCHEMATC
