File: hardware/3x127_254_adapter/3x127_254_adapter.kicad_pcb (KiCad board)
At the start: 2 copper layers, 9.9 x 8.1 mm, 2 parts, among them K1 CONN_3, K2 CONN_3

Commit message: moved modules
Parts:
- moved K2 406.6 mm to (386.6, 253.5)
- moved K1 406.6 mm to (391.7, 253.5)
Changed lines of the file:
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@@
   )
   (module Tsic_TO92 (layer F.Cu)
-    (at 48.26 27.94 270)
+    (at 386.588 253.492 270)
     (fp_text reference K2 (at 0 4.064 270) (layer F.SilkS)
       (effects (font (size 1 1) (thickness 0.15)))
@@
   )
   (module Stiftleiste_3x1 (layer F.Cu)
-    (at 53.34 27.94 90)
+    (at 391.668 253.492 90)
     (fp_text reference K1 (at 0 -2.032 90) (layer F.SilkS)
       (effects (font (size 1 1) (thickness 0.15)))
@@
     )
   )
-  (gr_line (start 54.864 32.004) (end 54.864 23.876) (angle 90) (layer Edge.Cuts) (width 0.1))
-  (gr_line (start 50.8 32.004) (end 54.864 32.004) (angle 90) (layer Edge.Cuts) (width 0.1))
-  (gr_line (start 49.53 30.734) (end 50.8 32.004) (angle 90) (layer Edge.Cuts) (width 0.1))
-  (gr_line (start 44.958 30.734) (end 49.53 30.734) (angle 90) (layer Edge.Cuts) (width 0.1))
-  (gr_line (start 44.958 25.146) (end 44.958 30.734) (angle 90) (layer Edge.Cuts) (width 0.1))
-  (gr_line (start 49.53 25.146) (end 44.958 25.146) (angle 90) (layer Edge.Cuts) (width 0.1))
-  (gr_line (start 50.8 23.876) (end 49.53 25.146) (angle 90) (layer Edge.Cuts) (width 0.1))
-  (gr_line (start 54.864 23.876) (end 50.8 23.876) (angle 90) (layer Edge.Cuts) (width 0.1))
-  (segment (start 46.348 26.67) (end 49.53 26.67) (width 0.6) (layer F.Cu) (net 1) (status 400000))
-  (segment (start 50.8 25.4) (end 53.34 25.4) (width 0.6) (layer F.Cu) (net 1) (status 800000))
-  (segment (start 49.53 26.67) (end 50.8 25.4) (width 0.6) (layer F.Cu) (net 1))
-  (segment (start 46.348 27.94) (end 53.34 27.94) (width 0.6) (layer F.Cu) (net 2) (status C00000))
-  (segment (start 46.348 29.21) (end 49.53 29.21) (width 0.6) (layer F.Cu) (net 3) (status 400000))
-  (segment (start 50.8 30.48) (end 53.34 30.48) (width 0.6) (layer F.Cu) (net 3) (status 800000))
-  (segment (start 49.53 29.21) (end 50.8 30.48) (width 0.6) (layer F.Cu) (net 3))
+  (gr_line (start 393.192 257.556) (end 393.192 249.428) (angle 90) (layer Edge.Cuts) (width 0.1))
+  (gr_line (start 389.128 257.556) (end 393.192 257.556) (angle 90) (layer Edge.Cuts) (width 0.1))
+  (gr_line (start 387.858 256.286) (end 389.128 257.556) (angle 90) (layer Edge.Cuts) (width 0.1))
+  (gr_line (start 383.286 256.286) (end 387.858 256.286) (angle 90) (layer Edge.Cuts) (width 0.1))
+  (gr_line (start 383.286 250.698) (end 383.286 256.286) (angle 90) (layer Edge.Cuts) (width 0.1))
+  (gr_line (start 387.858 250.698) (end 383.286 250.698) (angle 90) (layer Edge.Cuts) (width 0.1))
+  (gr_line (start 389.128 249.428) (end 387.858 250.698) (angle 90) (layer Edge.Cuts) (width 0.1))
+  (gr_line (start 393.192 249.428) (end 389.128 249.428) (angle 90) (layer Edge.Cuts) (width 0.1))
+  (segment (start 384.676 252.222) (end 387.858 252.222) (width 0.6) (layer F.Cu) (net 1))
+  (segment (start 389.128 250.952) (end 391.668 250.952) (width 0.6) (layer F.Cu) (net 1))
+  (segment (start 387.858 252.222) (end 389.128 250.952) (width 0.6) (layer F.Cu) (net 1))
+  (segment (start 384.676 253.492) (end 391.668 253.492) (width 0.6) (layer F.Cu) (net 2))
+  (segment (start 384.676 254.762) (end 387.858 254.762) (width 0.6) (layer F.Cu) (net 3))
+  (segment (start 389.128 256.032) (end 391.668 256.032) (width 0.6) (layer F.Cu) (net 3))
+  (segment (start 387.858 254.762) (end 389.128 256.032) (width 0.6) (layer F.Cu) (net 3))
 )
