File: hardware/4x127_254_adapter/4x127_254_adapter.kicad_pcb (KiCad board)
At the start: 2 copper layers, 8.1 x 10.7 mm, 2 parts, among them P1 CONN_4, P2 CONN_4

Commit message: moved modules
Parts:
- moved P1 420.3 mm to (394.2, 240.3)
- moved P2 420.3 mm to (399.3, 240.3)
Changed lines of the file:
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@@
     (links 4)
     (no_connects 0)
-    (area 0 0 0 0)
+    (area 28.762 19.990999 41.215 30.878214)
     (thickness 1.6)
     (drawings 8)
@@
     (pad_to_mask_clearance 0)
     (aux_axis_origin 0 0)
-    (visible_elements FFFFFFBF)
+    (visible_elements 7FFFFFFF)
     (pcbplotparams
       (layerselection 3178497)
@@
   )
   (module Stiftleiste_4x1 (layer F.Cu)
-    (at 38.1 25.4 90)
+    (at 399.288 240.284 90)
     (fp_text reference P2 (at 0 -2.032 90) (layer F.SilkS)
       (effects (font (size 1 1) (thickness 0.15)))
@@
   )
   (module HYT271 (layer F.Cu)
-    (at 33.02 25.4 270)
+    (at 394.208 240.284 270)
     (fp_text reference P1 (at 0 3.429 270) (layer F.SilkS)
       (effects (font (size 1 1) (thickness 0.15)))
@@
     )
   )
-  (gr_line (start 39.624 30.734) (end 39.624 20.066) (angle 90) (layer Edge.Cuts) (width 0.1))
-  (gr_line (start 35.814 30.734) (end 39.624 30.734) (angle 90) (layer Edge.Cuts) (width 0.1))
-  (gr_line (start 34.036 28.956) (end 35.814 30.734) (angle 90) (layer Edge.Cuts) (width 0.1))
-  (gr_line (start 31.496 28.956) (end 34.036 28.956) (angle 90) (layer Edge.Cuts) (width 0.1))
-  (gr_line (start 31.496 21.844) (end 31.496 28.956) (angle 90) (layer Edge.Cuts) (width 0.1))
-  (gr_line (start 34.036 21.844) (end 31.496 21.844) (angle 90) (layer Edge.Cuts) (width 0.1))
-  (gr_line (start 35.814 20.066) (end 34.036 21.844) (angle 90) (layer Edge.Cuts) (width 0.1))
-  (gr_line (start 39.624 20.066) (end 35.814 20.066) (angle 90) (layer Edge.Cuts) (width 0.1))
-  (segment (start 32.893 27.305) (end 34.163 27.305) (width 0.6) (layer F.Cu) (net 1))
-  (segment (start 36.068 29.21) (end 38.1 29.21) (width 0.6) (layer F.Cu) (net 1))
-  (segment (start 34.163 27.305) (end 36.068 29.21) (width 0.6) (layer F.Cu) (net 1))
-  (segment (start 32.893 26.035) (end 35.179 26.035) (width 0.6) (layer F.Cu) (net 2) (status 400000))
-  (segment (start 35.814 26.67) (end 38.1 26.67) (width 0.6) (layer F.Cu) (net 2) (status 800000))
-  (segment (start 35.179 26.035) (end 35.814 26.67) (width 0.6) (layer F.Cu) (net 2))
-  (segment (start 32.893 24.765) (end 35.179 24.765) (width 0.6) (layer F.Cu) (net 3))
-  (segment (start 35.814 24.13) (end 38.1 24.13) (width 0.6) (layer F.Cu) (net 3))
-  (segment (start 35.179 24.765) (end 35.814 24.13) (width 0.6) (layer F.Cu) (net 3))
-  (segment (start 32.893 23.495) (end 34.163 23.495) (width 0.6) (layer F.Cu) (net 4))
-  (segment (start 36.068 21.59) (end 38.1 21.59) (width 0.6) (layer F.Cu) (net 4))
-  (segment (start 34.163 23.495) (end 36.068 21.59) (width 0.6) (layer F.Cu) (net 4))
+  (gr_line (start 400.812 245.618) (end 400.812 234.95) (angle 90) (layer Edge.Cuts) (width 0.1))
+  (gr_line (start 397.002 245.618) (end 400.812 245.618) (angle 90) (layer Edge.Cuts) (width 0.1))
+  (gr_line (start 395.224 243.84) (end 397.002 245.618) (angle 90) (layer Edge.Cuts) (width 0.1))
+  (gr_line (start 392.684 243.84) (end 395.224 243.84) (angle 90) (layer Edge.Cuts) (width 0.1))
+  (gr_line (start 392.684 236.728) (end 392.684 243.84) (angle 90) (layer Edge.Cuts) (width 0.1))
+  (gr_line (start 395.224 236.728) (end 392.684 236.728) (angle 90) (layer Edge.Cuts) (width 0.1))
+  (gr_line (start 397.002 234.95) (end 395.224 236.728) (angle 90) (layer Edge.Cuts) (width 0.1))
+  (gr_line (start 400.812 234.95) (end 397.002 234.95) (angle 90) (layer Edge.Cuts) (width 0.1))
+  (segment (start 394.081 242.189) (end 395.351 242.189) (width 0.6) (layer F.Cu) (net 1))
+  (segment (start 397.256 244.094) (end 399.288 244.094) (width 0.6) (layer F.Cu) (net 1))
+  (segment (start 395.351 242.189) (end 397.256 244.094) (width 0.6) (layer F.Cu) (net 1))
+  (segment (start 394.081 240.919) (end 396.367 240.919) (width 0.6) (layer F.Cu) (net 2))
+  (segment (start 397.002 241.554) (end 399.288 241.554) (width 0.6) (layer F.Cu) (net 2))
+  (segment (start 396.367 240.919) (end 397.002 241.554) (width 0.6) (layer F.Cu) (net 2))
+  (segment (start 394.081 239.649) (end 396.367 239.649) (width 0.6) (layer F.Cu) (net 3))
+  (segment (start 397.002 239.014) (end 399.288 239.014) (width 0.6) (layer F.Cu) (net 3))
+  (segment (start 396.367 239.649) (end 397.002 239.014) (width 0.6) (layer F.Cu) (net 3))
+  (segment (start 394.081 238.379) (end 395.351 238.379) (width 0.6) (layer F.Cu) (net 4))
+  (segment (start 397.256 236.474) (end 399.288 236.474) (width 0.6) (layer F.Cu) (net 4))
+  (segment (start 395.351 238.379) (end 397.256 236.474) (width 0.6) (layer F.Cu) (net 4))
 )
