File: hardware/arduino_adapter/main.kicad_pcb (KiCad board)
At the start: 2 copper layers, 60 x 65 mm, 15 parts, among them P1 CONN_8, P10 CONN_10, P11 CONN_8, P2 CONN_6, P3 CONN_6, P4 CONN_8, P5 POW, P6 TWI, P7 TWI_POW, P8 CONN_10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

Commit message: again
Parts:
- moved D1 1.50 mm to (95.0, 106.5)
- moved P5 1.50 mm to (90.0, 107.5)
- moved P6 1.50 mm to (104.5, 106.0)
- moved P7 1.50 mm to (75.0, 106.0)
- moved R1 1.50 mm to (94.0, 103.0)
- moved R2 1.50 mm to (84.5, 103.5)
- moved R3 1.50 mm to (87.0, 103.5)
Routing:
- net GND: track 164.8 -> 168.3 mm
- net VCC: track 95.0 -> 97.0 mm
- net /SDA: track 108.1 -> 109.6 mm
- net /LED: track 37.2 -> 38.7 mm
- net /SCL: track 104.3 -> 105.8 mm
Other:
- board size 60 x 65 mm -> 60 x 66.5 mm
