File: hardware/order/order.kicad_pcb (KiCad board)
At the start: 2 copper layers, 971 x 704.8 mm, 747 parts, among them IC1 ATMEGA88-A, IC1 ATMEGA88A-A, J1 RJ45, J1 RJ45_8P8C_8FACH, K1 pow_sel, P1 ISP, P1 UART, P2 Shield, P2 UART, P3 i2c_pow, P4 i2c_chain, P5 12Vin, P6 HOHLBUCHSE, P7 Vccin, P8 ISP, P9 5Vin, SW1 SW1, SW1 SW_RESET, SW2 SCHALTER_2POL, SW3 SW_RESET, U1 LM7805, U1 ST485, U1 TSIC50XF, U2 HYT271, U2 ST485, U3 ST485, U4 ST485, U5 ST485, U6 ST485, U7 ST485, U8 ST485, U9 ST485, X1 20MHz, m3_loch VAL**

Commit message: moved modules
Parts:
- added C1: 10u, SM0805_big, F.Cu at (44.0, 155.8)
- added C10: 100n, SM0603_big, F.Cu at (81.8, 123.8)
- added C11: 100n, SM0603_big, F.Cu at (67.8, 123.8)
- added C12: 100n, SM0603_big, F.Cu at (53.8, 123.8)
- added C13: 100n, SM0603_big, F.Cu at (39.8, 123.8)
- added C14: 100n, SM0603_big, F.Cu at (25.8, 123.8)
- added C15: 100n, SM0603_big, F.Cu at (17.2, 120.4)
- added C16: 100n, SM0603_big, F.Cu at (31.2, 120.4)
- added C17: 100n, SM0603_big, F.Cu at (45.2, 120.4)
- added C18: 100n, SM0603_big, F.Cu at (59.2, 120.4)
- added C19: 100n, SM0603_big, F.Cu at (73.2, 120.4)
- added C2: 100n, SM0603_big, F.Cu at (80.4, 147.8)
- added C20: 100n, SM0603_big, F.Cu at (87.2, 120.4)
- added C21: 100n, SM0603_big, F.Cu at (101.2, 120.2)
- added C22: 100n, SM0603_big, F.Cu at (115.2, 120.2)
- added C23: 10u, SM0805_big, F.Cu at (44.0, 150.6)
- added C24: 10u, SM0805_big, F.Cu at (44.0, 153.2)
- added C25: 100n, SM0603_big, F.Cu at (19.4, 134.4)
- added C26: 100n, SM0603_big, F.Cu at (31.2, 134.2)
- added C27: 100n, SM0603_big, F.Cu at (45.1, 134.1)
- added C28: 100n, SM0603_big, F.Cu at (59.1, 134.1)
- added C29: 100n, SM0603_big, F.Cu at (75.7, 134.3)
- added C3: 22p, SM0603_big, F.Cu at (58.1, 146.8)
- added C30: 100n, SM0603_big, F.Cu at (87.2, 134.1)
- added C31: 100n, SM0603_big, F.Cu at (101.3, 134.1)
- added C32: 100n, SM0603_big, F.Cu at (115.2, 134.3)
- added C4: 22p, SM0603_big, F.Cu at (58.1, 152.0)
- added C5: 330nF, SM0603_big, F.Cu at (9.40, 123.6)
- added C6: 100nF, SM0603_big, F.Cu at (4.40, 123.6)
- added C7: 100n, SM0603_big, F.Cu at (123.8, 123.8)
- added C8: 100n, SM0603_big, F.Cu at (109.8, 123.8)
- added C9: 100n, SM0603_big, F.Cu at (95.8, 123.8)
- added D1: LED1, SM0603_big, F.Cu at (84.8, 149.4)
- added D2: LED2, SM0603_big, F.Cu at (87.2, 149.4)
- added D3: LED3, SM0603_big, F.Cu at (89.6, 149.4)
- added D4: LED4, SM0603_big, F.Cu at (92.0, 149.4)
- added D5: LED_POW, SM0603_big, F.Cu at (44.0, 145.6)
- added IC1: ATMEGA88A-A, TQFP32, F.Cu at (73.0, 147.0)
- added J1: RJ45_8P8C_8FACH, RJ45_8P8C_8x, F.Cu at (69.0, 103.0)
- added K1: pow_sel, Stiftleiste_3x1, F.Cu at (33.0, 152.0)
- added K1: CONN_3, Stiftleiste_3x1, F.Cu at (301.7, 43.5)
- added K2: CONN_3, Tsic_TO92, F.Cu at (296.6, 43.5)
- added P1: CONN_4, Stiftleiste_4x1, F.Cu at (6.66, 15.3)
- added P1: CONN_4, Stiftleiste_4x1, F.Cu at (232.7, 47.3)
- added P1: CONN_4, HYT271, F.Cu at (269.2, 41.3)
- added P1: UART, Stiftleiste_4x1, F.Cu at (58.0, 160.0)
- added P2: so8, st485, F.Cu at (6.66, 10.9)
- added P2: so8, st485, F.Cu at (232.7, 42.9)
- added P2: CONN_4, Stiftleiste_4x1, F.Cu at (274.3, 41.3)
- added P2: Shield, m3_scheibe, F.Cu at (5.00, 107.0)
- added P3: CONN_4, Stiftleiste_4x1, F.Cu at (6.66, 2.63)
- added P3: i2c_pow, wannenstecker_2x3_rm254, F.Cu at (119.5, 160.0)
- added P3: CONN_4, Stiftleiste_4x1, F.Cu at (232.7, 34.6)
- added P4: i2c_chain, wannenstecker_2x3_rm254, F.Cu at (101.5, 160.0)
- added P5: 12Vin, LPV_Stiftleiste_2pol, F.Cu at (30.0, 160.0)
- added P6: HOHLBUCHSE, hohlbuchse_475_17, F.Cu at (20.0, 158.0)
- added P7: Vccin, LPV_Stiftleiste_2pol, F.Cu at (44.0, 160.0)
- added P8: ISP, wannenstecker_2x5_rm254, F.Cu at (80.5, 160.0)
- added P9: 5Vin, LPV_Stiftleiste_2pol, F.Cu at (37.0, 160.0)
- added R1: 10k, SM0603_big, F.Cu at (99.2, 151.4)
- added R10: 22k, SM0603_big, F.Cu at (116.8, 130.8)
- added R11: 22k, SM0603_big, F.Cu at (102.8, 130.8)
- added R12: 22k, SM0603_big, F.Cu at (88.8, 130.8)
- added R13: 22k, SM0603_big, F.Cu at (74.8, 130.8)
- added R14: 22k, SM0603_big, F.Cu at (126.8, 130.8)
- added R15: 22k, SM0603_big, F.Cu at (112.8, 130.8)
- added R16: 22k, SM0603_big, F.Cu at (98.8, 130.8)
- added R17: 22k, SM0603_big, F.Cu at (84.8, 130.8)
- added R18: 120, SM0603_big, F.Cu at (119.8, 123.8)
- added R19: 120, SM0603_big, F.Cu at (105.8, 123.8)
- added R2: 150, SM0805_big, F.Cu at (84.8, 144.4)
- added R20: 120, SM0603_big, F.Cu at (91.6, 123.8)
- added R21: 120, SM0603_big, F.Cu at (77.8, 123.8)
- added R22: 22k, SM0603_big, F.Cu at (60.8, 130.8)
- added R23: 22k, SM0603_big, F.Cu at (46.8, 130.8)
- added R24: 22k, SM0603_big, F.Cu at (32.8, 130.8)
- added R25: 22k, SM0603_big, F.Cu at (18.8, 130.8)
- added R26: 22k, SM0603_big, F.Cu at (70.8, 130.8)
- added R27: 22k, SM0603_big, F.Cu at (56.8, 130.8)
- added R28: 22k, SM0603_big, F.Cu at (42.8, 130.8)
- added R29: 22k, SM0603_big, F.Cu at (28.8, 130.8)
- added R3: 150, SM0805_big, F.Cu at (87.2, 144.4)
- added R30: 120, SM0603_big, F.Cu at (63.8, 123.8)
- added R31: 120, SM0603_big, F.Cu at (49.8, 123.8)
- added R32: 120, SM0603_big, F.Cu at (35.8, 123.8)
- added R33: 120, SM0603_big, F.Cu at (21.8, 123.8)
- added R34: 0, SM0805_big, F.Cu at (5.00, 116.8)
- added R4: 150, SM0805_big, F.Cu at (89.6, 144.4)
- added R5: 150, SM0805_big, F.Cu at (92.0, 144.4)
- added R6: 2k2, SM0603_big, F.Cu at (105.4, 145.4)
- added R7: 2k2, SM0603_big, F.Cu at (115.4, 145.4)
- added R8: 150, SM0805_big, F.Cu at (44.0, 148.0)
- added R9: 10k, SM0603_big, F.Cu at (72.0, 135.0)
- added SW1: SW1, Taster_6mm, F.Cu at (99.2, 147.0)
- added SW2: SCHALTER_2POL, DIP_Schalter_2pol, F.Cu at (110.4, 148.2)
- added SW3: SW_RESET, Taster_6mm, F.Cu at (121.6, 147.0)
- added U1: LM7805, lm7805_lying, F.Cu at (7.00, 146.0)
- added U2: ST485, st485, F.Cu at (121.8, 131.8)
- added U3: ST485, st485, F.Cu at (107.8, 131.8)
- added U4: ST485, st485, F.Cu at (93.8, 131.8)
- added U5: ST485, st485, F.Cu at (79.8, 131.8)
- added U6: ST485, st485, F.Cu at (65.8, 131.8)
- added U7: ST485, st485, F.Cu at (51.8, 131.8)
- added U8: ST485, st485, F.Cu at (37.8, 131.8)
- added U9: ST485, st485, F.Cu at (23.8, 131.8)
- added X1: 20MHz, HC-49_quarz_big, F.Cu at (63.3, 149.4)
- added m3_loch: VAL**, m3_loch, F.Cu at (5.00, 159.0)
- added m3_loch: VAL**, m3_loch, F.Cu at (132.0, 159.0)
- added m3_loch: VAL**, m3_loch, F.Cu at (132.0, 107.0)
- moved C1 614.4 mm to (646.0, 278.8)
- moved C10 614.4 mm to (683.8, 246.8)
- moved C11 614.4 mm to (669.8, 246.8)
- moved C12 614.4 mm to (655.8, 246.8)
- moved C13 614.4 mm to (641.8, 246.8)
- moved C14 614.4 mm to (627.8, 246.8)
- moved C15 614.4 mm to (619.2, 243.4)
- moved C16 614.4 mm to (633.2, 243.4)
- moved C17 614.4 mm to (647.2, 243.4)
- moved C18 614.4 mm to (661.2, 243.4)
- moved C19 614.4 mm to (675.2, 243.4)
- moved C2 614.4 mm to (682.4, 270.8)
- moved C20 614.4 mm to (689.2, 243.4)
- moved C21 614.4 mm to (703.2, 243.2)
- moved C22 614.4 mm to (717.2, 243.2)
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Routing:
- net GND: track 6642.6 -> 7525.9 mm, vias 108 -> 111
- net VCC: track 4625.9 -> 5182.4 mm, vias 93 -> 96
- net /Vi2c: track 292.4 -> 438.6 mm, vias 2 -> 3
- net /RESET: track 883.3 -> 990.2 mm, vias 28 -> 30
- net /SCL: track 657.3 -> 746.5 mm, vias 4 -> 6
- net /SDA: track 653.5 -> 734.7 mm, vias 4 -> 6
- net /Vreg: track 130.2 -> 195.3 mm
- net /ZAC_08: track 127.4 -> 191.1 mm
- net +12V: track 107.5 -> 161.3 mm
- net /MOSI: track 240.5 -> 290.1 mm, vias 16 -> 18
- net /TX: track 170.8 -> 219.4 mm, vias 4 -> 6
- net /ZAC_01: track 94.4 -> 141.6 mm
- net /RX: track 213.4 -> 259.8 mm, vias 4 -> 6
- net /SW1: track 85.0 -> 127.6 mm
- net /ZAC_07: track 73.4 -> 110.1 mm
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Other:
- board size 971 x 704.8 mm -> 1327 x 704.8 mm
- net class Default: trace_width 0.7 -> 0.6; via_dia 1.2 -> 0.889; via_drill 0.6 -> 0.635
- net class uc removed
- board text added: "SO8"

Commit message: moved again...
Parts:
- added K1: CONN_3, Stiftleiste_3x1, F.Cu at (159.7, 56.5)
- added K1: CONN_3, Stiftleiste_3x1, F.Cu at (151.7, 87.5)
- added K2: CONN_3, Tsic_TO92, F.Cu at (154.6, 56.5)
- added K2: CONN_3, Tsic_TO92, F.Cu at (146.6, 87.5)
- added P1: CONN_4, HYT271, F.Cu at (164.2, 1.71)
- added P1: CONN_4, Stiftleiste_4x1, F.Cu at (163.7, 25.3)
- added P1: CONN_4, Stiftleiste_4x1, F.Cu at (163.7, 43.3)
- added P1: CONN_4, HYT271, F.Cu at (153.2, 68.3)
- added P1: CONN_4, Stiftleiste_4x1, F.Cu at (193.7, 94.3)
- added P1: CONN_4, HYT271, F.Cu at (147.2, 95.7)
- added P1: CONN_4, HYT271, F.Cu at (248.2, 90.7)
- added P1: CONN_4, Stiftleiste_4x1, F.Cu at (270.3, 43.3)
- added P2: CONN_4, Stiftleiste_4x1, F.Cu at (164.2, 6.79)
- added P2: so8, st485, F.Cu at (163.7, 20.9)
- added P2: so8, st485, F.Cu at (163.7, 38.9)
- added P2: CONN_4, Stiftleiste_4x1, F.Cu at (158.3, 68.3)
- added P2: so8, st485, F.Cu at (193.7, 89.9)
- added P2: CONN_4, Stiftleiste_4x1, F.Cu at (147.2, 100.8)
- added P2: CONN_4, Stiftleiste_4x1, F.Cu at (248.2, 95.8)
- added P2: so8, st485, F.Cu at (265.9, 43.3)
- added P3: CONN_4, Stiftleiste_4x1, F.Cu at (163.7, 12.6)
- added P3: CONN_4, Stiftleiste_4x1, F.Cu at (163.7, 30.6)
- added P3: CONN_4, Stiftleiste_4x1, F.Cu at (193.7, 81.6)
- added P3: CONN_4, Stiftleiste_4x1, F.Cu at (257.6, 43.3)
- moved C1 326.0 mm to (190.5, 55.1)
- moved C1 326.0 mm to (159.0, 98.8)
- moved C2 326.0 mm to (175.5, 42.2)
- moved C2 326.0 mm to (174.0, 111.7)
- moved C3 326.0 mm to (188.5, 39.0)
- moved C3 326.0 mm to (161.0, 115.0)
- moved C4 326.0 mm to (175.5, 39.2)
- moved C4 326.0 mm to (174.0, 114.7)
- moved C5 326.0 mm to (182.0, 33.7)
- moved C5 326.0 mm to (167.5, 120.2)
- moved C6 326.0 mm to (190.0, 71.7)
- moved C6 326.0 mm to (159.5, 82.2)
- moved D1 326.0 mm to (176.5, 61.8)
- moved D1 326.0 mm to (173.0, 92.1)
- moved D2 326.0 mm to (174.1, 61.8)
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Routing:
- net N-000002: track 21.3 -> 74.8 mm
- net N-000001: track 20.6 -> 73.7 mm
- net N-000003: track 64.1 -> 114.7 mm
- net N-000004: track 15.1 -> 57.4 mm
- net N-000008: track 20.5 -> 38.9 mm
- net N-000006: track 8.63 -> 25.9 mm
- net N-000005: track 7.04 -> 21.1 mm
- net N-000007: track 974.2 -> 987.8 mm
Other:
- outline, holes or cut-outs redrawn
- net class Default: trace_width 0.6 -> 0.7; via_dia 0.889 -> 1.2; via_drill 0.635 -> 0.6

Commit message: order
Parts:
- removed the R31 at (49.8, 123.8)
- added D1: LED, SM0603_big, F.Cu at (175.0, 158.5)
- added P1: CONN_8, Stiftleiste_8x1, F.Cu at (142.7, 120.2)
- added P10: CONN_10, Stiftleiste_10x1, F.Cu at (197.0, 112.5)
- added P11: CONN_8, Stiftleiste_8x1, F.Cu at (197.0, 138.0)
- added P2: CONN_6, Stiftleiste_6x1, F.Cu at (142.7, 140.5)
- added P3: CONN_6, Stiftleiste_6x1, B.Cu at (145.7, 140.5)
- added P4: CONN_8, Stiftleiste_8x1, B.Cu at (145.7, 120.2)
- added P5: POW, Stiftleiste_2x1, F.Cu at (170.0, 159.5)
- added P6: HOHLBUCHSE, hohlbuchse_475_17, F.Cu at (20.0, 158.0)
- added P6: TWI, wannenstecker_2x3_rm254, F.Cu at (184.5, 158.0)
- added P7: TWI_POW, wannenstecker_2x3_rm254, F.Cu at (155.0, 158.0)
- added P8: CONN_10, Stiftleiste_10x1, B.Cu at (194.0, 113.5)
- added P9: CONN_8, Stiftleiste_8x1, B.Cu at (194.0, 138.0)
- added R1: 150, SM0805_big, F.Cu at (174.0, 155.0)
- added R2: 2k2, SM0603_big, F.Cu at (164.5, 155.5)
- added R3: 2k2, SM0603_big, F.Cu at (167.0, 155.5)
- R31: renamed from P6; value HOHLBUCHSE -> 120; footprint hohlbuchse_475_17 -> SM0603_big
- moved R31 45.4 mm to (49.8, 123.8), turned to 0 degrees
- moved P1 31.4 mm to (264.2, 63.7)
- moved P2 31.4 mm to (264.2, 68.8)
Connections:
- R31 pad 1: +12V -> /z6b
- R31 pad 2: (no net) -> N-0000029
Routing:
- net GND: track 7525.9 -> 7694.2 mm, vias 111 -> 113
- net /SDA: track 734.7 -> 844.3 mm
- net /SCL: track 746.5 -> 852.3 mm, vias 6 -> 8
- net VCC: track 5182.4 -> 5279.4 mm
- net /LED: track 0.00 -> 38.7 mm, vias 0 -> 1
- net N-0000033: track 0.00 -> 3.98 mm
- net N-0000010: track 829.5 -> 833.0 mm
- net N-0000012: track 0.00 -> 3.42 mm
- net N-000008: track 38.9 -> 42.3 mm
- net N-000009: track 0.00 -> 3.42 mm
- net N-0000013: track 0.00 -> 3.42 mm
- net N-0000011: track 0.00 -> 3.42 mm
- net N-0000014: track 25.3 -> 28.7 mm
- net N-000004: track 57.4 -> 60.4 mm
- net N-000007: track 987.8 -> 990.8 mm
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Other:
- outline, holes or cut-outs redrawn
