File: hardware/order2/newOrder.kicad_pcb (KiCad board)
At the start: 2 copper layers, 527 x 353 mm, 706 parts, among them IC1 ATMEGA88-A, IC1 ATMEGA88A-A, J1 RJ45, J1 RJ45_8P8C_8FACH, K1 pow_sel, P1 CONN_4, P1 ISP, P1 UART, P2 CONN_4, P2 Shield, P2 UART, P3 i2c_pow, P4 i2c_chain, P5 12Vin, P6 HOHLBUCHSE, P7 Vccin, P8 ISP, P9 5Vin, SW1 SW1, SW1 SW_RESET, SW2 SCHALTER_2POL, SW3 SW_RESET, U1 LM7805, U1 ST485, U1 TSIC50XF, U2 HYT271, U2 ST485, U3 ST485, U4 ST485, U5 ST485, U6 ST485, U7 ST485, U8 ST485, U9 ST485, X1 20MHz, m3_loch VAL**

Commit message: 23 temperature 2 humility
Parts:
- removed the C1 at (61.5, 97.8)
- removed the C1 at (172.8, 72.5)
- removed the C1 at (202.8, 72.5)
- removed the C1 at (61.5, 67.8)
- removed the C1 at (388.5, 66.8)
- removed the C1 at (72.5, 97.2)
- removed the C1 at (113.1, 68.0)
- removed the C2 at (52.8, 112.2)
- removed the C2 at (187.2, 81.2)
- removed the C2 at (217.2, 81.2)
- removed the C2 at (52.8, 82.2)
- removed the C2 at (379.8, 81.2)
- removed the C2 at (81.2, 82.8)
- removed the C2 at (126.0, 53.0)
- removed the C3 at (49.2, 112.2)
- removed the C3 at (187.2, 84.8)
- removed the C3 at (217.2, 84.8)
- removed the C3 at (49.2, 82.2)
- removed the C3 at (376.2, 81.2)
- removed the C3 at (84.8, 82.8)
- removed the C3 at (129.2, 66.0)
- removed the C4 at (42.0, 106.8)
- removed the C4 at (181.8, 92.0)
- removed the C4 at (211.8, 92.0)
- removed the C4 at (42.0, 76.8)
- removed the C4 at (369.0, 75.8)
- removed the C4 at (92.0, 88.2)
- removed the C4 at (129.0, 53.0)
- removed the C5 at (134.5, 59.5)
- removed the C6 at (96.5, 67.5)
- removed the D1 at (106.4, 54.0)
- removed the D2 at (106.4, 51.6)
- removed the IC1 at (108.0, 62.0)
- removed the J1 at (36.0, 105.0)
- removed the J1 at (180.0, 98.0)
- removed the J1 at (210.0, 98.0)
- removed the J1 at (36.0, 75.0)
- removed the J1 at (363.0, 74.0)
- removed the J1 at (98.0, 90.0)
- removed the J1 at (147.0, 60.0)
- removed the P1 at (119.0, 60.0)
- removed the P1 at (172.6, 45.7)
- removed the P1 at (172.6, 58.7)
- removed the P2 at (98.6, 65.8)
- removed the P2 at (167.5, 45.7)
- removed the P2 at (167.5, 58.7)
- removed the R1 at (57.5, 97.8)
- removed the R1 at (172.8, 76.5)
- removed the R1 at (202.8, 76.5)
- removed the R1 at (57.5, 67.8)
- removed the R1 at (384.5, 66.8)
- removed the R1 at (76.5, 97.2)
- removed the R1 at (111.0, 54.0)
- removed the R2 at (45.8, 107.5)
- removed the R2 at (182.5, 88.2)
- removed the R2 at (212.5, 88.2)
- removed the R2 at (45.8, 77.5)
- removed the R2 at (372.8, 76.5)
- removed the R2 at (88.2, 87.5)
- removed the R2 at (111.0, 51.6)
- removed the R3 at (45.8, 112.5)
- removed the R3 at (187.5, 88.2)
- removed the R3 at (217.5, 88.2)
- removed the R3 at (45.8, 82.5)
- removed the R3 at (372.8, 81.5)
- removed the R3 at (88.2, 82.5)
- removed the R3 at (125.7, 66.0)
- removed the R4 at (42.0, 110.8)
- removed the R4 at (185.8, 92.0)
- removed the R4 at (215.8, 92.0)
- removed the R4 at (42.0, 80.8)
- removed the R4 at (369.0, 79.8)
- removed the R4 at (92.0, 84.2)
- removed the R4 at (132.2, 66.0)
- removed the R5 at (132.0, 53.0)
- removed the R6 at (134.5, 55.5)
- removed the R7 at (91.8, 59.4)
- removed the R8 at (91.8, 63.2)
- removed the SW1 at (140.5, 54.0)
- removed the U1 at (92.5, 105.0)
- removed the U1 at (180.0, 41.5)
- removed the U1 at (210.0, 41.5)
- removed the U1 at (92.5, 75.0)
- removed the U1 at (419.5, 74.0)
- removed the U1 at (41.5, 90.0)
- removed the U1 at (130.0, 60.0)
- removed the U2 at (51.8, 105.0)
- removed the U2 at (180.0, 82.2)
- removed the U2 at (210.0, 82.2)
- removed the U2 at (51.8, 75.0)
- removed the U2 at (378.8, 74.0)
- removed the U2 at (82.2, 90.0)
- removed the U2 at (63.5, 60.0)
- removed the m3_loch at (60.2, 110.0)
- removed the m3_loch at (139.5, 65.0)
- removed the m3_loch at (44.2, 100.0)
- removed the m3_loch at (175.0, 89.8)
- removed the m3_loch at (185.0, 73.8)
- removed the m3_loch at (60.2, 80.0)
- removed the m3_loch at (205.0, 89.8)
- removed the m3_loch at (215.0, 73.8)
- removed the m3_loch at (44.2, 70.0)
- removed the m3_loch at (371.2, 69.0)
- removed the m3_loch at (387.2, 79.0)
- removed the m3_loch at (73.8, 85.0)
- removed the m3_loch at (89.8, 95.0)
- removed the m3_loch at (98.0, 55.0)
- added C1: 100nF, SM0603_big, F.Cu at (75.8, 72.5)
- added C1: 100nF, SM0603_big, F.Cu at (38.0, 68.9)
- added C1: 100nF, SM0603_big, F.Cu at (599.0, 172.9)
- added C1: 100nF, SM0603_big, F.Cu at (105.2, 61.5)
- added C1: 100nF, SM0603_big, F.Cu at (135.2, 61.5)
- added C1: 100nF, SM0603_big, F.Cu at (135.8, 72.5)
- added C1: 100nF, SM0603_big, F.Cu at (105.8, 72.5)
- added C1: 100nF, SM0603_big, F.Cu at (165.8, 72.5)
- added C1: 100nF, SM0603_big, F.Cu at (195.2, 61.5)
- added C1: 100nF, SM0603_big, F.Cu at (45.8, 72.5)
- added C1: 100nF, SM0603_big, F.Cu at (75.2, 61.5)
- added C1: 100nF, SM0603_big, F.Cu at (218.0, 68.9)
- added C2: 100nF, SM0603_big, F.Cu at (90.2, 81.2)
- added C2: 10uF, SM0805_big, F.Cu at (23.0, 56.0)
- added C2: 10uF, SM0805_big, F.Cu at (584.0, 160.0)
- added C2: 100nF, SM0603_big, F.Cu at (90.8, 52.8)
- added C2: 100nF, SM0603_big, F.Cu at (120.8, 52.8)
- added C2: 100nF, SM0603_big, F.Cu at (150.2, 81.2)
- added C2: 100nF, SM0603_big, F.Cu at (120.2, 81.2)
- added C2: 100nF, SM0603_big, F.Cu at (180.2, 81.2)
- added C2: 100nF, SM0603_big, F.Cu at (180.8, 52.8)
- added C2: 100nF, SM0603_big, F.Cu at (60.2, 81.2)
- added C2: 100nF, SM0603_big, F.Cu at (60.8, 52.8)
- added C2: 10uF, SM0805_big, F.Cu at (203.0, 56.0)
- added C3: 10uF, SM0805_big, F.Cu at (90.2, 84.8)
- added C3: 100nF, SM0603_big, F.Cu at (36.0, 52.8)
- added C3: 100nF, SM0603_big, F.Cu at (597.0, 156.8)
- added C3: 10uF, SM0805_big, F.Cu at (90.8, 49.2)
- added C3: 10uF, SM0805_big, F.Cu at (120.8, 49.2)
- added C3: 10uF, SM0805_big, F.Cu at (150.2, 84.8)
- added C3: 10uF, SM0805_big, F.Cu at (120.2, 84.8)
- added C3: 10uF, SM0805_big, F.Cu at (180.2, 84.8)
- added C3: 10uF, SM0805_big, F.Cu at (180.8, 49.2)
- added C3: 10uF, SM0805_big, F.Cu at (60.2, 84.8)
- added C3: 10uF, SM0805_big, F.Cu at (60.8, 49.2)
- added C3: 100nF, SM0603_big, F.Cu at (216.0, 52.8)
- added C4: 100nF, SM0603_big, F.Cu at (84.8, 92.0)
- added C4: 10uF, SM0805_big, F.Cu at (23.0, 53.0)
- added C4: 10uF, SM0805_big, F.Cu at (584.0, 157.0)
- added C4: 100nF, SM0603_big, F.Cu at (96.2, 42.0)
- added C4: 100nF, SM0603_big, F.Cu at (126.2, 42.0)
- added C4: 100nF, SM0603_big, F.Cu at (144.8, 92.0)
- added C4: 100nF, SM0603_big, F.Cu at (114.8, 92.0)
- added C4: 100nF, SM0603_big, F.Cu at (174.8, 92.0)
- added C4: 100nF, SM0603_big, F.Cu at (186.2, 42.0)
- added C4: 100nF, SM0603_big, F.Cu at (54.8, 92.0)
- added C4: 100nF, SM0603_big, F.Cu at (66.2, 42.0)
- added C4: 10uF, SM0805_big, F.Cu at (203.0, 53.0)
- added C5: 100nF, SM0603_big, F.Cu at (209.5, 47.5)
- added C5: 100nF, SM0603_big, F.Cu at (29.5, 47.5)
- added C5: 100nF, SM0603_big, F.Cu at (590.5, 151.5)
- added C6: 100nF, SM0603_big, F.Cu at (217.5, 85.5)
- added C6: 100nF, SM0603_big, F.Cu at (37.5, 85.5)
- added C6: 100nF, SM0603_big, F.Cu at (598.5, 189.5)
- added D1: LED, SM0603_big, F.Cu at (204.0, 75.6)
- added D1: LED, SM0603_big, F.Cu at (24.0, 75.6)
- added D1: LED, SM0603_big, F.Cu at (585.0, 179.6)
- added D2: LED, SM0603_big, F.Cu at (201.6, 75.6)
- added D2: LED, SM0603_big, F.Cu at (21.6, 75.6)
- added D2: LED, SM0603_big, F.Cu at (582.6, 179.6)
- added IC1: ATMEGA88-A, TQFP32, F.Cu at (212.0, 74.0)
- added IC1: ATMEGA88-A, TQFP32, F.Cu at (32.0, 74.0)
- added IC1: ATMEGA88-A, TQFP32, F.Cu at (593.0, 178.0)
- added J1: RJ45, RJ45_8P8_simple, F.Cu at (83.0, 98.0)
- added J1: RJ45, RJ45_8P8_simple, F.Cu at (30.0, 35.0)
- added J1: RJ45, RJ45_8P8_simple, F.Cu at (591.0, 139.0)
- added J1: RJ45, RJ45_8P8_simple, F.Cu at (98.0, 36.0)
- added J1: RJ45, RJ45_8P8_simple, F.Cu at (128.0, 36.0)
- added J1: RJ45, RJ45_8P8_simple, F.Cu at (143.0, 98.0)
- added J1: RJ45, RJ45_8P8_simple, F.Cu at (113.0, 98.0)
- added J1: RJ45, RJ45_8P8_simple, F.Cu at (173.0, 98.0)
- added J1: RJ45, RJ45_8P8_simple, F.Cu at (188.0, 36.0)
- added J1: RJ45, RJ45_8P8_simple, F.Cu at (53.0, 98.0)
- added J1: RJ45, RJ45_8P8_simple, F.Cu at (68.0, 36.0)
- added J1: RJ45, RJ45_8P8_simple, F.Cu at (210.0, 35.0)
- added P1: ISP, wannenstecker_2x5_rm254, F.Cu at (210.0, 63.0)
- added P1: ISP, wannenstecker_2x5_rm254, F.Cu at (30.0, 63.0)
- added P1: ISP, wannenstecker_2x5_rm254, F.Cu at (591.0, 167.0)
- added P2: UART, Stiftleiste_4x1, F.Cu at (215.8, 83.4)
- added P2: UART, Stiftleiste_4x1, F.Cu at (35.8, 83.4)
- added P2: UART, Stiftleiste_4x1, F.Cu at (596.8, 187.4)
- added R1: 220, SM0603_big, F.Cu at (75.8, 76.5)
- added R1: 150, SM0805_big, F.Cu at (24.0, 71.0)
- added R1: 150, SM0805_big, F.Cu at (585.0, 175.0)
- added R1: 220, SM0603_big, F.Cu at (105.2, 57.5)
- added R1: 220, SM0603_big, F.Cu at (135.2, 57.5)
- added R1: 220, SM0603_big, F.Cu at (135.8, 76.5)
- added R1: 220, SM0603_big, F.Cu at (105.8, 76.5)
- added R1: 220, SM0603_big, F.Cu at (165.8, 76.5)
- added R1: 220, SM0603_big, F.Cu at (195.2, 57.5)
- added R1: 220, SM0603_big, F.Cu at (45.8, 76.5)
- added R1: 220, SM0603_big, F.Cu at (75.2, 57.5)
- added R1: 150, SM0805_big, F.Cu at (204.0, 71.0)
- added R2: 22k, SM0603_big, F.Cu at (85.5, 88.2)
- added R2: 150, SM0805_big, F.Cu at (21.6, 71.0)
- added R2: 150, SM0805_big, F.Cu at (582.6, 175.0)
- added R2: 22k, SM0603_big, F.Cu at (95.5, 45.8)
- added R2: 22k, SM0603_big, F.Cu at (125.5, 45.8)
- added R2: 22k, SM0603_big, F.Cu at (145.5, 88.2)
- added R2: 22k, SM0603_big, F.Cu at (115.5, 88.2)
- added R2: 22k, SM0603_big, F.Cu at (175.5, 88.2)
- added R2: 22k, SM0603_big, F.Cu at (185.5, 45.8)
- added R2: 22k, SM0603_big, F.Cu at (55.5, 88.2)
- added R2: 22k, SM0603_big, F.Cu at (65.5, 45.8)
- added R2: 150, SM0805_big, F.Cu at (201.6, 71.0)
- added R3: 22k, SM0603_big, F.Cu at (90.5, 88.2)
- added R3: 10k, SM0603_big, F.Cu at (36.0, 56.3)
- added R3: 10k, SM0603_big, F.Cu at (597.0, 160.3)
- added R3: 22k, SM0603_big, F.Cu at (90.5, 45.8)
- added R3: 22k, SM0603_big, F.Cu at (120.5, 45.8)
- added R3: 22k, SM0603_big, F.Cu at (150.5, 88.2)
- added R3: 22k, SM0603_big, F.Cu at (120.5, 88.2)
- added R3: 22k, SM0603_big, F.Cu at (180.5, 88.2)
- added R3: 22k, SM0603_big, F.Cu at (180.5, 45.8)
- added R3: 22k, SM0603_big, F.Cu at (60.5, 88.2)
- added R3: 22k, SM0603_big, F.Cu at (60.5, 45.8)
- added R3: 10k, SM0603_big, F.Cu at (216.0, 56.3)
- added R4: 120, SM0603_big, F.Cu at (88.8, 92.0)
- added R4: 22k, SM0603_big, F.Cu at (36.0, 49.8)
- added R4: 22k, SM0603_big, F.Cu at (597.0, 153.8)
- added R4: 120, SM0603_big, F.Cu at (92.2, 42.0)
- added R4: 120, SM0603_big, F.Cu at (122.2, 42.0)
- added R4: 120, SM0603_big, F.Cu at (148.8, 92.0)
- added R4: 120, SM0603_big, F.Cu at (118.8, 92.0)
- added R4: 120, SM0603_big, F.Cu at (178.8, 92.0)
- added R4: 120, SM0603_big, F.Cu at (182.2, 42.0)
- added R4: 120, SM0603_big, F.Cu at (58.8, 92.0)
- added R4: 120, SM0603_big, F.Cu at (62.2, 42.0)
- added R4: 22k, SM0603_big, F.Cu at (216.0, 49.8)
- added R5: 22k, SM0603_big, F.Cu at (203.0, 50.0)
- added R5: 22k, SM0603_big, F.Cu at (23.0, 50.0)
- added R5: 22k, SM0603_big, F.Cu at (584.0, 154.0)
- added R6: 120, SM0603_big, F.Cu at (205.5, 47.5)
- added R6: 120, SM0603_big, F.Cu at (25.5, 47.5)
- added R6: 120, SM0603_big, F.Cu at (586.5, 151.5)
- added R7: 2k2, SM0603_big, F.Cu at (209.4, 90.2)
- added R7: 2k2, SM0603_big, F.Cu at (29.4, 90.2)
- added R7: 2k2, SM0603_big, F.Cu at (590.4, 194.2)
- added R8: 2k2, SM0603_big, F.Cu at (213.2, 90.2)
- added R8: 2k2, SM0603_big, F.Cu at (33.2, 90.2)
- added R8: 2k2, SM0603_big, F.Cu at (594.2, 194.2)
- added SW1: SW_RESET, Taster_6mm, F.Cu at (204.0, 41.5)
- added SW1: SW_RESET, Taster_6mm, F.Cu at (24.0, 41.5)
- added SW1: SW_RESET, Taster_6mm, F.Cu at (585.0, 145.5)
- added U1: TSIC50XF, Tsic_TO92, F.Cu at (83.0, 41.5)
- added U1: ST485, st485, F.Cu at (30.0, 52.0)
- added U1: ST485, st485, F.Cu at (591.0, 156.0)
- added U1: TSIC50XF, Tsic_TO92, F.Cu at (98.0, 92.5)
- added U1: TSIC50XF, Tsic_TO92, F.Cu at (128.0, 92.5)
- added U1: TSIC50XF, Tsic_TO92, F.Cu at (143.0, 41.5)
- added U1: TSIC50XF, Tsic_TO92, F.Cu at (113.0, 41.5)
- added U1: TSIC50XF, Tsic_TO92, F.Cu at (173.0, 41.5)
- added U1: TSIC50XF, Tsic_TO92, F.Cu at (188.0, 92.5)
- added U1: TSIC50XF, Tsic_TO92, F.Cu at (53.0, 41.5)
- added U1: TSIC50XF, Tsic_TO92, F.Cu at (68.0, 92.5)
- added U1: ST485, st485, F.Cu at (210.0, 52.0)
- added U2: ST485, st485, F.Cu at (83.0, 82.2)
- added U2: HYT271, HYT271, F.Cu at (30.0, 118.5)
- added U2: HYT271, HYT271, F.Cu at (591.0, 222.5)
- added U2: ST485, st485, F.Cu at (98.0, 51.8)
- added U2: ST485, st485, F.Cu at (128.0, 51.8)
- added U2: ST485, st485, F.Cu at (143.0, 82.2)
- added U2: ST485, st485, F.Cu at (113.0, 82.2)
- added U2: ST485, st485, F.Cu at (173.0, 82.2)
- added U2: ST485, st485, F.Cu at (188.0, 51.8)
- added U2: ST485, st485, F.Cu at (53.0, 82.2)
- added U2: ST485, st485, F.Cu at (68.0, 51.8)
- added U2: HYT271, HYT271, F.Cu at (210.0, 118.5)
- added m3_loch: VAL**, m3_loch, F.Cu at (88.0, 73.8)
- added m3_loch: VAL**, m3_loch, F.Cu at (168.0, 89.8)
- added m3_loch: VAL**, m3_loch, F.Cu at (183.0, 60.2)
- added m3_loch: VAL**, m3_loch, F.Cu at (193.0, 44.2)
- added m3_loch: VAL**, m3_loch, F.Cu at (58.0, 73.8)
- added m3_loch: VAL**, m3_loch, F.Cu at (48.0, 89.8)
- added m3_loch: VAL**, m3_loch, F.Cu at (63.0, 60.2)
- added m3_loch: VAL**, m3_loch, F.Cu at (73.0, 44.2)
- added m3_loch: VAL**, m3_loch, F.Cu at (215.0, 42.5)
- added m3_loch: VAL**, m3_loch, F.Cu at (205.0, 84.0)
- added m3_loch: VAL**, m3_loch, F.Cu at (35.0, 42.5)
- added m3_loch: VAL**, m3_loch, F.Cu at (78.0, 89.8)
- added m3_loch: VAL**, m3_loch, F.Cu at (25.0, 84.0)
- added m3_loch: VAL**, m3_loch, F.Cu at (586.0, 188.0)
- added m3_loch: VAL**, m3_loch, F.Cu at (596.0, 146.5)
- added m3_loch: VAL**, m3_loch, F.Cu at (93.0, 60.2)
- added m3_loch: VAL**, m3_loch, F.Cu at (103.0, 44.2)
- added m3_loch: VAL**, m3_loch, F.Cu at (133.0, 44.2)
- added m3_loch: VAL**, m3_loch, F.Cu at (123.0, 60.2)
- added m3_loch: VAL**, m3_loch, F.Cu at (108.0, 89.8)
- added m3_loch: VAL**, m3_loch, F.Cu at (138.0, 89.8)
- added m3_loch: VAL**, m3_loch, F.Cu at (148.0, 73.8)
- added m3_loch: VAL**, m3_loch, F.Cu at (118.0, 73.8)
- added m3_loch: VAL**, m3_loch, F.Cu at (178.0, 73.8)
- moved R3 466.2 mm to (591.7, 50.0)
- moved R7 466.2 mm to (556.2, 59.6)
- moved R8 466.2 mm to (556.2, 55.8)
- moved C1 466.2 mm to (579.1, 52.0)
- moved C1 466.2 mm to (534.9, 51.0)
- moved C1 466.2 mm to (668.2, 75.5)
- moved C2 466.2 mm to (592.0, 37.0)
- moved C2 466.2 mm to (522.0, 66.0)
- moved C2 466.2 mm to (653.8, 66.8)
- moved C3 466.2 mm to (595.2, 50.0)
- moved C3 466.2 mm to (518.8, 53.0)
- moved C3 466.2 mm to (653.8, 63.2)
- moved C4 466.2 mm to (595.0, 37.0)
- moved C4 466.2 mm to (519.0, 66.0)
- moved C4 466.2 mm to (659.2, 56.0)
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Routing:
- net GND: track 6304.5 -> 7053.8 mm, vias 75 -> 91
- net VCC: track 3792.6 -> 4363.9 mm, vias 94 -> 111
- net N-000007: track 1058.4 -> 1195.0 mm
- net /za: track 671.3 -> 802.0 mm, vias 4 -> 6
- net /zb: track 684.1 -> 814.3 mm
- net N-0000010: track 908.5 -> 1027.0 mm
- net /RESET: track 543.9 -> 655.4 mm, vias 14 -> 18
- net /SDA: track 413.6 -> 498.6 mm
- net /SCL: track 436.3 -> 520.7 mm
- net /DI: track 74.1 -> 111.1 mm
- net /MOSI: track 196.0 -> 219.5 mm, vias 10 -> 12
- net /SCK: track 78.3 -> 99.6 mm
- net /RX: track 179.3 -> 199.5 mm
- net /MISO: track 65.1 -> 84.6 mm
- net /LED2: track 81.8 -> 96.1 mm
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Other:
- board size 527 x 353 mm -> 720.1 x 375 mm

Commit message: finished
Parts:
- removed the C1 at (599.0, 172.9)
- removed the C1 at (449.8, 221.0)
- removed the C1 at (364.5, 370.2)
- removed the C1 at (579.1, 52.0)
- removed the C1 at (534.9, 51.0)
- removed the C1 at (668.2, 75.5)
- removed the C1 at (498.1, 363.0)
- removed the C2 at (584.0, 160.0)
- removed the C2 at (435.2, 212.2)
- removed the C2 at (373.2, 355.8)
- removed the C2 at (592.0, 37.0)
- removed the C2 at (522.0, 66.0)
- removed the C2 at (653.8, 66.8)
- removed the C2 at (511.0, 348.0)
- removed the C3 at (597.0, 156.8)
- removed the C3 at (435.2, 208.8)
- removed the C3 at (376.8, 355.8)
- removed the C3 at (595.2, 50.0)
- removed the C3 at (518.8, 53.0)
- removed the C3 at (653.8, 63.2)
- removed the C3 at (514.2, 361.0)
- removed the C4 at (584.0, 157.0)
- removed the C4 at (440.8, 201.5)
- removed the C4 at (384.0, 361.2)
- removed the C4 at (595.0, 37.0)
- removed the C4 at (519.0, 66.0)
- removed the C4 at (659.2, 56.0)
- removed the C4 at (514.0, 348.0)
- removed the C5 at (590.5, 151.5)
- removed the C5 at (600.5, 43.5)
- removed the C5 at (513.5, 59.5)
- removed the C5 at (519.5, 354.5)
- removed the C6 at (598.5, 189.5)
- removed the C6 at (562.5, 51.5)
- removed the C6 at (551.5, 51.5)
- removed the C6 at (481.5, 362.5)
- removed the D1 at (585.0, 179.6)
- removed the D1 at (572.4, 38.0)
- removed the D1 at (541.6, 65.0)
- removed the D1 at (491.4, 349.0)
- removed the D2 at (582.6, 179.6)
- removed the D2 at (572.4, 35.6)
- removed the D2 at (541.6, 67.4)
- removed the D2 at (491.4, 346.6)
- removed the IC1 at (593.0, 178.0)
- removed the IC1 at (574.0, 46.0)
- removed the IC1 at (540.0, 57.0)
- removed the IC1 at (493.0, 357.0)
- removed the J1 at (591.0, 139.0)
- removed the J1 at (442.5, 195.5)
- removed the J1 at (390.0, 363.0)
- removed the J1 at (613.0, 44.0)
- removed the J1 at (501.0, 59.0)
- removed the J1 at (661.0, 50.0)
- removed the J1 at (532.0, 355.0)
- removed the P1 at (504.0, 355.0)
- removed the P1 at (591.0, 167.0)
- removed the P1 at (585.0, 44.0)
- removed the P1 at (529.0, 59.0)
- removed the P1 at (680.6, 42.7)
- removed the P1 at (430.6, 389.7)
- removed the P1 at (-31.4, 126.7)
- removed the P2 at (483.6, 360.8)
- removed the P2 at (596.8, 187.4)
- removed the P2 at (564.6, 49.8)
- removed the P2 at (549.4, 53.2)
- removed the P2 at (675.5, 42.7)
- removed the P2 at (425.5, 389.7)
- removed the P2 at (-36.5, 126.7)
- removed the R1 at (585.0, 175.0)
- removed the R1 at (449.8, 217.0)
- removed the R1 at (368.5, 370.2)
- removed the R1 at (577.0, 38.0)
- removed the R1 at (537.0, 65.0)
- removed the R1 at (668.2, 71.5)
- removed the R1 at (496.0, 349.0)
- removed the R2 at (582.6, 175.0)
- removed the R2 at (440.0, 205.2)
- removed the R2 at (380.2, 360.5)
- removed the R2 at (577.0, 35.6)
- removed the R2 at (537.0, 67.4)
- removed the R2 at (658.5, 59.8)
- removed the R2 at (496.0, 346.6)
- removed the R3 at (597.0, 160.3)
- removed the R3 at (435.0, 205.2)
- removed the R3 at (380.2, 355.5)
- removed the R3 at (591.7, 50.0)
- removed the R3 at (522.3, 53.0)
- removed the R3 at (653.5, 59.8)
- removed the R3 at (510.7, 361.0)
- removed the R4 at (597.0, 153.8)
- removed the R4 at (436.8, 201.5)
- removed the R4 at (384.0, 357.2)
- removed the R4 at (598.2, 50.0)
- removed the R4 at (515.8, 53.0)
- removed the R4 at (655.2, 56.0)
- removed the R4 at (517.2, 361.0)
- removed the R5 at (584.0, 154.0)
- removed the R5 at (598.0, 37.0)
- removed the R5 at (516.0, 66.0)
- removed the R5 at (517.0, 348.0)
- removed the R6 at (586.5, 151.5)
- removed the R6 at (600.5, 39.5)
- removed the R6 at (513.5, 63.5)
- removed the R6 at (519.5, 350.5)
- removed the R7 at (590.4, 194.2)
- removed the R7 at (557.8, 43.4)
- removed the R7 at (556.2, 59.6)
- removed the R7 at (476.8, 354.4)
- removed the R8 at (594.2, 194.2)
- removed the R8 at (557.8, 47.2)
- removed the R8 at (556.2, 55.8)
- removed the R8 at (476.8, 358.2)
- removed the SW1 at (585.0, 145.5)
- removed the SW1 at (606.5, 38.0)
- removed the SW1 at (507.5, 65.0)
- removed the SW1 at (525.5, 349.0)
- removed the U1 at (591.0, 156.0)
- removed the U1 at (442.5, 252.0)
- removed the U1 at (333.5, 363.0)
- removed the U1 at (596.0, 44.0)
- removed the U1 at (518.0, 59.0)
- removed the U1 at (661.0, 106.5)
- removed the U1 at (515.0, 355.0)
- removed the U2 at (591.0, 222.5)
- removed the U2 at (442.5, 211.2)
- removed the U2 at (374.2, 363.0)
- removed the U2 at (529.5, 44.0)
- removed the U2 at (584.5, 59.0)
- removed the U2 at (661.0, 65.8)
- removed the U2 at (448.5, 355.0)
- removed the m3_loch at (586.0, 188.0)
- removed the m3_loch at (596.0, 146.5)
- removed the m3_loch at (447.5, 203.8)
- removed the m3_loch at (437.5, 219.8)
- removed the m3_loch at (365.8, 358.0)
- removed the m3_loch at (381.8, 368.0)
- removed the m3_loch at (564.0, 39.0)
- removed the m3_loch at (605.5, 49.0)
- removed the m3_loch at (550.0, 64.0)
- removed the m3_loch at (508.5, 54.0)
- removed the m3_loch at (656.0, 74.2)
- removed the m3_loch at (666.0, 58.2)
- removed the m3_loch at (524.5, 360.0)
- removed the m3_loch at (483.0, 350.0)
- added P1: CONN_4, HYT271, F.Cu at (199.6, 96.7)
- added P1: CONN_4, HYT271, F.Cu at (198.4, 109.3)
- added P1: CONN_4, HYT271, F.Cu at (26.6, 127.7)
- added P1: CONN_4, HYT271, F.Cu at (213.4, 127.3)
- added P1: CONN_4, HYT271, F.Cu at (187.4, 109.3)
- added P2: CONN_4, Stiftleiste_4x1, F.Cu at (194.5, 96.7)
- added P2: CONN_4, Stiftleiste_4x1, F.Cu at (203.5, 109.3)
- added P2: CONN_4, Stiftleiste_4x1, F.Cu at (21.5, 127.7)
- added P2: CONN_4, Stiftleiste_4x1, F.Cu at (218.5, 127.3)
- added P2: CONN_4, Stiftleiste_4x1, F.Cu at (192.5, 109.3)
Routing:
- net GND: track 7053.8 -> 5935.8 mm, vias 91 -> 65
- net VCC: track 4363.9 -> 3394.3 mm, vias 111 -> 86
- net /RESET: track 655.4 -> 432.3 mm, vias 18 -> 10
- net /za: track 802.0 -> 613.0 mm, vias 6 -> 2
- net /zb: track 814.3 -> 628.7 mm
- net /SDA: track 498.6 -> 328.5 mm
- net /SCL: track 520.7 -> 351.9 mm
- net N-000007: track 1195.0 -> 1058.4 mm
- net N-0000010: track 1027.0 -> 908.5 mm
- net /DI: track 111.1 -> 37.0 mm
- net /MOSI: track 219.5 -> 172.4 mm, vias 12 -> 8
- net /SCK: track 99.6 -> 57.0 mm
- net /RX: track 199.5 -> 159.2 mm
- net /MISO: track 84.6 -> 45.7 mm
- net /LED2: track 96.1 -> 67.6 mm
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Other:
- board size 720.1 x 375 mm -> 200 x 330 mm
