File: hardware/order2/newOrder.kicad_pcb (KiCad board)
At the start: 2 copper layers, 200 x 330 mm, 656 parts, among them IC1 ATMEGA88-A, IC1 ATMEGA88A-A, J1 RJ45, J1 RJ45_8P8C_8FACH, K1 pow_sel, P1 CONN_4, P1 ISP, P1 UART, P2 CONN_4, P2 Shield, P2 UART, P3 i2c_pow, P4 i2c_chain, P5 12Vin, P6 HOHLBUCHSE, P7 Vccin, P8 ISP, P9 5Vin, SW1 SW1, SW1 SW_RESET, SW2 SCHALTER_2POL, SW3 SW_RESET, U1 LM7805, U1 ST485, U1 TSIC50XF, U2 HYT271, U2 ST485, U3 ST485, U4 ST485, U5 ST485, U6 ST485, U7 ST485, U8 ST485, U9 ST485, X1 20MHz, m3_loch VAL**

Commit message: finished and can be plot
Other:
- rule pad_to_mask_clearance: 0 -> 0.15
Changed lines of the file:
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@@
     (links 1934)
     (no_connects 327)
-    (area 12.3316 3.150001 554.6684 366.671)
+    (area 18.329 3.150001 285.714285 351.671)
     (thickness 1.6)
-    (drawings 296)
+    (drawings 295)
     (tracks 6549)
     (zones 0)
@@
     (pad_size 3.4 3.4)
     (pad_drill 3.2)
-    (pad_to_mask_clearance 0)
-    (solder_mask_min_width 0.1)
+    (pad_to_mask_clearance 0.15)
     (aux_axis_origin 0 0)
     (visible_elements 7FFFFBFF)
     (pcbplotparams
-      (layerselection 32769)
+      (layerselection 281051137)
       (usegerberextensions false)
-      (excludeedgelayer false)
+      (excludeedgelayer true)
       (linewidth 0.150000)
       (plotframeref false)
@@
       (padsonsilk false)
       (subtractmaskfromsilk false)
-      (outputformat 2)
+      (outputformat 1)
       (mirror false)
-      (drillshape 2)
+      (drillshape 0)
       (scaleselection 1)
       (outputdirectory ""))
@@
   (gr_line (start 200 86.5) (end 207 93.5) (angle 90) (layer Edge.Cuts) (width 0.1))
   (gr_line (start 200 20) (end 200 86.5) (angle 90) (layer Edge.Cuts) (width 0.1))
-  (dimension 10 (width 0.3) (layer Cmts.User)
-    (gr_text "10.000 mm" (at 1.650001 127.999998 270) (layer Cmts.User)
-      (effects (font (size 1.5 1.5) (thickness 0.3)))
-    )
-    (feature1 (pts (xy 29 133) (xy 0.300001 132.999998)))
-    (feature2 (pts (xy 29 123) (xy 0.300001 122.999998)))
-    (crossbar (pts (xy 3.000001 122.999998) (xy 3.000001 132.999998)))
-    (arrow1a (pts (xy 3.000001 132.999998) (xy 2.413581 131.873495)))
-    (arrow1b (pts (xy 3.000001 132.999998) (xy 3.586421 131.873495)))
-    (arrow2a (pts (xy 3.000001 122.999998) (xy 2.413581 124.126501)))
-    (arrow2b (pts (xy 3.000001 122.999998) (xy 3.586421 124.126501)))
-  )
   (gr_text v1.1 (at 21.4 30.5 90) (layer F.Cu)
     (effects (font (size 1.5 1.5) (thickness 0.3)))

Commit message: save
Parts:
- removed the P1 at (198.4, 109.3)
- removed the P1 at (187.4, 109.3)
- removed the P2 at (203.5, 109.3)
- removed the P2 at (192.5, 109.3)
- added P1: CONN_4, Stiftleiste_4x1, F.Cu at (201.2, 109.3)
- added P1: CONN_4, Stiftleiste_4x1, F.Cu at (48.7, 34.2)
- added P2: so8, st485, F.Cu at (196.8, 109.3)
- added P2: so8, st485, F.Cu at (48.7, 29.8)
- added P3: CONN_4, Stiftleiste_4x1, F.Cu at (188.5, 109.3)
- added P3: CONN_4, Stiftleiste_4x1, F.Cu at (48.7, 21.5)
Routing:
- net N-000008: track 11.3 -> 20.5 mm
- net N-000006: track 0.00 -> 8.63 mm
- net N-000005: track 0.00 -> 7.04 mm
- net N-000007: track 1058.4 -> 1065.2 mm
- net N-000001: track 30.0 -> 25.0 mm
- net N-000003: track 75.9 -> 71.8 mm
- net N-000004: track 30.0 -> 27.1 mm
- net N-000002: track 32.4 -> 30.3 mm
Other:
- outline, holes or cut-outs redrawn
- net class Default: trace_width 0.7 -> 0.6; via_dia 1.2 -> 0.889; via_drill 0.6 -> 0.635
- net class uc removed
- rule pad_to_mask_clearance: 0.15 -> 0
- board text added: "SO8"

Commit message: collector board: twi state machine
Other:
- rule pad_to_mask_clearance: 0 -> 0.15
Changed lines of the file:
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@@
     (links 1948)
     (no_connects 333)
-    (area 18.329 3.150001 529.989 378.636214)
+    (area 18.329 3.150001 285.714285 351.671)
     (thickness 1.6)
     (drawings 289)
@@
     (pad_size 1.5 1.5)
     (pad_drill 0.6)
-    (pad_to_mask_clearance 0)
+    (pad_to_mask_clearance 0.15)
     (aux_axis_origin 0 0)
     (visible_elements 7FFFFBFF)
@@
       (outputformat 1)
       (mirror false)
-      (drillshape 1)
+      (drillshape 0)
       (scaleselection 1)
       (outputdirectory ""))
