File: hardware/order2/order2.kicad_pcb (KiCad board)
At the start: 2 copper layers, 310 x 251.6 mm, 222 parts, among them IC1 ATMEGA88-A, IC1 ATMEGA88A-A, J1 RJ45, J1 RJ45_8P8C_8FACH, K1 CONN_3, K1 pow_sel, K2 CONN_3, P1 CONN_4, P1 CONN_8, P1 ISP, P1 UART, P10 CONN_10, P11 CONN_8, P2 CONN_4, P2 CONN_6, P2 Shield, P2 UART, P2 so8, P3 CONN_4, P3 CONN_6, P3 i2c_pow, P4 CONN_8, P4 i2c_chain, P5 12Vin, P5 POW, P6 HOHLBUCHSE, P6 TWI, P7 TWI_POW, P7 Vccin, P8 CONN_10, P8 ISP, P9 5Vin, P9 CONN_8, SW1 SW1, SW1 SW_RESET, SW2 SCHALTER_2POL, SW3 SW_RESET, U1 LM7805, U1 ST485, U1 TSIC50XF, U2 HYT271, U2 ST485, U3 ST485, U4 ST485, U5 ST485, U6 ST485, U7 ST485, U8 ST485, U9 ST485, X1 20MHz, m3_loch VAL**

Commit message: save
Parts:
- removed the C1 at (181.2, 63.5)
- removed the C1 at (151.8, 74.5)
- removed the C1 at (178.5, 119.6)
- removed the C1 at (210.0, 74.9)
- removed the C1 at (327.2, 71.5)
- removed the C2 at (166.8, 54.8)
- removed the C2 at (166.2, 83.2)
- removed the C2 at (193.5, 132.5)
- removed the C2 at (195.0, 62.0)
- removed the C2 at (312.8, 62.8)
- removed the C3 at (166.8, 51.2)
- removed the C3 at (166.2, 86.8)
- removed the C3 at (180.5, 135.8)
- removed the C3 at (208.0, 58.8)
- removed the C3 at (312.8, 59.2)
- removed the C4 at (172.2, 44.0)
- removed the C4 at (160.8, 94.0)
- removed the C4 at (193.5, 135.5)
- removed the C4 at (195.0, 59.0)
- removed the C4 at (318.2, 52.0)
- removed the C5 at (187.0, 141.0)
- removed the C5 at (201.5, 53.5)
- removed the C6 at (179.0, 103.0)
- removed the C6 at (209.5, 91.5)
- removed the D1 at (192.5, 112.9)
- removed the D1 at (196.0, 81.6)
- removed the D1 at (195.0, 178.5)
- removed the D2 at (194.9, 112.9)
- removed the D2 at (193.6, 81.6)
- removed the IC1 at (184.5, 114.5)
- removed the IC1 at (204.0, 80.0)
- removed the J1 at (174.0, 38.0)
- removed the J1 at (159.0, 100.0)
- removed the J1 at (186.5, 153.5)
- removed the J1 at (202.0, 41.0)
- removed the J1 at (320.0, 46.0)
- removed the K1 at (40.7, 269.5)
- removed K2: CONN_3, Tsic_TO92
- removed the P1 at (186.5, 125.5)
- removed the P1 at (48.7, 235.3)
- removed the P1 at (202.0, 69.0)
- removed the P1 at (162.7, 140.2)
- removed the P1 at (33.7, 236.3)
- removed the P1 at (61.2, 266.3)
- removed P10: CONN_10, Stiftleiste_10x1
- removed P11: CONN_8, Stiftleiste_8x1
- removed the P2 at (180.7, 105.1)
- removed the P2 at (48.7, 230.9)
- removed the P2 at (207.8, 89.4)
- removed the P2 at (162.7, 160.5)
- removed the P2 at (33.7, 231.9)
- removed the P2 at (66.3, 266.3)
- removed the P3 at (48.7, 222.6)
- removed the P3 at (165.7, 160.5)
- removed the P3 at (33.7, 223.6)
- removed the P4 at (165.7, 140.2)
- removed the P5 at (190.0, 179.5)
- removed the P6 at (204.5, 178.0)
- removed the P7 at (175.0, 178.0)
- removed the P8 at (214.0, 133.5)
- removed the P9 at (214.0, 158.0)
- removed the R1 at (181.2, 59.5)
- removed the R1 at (151.8, 78.5)
- removed the R1 at (192.5, 117.5)
- removed the R1 at (196.0, 77.0)
- removed the R1 at (327.2, 67.5)
- removed the R1 at (194.0, 175.0)
- removed the R2 at (171.5, 47.8)
- removed the R2 at (161.5, 90.2)
- removed the R2 at (194.9, 117.5)
- removed the R2 at (193.6, 77.0)
- removed the R2 at (317.5, 55.8)
- removed the R2 at (184.5, 175.5)
- removed the R3 at (166.5, 47.8)
- removed the R3 at (166.5, 90.2)
- removed the R3 at (180.5, 132.2)
- removed the R3 at (208.0, 62.3)
- removed the R3 at (312.5, 55.8)
- removed the R3 at (187.0, 175.5)
- removed the R4 at (168.2, 44.0)
- removed the R4 at (164.8, 94.0)
- removed the R4 at (180.5, 138.8)
- removed the R4 at (208.0, 55.8)
- removed the R4 at (314.2, 52.0)
- removed the R5 at (193.5, 138.5)
- removed the R5 at (195.0, 56.0)
- removed the R6 at (191.0, 141.0)
- removed the R6 at (197.5, 53.5)
- removed the SW1 at (192.5, 147.0)
- removed the SW1 at (196.0, 47.5)
- removed the U1 at (174.0, 94.5)
- removed the U1 at (159.0, 43.5)
- removed the U1 at (186.5, 136.5)
- removed the U1 at (202.0, 58.0)
- removed the U1 at (320.0, 102.5)
- removed the U2 at (174.0, 53.8)
- removed the U2 at (159.0, 84.2)
- removed the U2 at (186.5, 70.0)
- removed the U2 at (202.0, 124.5)
- removed the U2 at (320.0, 61.8)
- removed the m3_loch at (169.0, 62.2)
- removed the m3_loch at (207.0, 48.5)
- removed the m3_loch at (197.0, 90.0)
- removed the m3_loch at (325.0, 54.2)
- removed the m3_loch at (315.0, 70.2)
- removed the m3_loch at (179.0, 46.2)
- removed the m3_loch at (154.0, 91.8)
- removed the m3_loch at (164.0, 75.8)
- removed the m3_loch at (191.5, 104.5)
- removed the m3_loch at (181.5, 146.0)
- added C1: 100nF, SM0603_big, F.Cu at (75.8, 72.5)
- added C1: 100nF, SM0603_big, F.Cu at (38.0, 68.9)
- added C1: 100nF, SM0603_big, F.Cu at (165.2, 61.5)
- added C1: 100nF, SM0603_big, F.Cu at (202.8, 169.5)
- added C1: 100nF, SM0603_big, F.Cu at (112.2, 158.5)
- added C1: 100nF, SM0603_big, F.Cu at (82.8, 169.5)
- added C1: 100nF, SM0603_big, F.Cu at (112.8, 169.5)
- added C1: 100nF, SM0603_big, F.Cu at (142.2, 158.5)
- added C1: 100nF, SM0603_big, F.Cu at (172.2, 158.5)
- added C1: 100nF, SM0603_big, F.Cu at (142.8, 169.5)
- added C1: 100nF, SM0603_big, F.Cu at (172.8, 169.5)
- added C1: 100nF, SM0603_big, F.Cu at (105.2, 61.5)
- added C1: 100nF, SM0603_big, F.Cu at (202.2, 158.5)
- added C1: 100nF, SM0603_big, F.Cu at (82.2, 158.5)
- added C1: 100nF, SM0603_big, F.Cu at (52.8, 169.5)
- added C1: 10u, SM0805_big, F.Cu at (29.2, 257.0)
- added C1: 10u, SM0805_big, F.Cu at (96.2, 257.0)
- added C1: 100nF, SM0603_big, F.Cu at (52.2, 158.5)
- added C1: 100nF, SM0603_big, F.Cu at (135.8, 72.5)
- added C1: 100nF, SM0603_big, F.Cu at (135.2, 61.5)
- added C1: 100nF, SM0603_big, F.Cu at (105.8, 72.5)
- added C1: 100nF, SM0603_big, F.Cu at (165.8, 72.5)
- added C1: 100nF, SM0603_big, F.Cu at (195.2, 61.5)
- added C1: 100nF, SM0603_big, F.Cu at (45.8, 72.5)
- added C1: 100nF, SM0603_big, F.Cu at (75.2, 61.5)
- added C1: 100nF, SM0603_big, F.Cu at (218.0, 68.9)
- added C10: 100n, SM0603_big, F.Cu at (61.2, 294.8)
- added C10: 100n, SM0603_big, F.Cu at (128.2, 294.8)
- added C11: 100n, SM0603_big, F.Cu at (61.2, 280.8)
- added C11: 100n, SM0603_big, F.Cu at (128.2, 280.8)
- added C12: 100n, SM0603_big, F.Cu at (61.2, 266.8)
- added C12: 100n, SM0603_big, F.Cu at (128.2, 266.8)
- added C13: 100n, SM0603_big, F.Cu at (61.2, 252.8)
- added C13: 100n, SM0603_big, F.Cu at (128.2, 252.8)
- added C14: 100n, SM0603_big, F.Cu at (61.2, 238.8)
- added C14: 100n, SM0603_big, F.Cu at (128.2, 238.8)
- added C15: 100n, SM0603_big, F.Cu at (64.6, 230.2)
- added C15: 100n, SM0603_big, F.Cu at (131.6, 230.2)
- added C16: 100n, SM0603_big, F.Cu at (64.6, 244.2)
- added C16: 100n, SM0603_big, F.Cu at (131.6, 244.2)
- added C17: 100n, SM0603_big, F.Cu at (64.6, 258.2)
- added C17: 100n, SM0603_big, F.Cu at (131.6, 258.2)
- added C18: 100n, SM0603_big, F.Cu at (64.6, 272.2)
- added C18: 100n, SM0603_big, F.Cu at (131.6, 272.2)
- added C19: 100n, SM0603_big, F.Cu at (64.6, 286.2)
- added C19: 100n, SM0603_big, F.Cu at (131.6, 286.2)
- added C2: 100nF, SM0603_big, F.Cu at (90.2, 81.2)
- added C2: 10uF, SM0805_big, F.Cu at (23.0, 56.0)
- added C2: 100nF, SM0603_big, F.Cu at (150.8, 52.8)
- added C2: 100nF, SM0603_big, F.Cu at (217.2, 178.2)
- added C2: 100nF, SM0603_big, F.Cu at (97.8, 149.8)
- added C2: 100nF, SM0603_big, F.Cu at (97.2, 178.2)
- added C2: 100nF, SM0603_big, F.Cu at (127.2, 178.2)
- added C2: 100nF, SM0603_big, F.Cu at (127.8, 149.8)
- added C2: 100nF, SM0603_big, F.Cu at (157.8, 149.8)
- added C2: 100nF, SM0603_big, F.Cu at (157.2, 178.2)
- added C2: 100nF, SM0603_big, F.Cu at (187.2, 178.2)
- added C2: 100nF, SM0603_big, F.Cu at (90.8, 52.8)
- added C2: 100nF, SM0603_big, F.Cu at (187.8, 149.8)
- added C2: 100nF, SM0603_big, F.Cu at (67.8, 149.8)
- added C2: 100nF, SM0603_big, F.Cu at (67.2, 178.2)
- added C2: 100n, SM0603_big, F.Cu at (37.2, 293.4)
- added C2: 100n, SM0603_big, F.Cu at (104.2, 293.4)
- added C2: 100nF, SM0603_big, F.Cu at (37.8, 149.8)
- added C2: 100nF, SM0603_big, F.Cu at (150.2, 81.2)
- added C2: 100nF, SM0603_big, F.Cu at (120.8, 52.8)
- added C2: 100nF, SM0603_big, F.Cu at (120.2, 81.2)
- added C2: 100nF, SM0603_big, F.Cu at (180.2, 81.2)
- added C2: 100nF, SM0603_big, F.Cu at (180.8, 52.8)
- added C2: 100nF, SM0603_big, F.Cu at (60.2, 81.2)
- added C2: 100nF, SM0603_big, F.Cu at (60.8, 52.8)
- added C2: 10uF, SM0805_big, F.Cu at (203.0, 56.0)
- added C20: 100n, SM0603_big, F.Cu at (64.6, 300.2)
- added C20: 100n, SM0603_big, F.Cu at (131.6, 300.2)
- added C21: 100n, SM0603_big, F.Cu at (64.8, 314.2)
- added C21: 100n, SM0603_big, F.Cu at (131.8, 314.2)
- added C22: 100n, SM0603_big, F.Cu at (64.8, 328.2)
- added C22: 100n, SM0603_big, F.Cu at (131.8, 328.2)
- added C23: 10u, SM0805_big, F.Cu at (34.4, 257.0)
- added C23: 10u, SM0805_big, F.Cu at (101.4, 257.0)
- added C24: 10u, SM0805_big, F.Cu at (31.8, 257.0)
- added C24: 10u, SM0805_big, F.Cu at (98.8, 257.0)
- added C25: 100n, SM0603_big, F.Cu at (50.6, 232.4)
- added C25: 100n, SM0603_big, F.Cu at (117.6, 232.4)
- added C26: 100n, SM0603_big, F.Cu at (50.8, 244.2)
- added C26: 100n, SM0603_big, F.Cu at (117.8, 244.2)
- added C27: 100n, SM0603_big, F.Cu at (50.9, 258.1)
- added C27: 100n, SM0603_big, F.Cu at (117.9, 258.1)
- added C28: 100n, SM0603_big, F.Cu at (50.9, 272.1)
- added C28: 100n, SM0603_big, F.Cu at (117.9, 272.1)
- added C29: 100n, SM0603_big, F.Cu at (50.7, 288.7)
- added C29: 100n, SM0603_big, F.Cu at (117.7, 288.7)
- added C3: 10uF, SM0805_big, F.Cu at (90.2, 84.8)
- added C3: 100nF, SM0603_big, F.Cu at (36.0, 52.8)
- added C3: 10uF, SM0805_big, F.Cu at (150.8, 49.2)
- added C3: 10uF, SM0805_big, F.Cu at (217.2, 181.8)
- added C3: 10uF, SM0805_big, F.Cu at (97.8, 146.2)
- added C3: 10uF, SM0805_big, F.Cu at (97.2, 181.8)
- added C3: 10uF, SM0805_big, F.Cu at (127.2, 181.8)
- added C3: 10uF, SM0805_big, F.Cu at (127.8, 146.2)
- added C3: 10uF, SM0805_big, F.Cu at (157.8, 146.2)
- added C3: 10uF, SM0805_big, F.Cu at (157.2, 181.8)
- added C3: 10uF, SM0805_big, F.Cu at (187.2, 181.8)
- added C3: 10uF, SM0805_big, F.Cu at (90.8, 49.2)
- added C3: 10uF, SM0805_big, F.Cu at (187.8, 146.2)
- added C3: 10uF, SM0805_big, F.Cu at (67.8, 146.2)
- added C3: 10uF, SM0805_big, F.Cu at (67.2, 181.8)
- added C3: 22p, SM0603_big, F.Cu at (38.2, 271.1)
- added C3: 22p, SM0603_big, F.Cu at (105.2, 271.1)
- added C3: 10uF, SM0805_big, F.Cu at (37.8, 146.2)
- added C3: 10uF, SM0805_big, F.Cu at (150.2, 84.8)
- added C3: 10uF, SM0805_big, F.Cu at (120.8, 49.2)
- added C3: 10uF, SM0805_big, F.Cu at (120.2, 84.8)
- added C3: 10uF, SM0805_big, F.Cu at (180.2, 84.8)
- added C3: 10uF, SM0805_big, F.Cu at (180.8, 49.2)
- added C3: 10uF, SM0805_big, F.Cu at (60.2, 84.8)
- added C3: 10uF, SM0805_big, F.Cu at (60.8, 49.2)
- added C3: 100nF, SM0603_big, F.Cu at (216.0, 52.8)
- added C30: 100n, SM0603_big, F.Cu at (50.9, 300.2)
- added C30: 100n, SM0603_big, F.Cu at (117.9, 300.2)
- added C31: 100n, SM0603_big, F.Cu at (50.9, 314.3)
- added C31: 100n, SM0603_big, F.Cu at (117.9, 314.3)
- added C32: 100n, SM0603_big, F.Cu at (50.7, 328.2)
- added C32: 100n, SM0603_big, F.Cu at (117.7, 328.2)
- added C4: 100nF, SM0603_big, F.Cu at (84.8, 92.0)
- added C4: 10uF, SM0805_big, F.Cu at (23.0, 53.0)
- added C4: 100nF, SM0603_big, F.Cu at (156.2, 42.0)
- added C4: 100nF, SM0603_big, F.Cu at (211.8, 189.0)
- added C4: 100nF, SM0603_big, F.Cu at (103.2, 139.0)
- added C4: 100nF, SM0603_big, F.Cu at (91.8, 189.0)
- added C4: 100nF, SM0603_big, F.Cu at (121.8, 189.0)
- added C4: 100nF, SM0603_big, F.Cu at (133.2, 139.0)
- added C4: 100nF, SM0603_big, F.Cu at (163.2, 139.0)
- added C4: 100nF, SM0603_big, F.Cu at (151.8, 189.0)
- added C4: 100nF, SM0603_big, F.Cu at (181.8, 189.0)
- added C4: 100nF, SM0603_big, F.Cu at (96.2, 42.0)
- added C4: 100nF, SM0603_big, F.Cu at (193.2, 139.0)
- added C4: 100nF, SM0603_big, F.Cu at (73.2, 139.0)
- added C4: 100nF, SM0603_big, F.Cu at (61.8, 189.0)
- added C4: 22p, SM0603_big, F.Cu at (33.0, 271.1)
- added C4: 22p, SM0603_big, F.Cu at (100.0, 271.1)
- added C4: 100nF, SM0603_big, F.Cu at (43.2, 139.0)
- added C4: 100nF, SM0603_big, F.Cu at (144.8, 92.0)
- added C4: 100nF, SM0603_big, F.Cu at (126.2, 42.0)
- added C4: 100nF, SM0603_big, F.Cu at (114.8, 92.0)
- added C4: 100nF, SM0603_big, F.Cu at (174.8, 92.0)
- added C4: 100nF, SM0603_big, F.Cu at (186.2, 42.0)
- added C4: 100nF, SM0603_big, F.Cu at (54.8, 92.0)
- added C4: 100nF, SM0603_big, F.Cu at (66.2, 42.0)
- added C4: 10uF, SM0805_big, F.Cu at (203.0, 53.0)
- added C5: 100nF, SM0603_big, F.Cu at (209.5, 47.5)
- added C5: 100nF, SM0603_big, F.Cu at (29.5, 47.5)
- added C5: 330nF, SM0603_big, F.Cu at (61.4, 222.4)
- added C5: 330nF, SM0603_big, F.Cu at (128.4, 222.4)
- added C6: 100nF, SM0603_big, F.Cu at (217.5, 85.5)
- added C6: 100nF, SM0603_big, F.Cu at (37.5, 85.5)
- added C6: 100nF, SM0603_big, F.Cu at (61.4, 217.4)
- added C6: 100nF, SM0603_big, F.Cu at (128.4, 217.4)
- added C7: 100n, SM0603_big, F.Cu at (61.2, 336.8)
- added C7: 100n, SM0603_big, F.Cu at (128.2, 336.8)
- added C8: 100n, SM0603_big, F.Cu at (61.2, 322.8)
- added C8: 100n, SM0603_big, F.Cu at (128.2, 322.8)
- added C9: 100n, SM0603_big, F.Cu at (61.2, 308.8)
- added C9: 100n, SM0603_big, F.Cu at (128.2, 308.8)
- added D1: LED, SM0603_big, F.Cu at (204.0, 75.6)
- added D1: LED, SM0603_big, F.Cu at (24.0, 75.6)
- added D1: LED1, SM0603_big, F.Cu at (35.6, 297.8)
- added D1: LED1, SM0603_big, F.Cu at (102.6, 297.8)
- added D2: LED, SM0603_big, F.Cu at (201.6, 75.6)
- added D2: LED, SM0603_big, F.Cu at (21.6, 75.6)
- added D2: LED2, SM0603_big, F.Cu at (35.6, 300.2)
- added D2: LED2, SM0603_big, F.Cu at (102.6, 300.2)
- added D3: LED3, SM0603_big, F.Cu at (35.6, 302.6)
- added D3: LED3, SM0603_big, F.Cu at (102.6, 302.6)
- added D4: LED4, SM0603_big, F.Cu at (35.6, 305.0)
- added D4: LED4, SM0603_big, F.Cu at (102.6, 305.0)
- added D5: LED_POW, SM0603_big, F.Cu at (39.4, 257.0)
- added D5: LED_POW, SM0603_big, F.Cu at (106.4, 257.0)
- added IC1: ATMEGA88-A, TQFP32, F.Cu at (212.0, 74.0)
- added IC1: ATMEGA88-A, TQFP32, F.Cu at (32.0, 74.0)
- added IC1: ATMEGA88A-A, TQFP32, F.Cu at (38.0, 286.0)
- added IC1: ATMEGA88A-A, TQFP32, F.Cu at (105.0, 286.0)
- added J1: RJ45, RJ45_8P8_simple, F.Cu at (83.0, 98.0)
- added J1: RJ45, RJ45_8P8_simple, F.Cu at (30.0, 35.0)
- added J1: RJ45, RJ45_8P8_simple, F.Cu at (158.0, 36.0)
- added J1: RJ45, RJ45_8P8_simple, F.Cu at (210.0, 195.0)
- added J1: RJ45, RJ45_8P8_simple, F.Cu at (105.0, 133.0)
- added J1: RJ45, RJ45_8P8_simple, F.Cu at (90.0, 195.0)
- added J1: RJ45, RJ45_8P8_simple, F.Cu at (120.0, 195.0)
- added J1: RJ45, RJ45_8P8_simple, F.Cu at (135.0, 133.0)
- added J1: RJ45, RJ45_8P8_simple, F.Cu at (165.0, 133.0)
- added J1: RJ45, RJ45_8P8_simple, F.Cu at (150.0, 195.0)
- added J1: RJ45, RJ45_8P8_simple, F.Cu at (180.0, 195.0)
- added J1: RJ45, RJ45_8P8_simple, F.Cu at (98.0, 36.0)
- added J1: RJ45, RJ45_8P8_simple, F.Cu at (195.0, 133.0)
- added J1: RJ45, RJ45_8P8_simple, F.Cu at (75.0, 133.0)
- added J1: RJ45, RJ45_8P8_simple, F.Cu at (60.0, 195.0)
- added J1: RJ45_8P8C_8FACH, RJ45_8P8C_8x, F.Cu at (82.0, 282.0)
- added J1: RJ45_8P8C_8FACH, RJ45_8P8C_8x, F.Cu at (149.0, 282.0)
- added J1: RJ45, RJ45_8P8_simple, F.Cu at (45.0, 133.0)
- added J1: RJ45, RJ45_8P8_simple, F.Cu at (143.0, 98.0)
- added J1: RJ45, RJ45_8P8_simple, F.Cu at (128.0, 36.0)
- added J1: RJ45, RJ45_8P8_simple, F.Cu at (113.0, 98.0)
- added J1: RJ45, RJ45_8P8_simple, F.Cu at (173.0, 98.0)
- added J1: RJ45, RJ45_8P8_simple, F.Cu at (188.0, 36.0)
- added J1: RJ45, RJ45_8P8_simple, F.Cu at (53.0, 98.0)
- added J1: RJ45, RJ45_8P8_simple, F.Cu at (68.0, 36.0)
- added J1: RJ45, RJ45_8P8_simple, F.Cu at (210.0, 35.0)
- added K1: pow_sel, Stiftleiste_3x1, F.Cu at (33.0, 246.0)
- added K1: pow_sel, Stiftleiste_3x1, F.Cu at (100.0, 246.0)
- added P1: CONN_4, Stiftleiste_4x1, F.Cu at (201.2, 109.3)
- added P1: CONN_4, Stiftleiste_4x1, F.Cu at (48.7, 34.2)
- added P1: CONN_4, HYT271, F.Cu at (199.6, 96.7)
- added P1: CONN_4, HYT271, F.Cu at (26.6, 127.7)
- added P1: CONN_4, HYT271, F.Cu at (213.4, 127.3)
- added P1: ISP, wannenstecker_2x5_rm254, F.Cu at (210.0, 63.0)
- added P1: ISP, wannenstecker_2x5_rm254, F.Cu at (30.0, 63.0)
- added P1: UART, Stiftleiste_4x1, F.Cu at (25.0, 271.0)
- added P1: UART, Stiftleiste_4x1, F.Cu at (92.0, 271.0)
- added P2: so8, st485, F.Cu at (196.8, 109.3)
- added P2: so8, st485, F.Cu at (48.7, 29.8)
- added P2: CONN_4, Stiftleiste_4x1, F.Cu at (194.5, 96.7)
- added P2: CONN_4, Stiftleiste_4x1, F.Cu at (21.5, 127.7)
- added P2: CONN_4, Stiftleiste_4x1, F.Cu at (218.5, 127.3)
- added P2: UART, Stiftleiste_4x1, F.Cu at (215.8, 83.4)
- added P2: UART, Stiftleiste_4x1, F.Cu at (35.8, 83.4)
- added P2: Shield, m3_scheibe, F.Cu at (78.0, 218.0)
- added P2: Shield, m3_scheibe, F.Cu at (145.0, 218.0)
- added P3: CONN_4, Stiftleiste_4x1, F.Cu at (188.5, 109.3)
- added P3: CONN_4, Stiftleiste_4x1, F.Cu at (48.7, 21.5)
- added P3: i2c_pow, wannenstecker_2x3_rm254, F.Cu at (25.0, 332.5)
- added P3: i2c_pow, wannenstecker_2x3_rm254, F.Cu at (92.0, 332.5)
- added P4: i2c_chain, wannenstecker_2x3_rm254, F.Cu at (25.0, 314.5)
- added P4: i2c_chain, wannenstecker_2x3_rm254, F.Cu at (92.0, 314.5)
- added P5: 12Vin, LPV_Stiftleiste_2pol, F.Cu at (25.0, 243.0)
- added P5: 12Vin, LPV_Stiftleiste_2pol, F.Cu at (92.0, 243.0)
- added P6: HOHLBUCHSE, hohlbuchse_475_17, F.Cu at (27.0, 233.0)
- added P6: HOHLBUCHSE, hohlbuchse_475_17, F.Cu at (94.0, 233.0)
- added P7: Vccin, LPV_Stiftleiste_2pol, F.Cu at (25.0, 257.0)
- added P7: Vccin, LPV_Stiftleiste_2pol, F.Cu at (92.0, 257.0)
- added P8: ISP, wannenstecker_2x5_rm254, F.Cu at (25.0, 293.5)
- added P8: ISP, wannenstecker_2x5_rm254, F.Cu at (92.0, 293.5)
- added P9: 5Vin, LPV_Stiftleiste_2pol, F.Cu at (25.0, 250.0)
- added P9: 5Vin, LPV_Stiftleiste_2pol, F.Cu at (92.0, 250.0)
- added R1: 220, SM0603_big, F.Cu at (75.8, 76.5)
- added R1: 150, SM0805_big, F.Cu at (24.0, 71.0)
- added R1: 220, SM0603_big, F.Cu at (165.2, 57.5)
- added R1: 220, SM0603_big, F.Cu at (202.8, 173.5)
- added R1: 220, SM0603_big, F.Cu at (112.2, 154.5)
- added R1: 220, SM0603_big, F.Cu at (82.8, 173.5)
- added R1: 220, SM0603_big, F.Cu at (112.8, 173.5)
- added R1: 220, SM0603_big, F.Cu at (142.2, 154.5)
- added R1: 220, SM0603_big, F.Cu at (172.2, 154.5)
- added R1: 220, SM0603_big, F.Cu at (142.8, 173.5)
- added R1: 220, SM0603_big, F.Cu at (172.8, 173.5)
- added R1: 220, SM0603_big, F.Cu at (105.2, 57.5)
- added R1: 220, SM0603_big, F.Cu at (202.2, 154.5)
- added R1: 220, SM0603_big, F.Cu at (82.2, 154.5)
- added R1: 220, SM0603_big, F.Cu at (52.8, 173.5)
- added R1: 10k, SM0603_big, F.Cu at (33.6, 312.2)
- added R1: 10k, SM0603_big, F.Cu at (100.6, 312.2)
- added R1: 220, SM0603_big, F.Cu at (52.2, 154.5)
- added R1: 220, SM0603_big, F.Cu at (135.8, 76.5)
- added R1: 220, SM0603_big, F.Cu at (135.2, 57.5)
- added R1: 220, SM0603_big, F.Cu at (105.8, 76.5)
- added R1: 220, SM0603_big, F.Cu at (165.8, 76.5)
- added R1: 220, SM0603_big, F.Cu at (195.2, 57.5)
- added R1: 220, SM0603_big, F.Cu at (45.8, 76.5)
- added R1: 220, SM0603_big, F.Cu at (75.2, 57.5)
- added R1: 150, SM0805_big, F.Cu at (204.0, 71.0)
- added R10: 22k, SM0603_big, F.Cu at (54.2, 329.8)
- added R10: 22k, SM0603_big, F.Cu at (121.2, 329.8)
- added R11: 22k, SM0603_big, F.Cu at (54.2, 315.8)
- added R11: 22k, SM0603_big, F.Cu at (121.2, 315.8)
- added R12: 22k, SM0603_big, F.Cu at (54.2, 301.8)
- added R12: 22k, SM0603_big, F.Cu at (121.2, 301.8)
- added R13: 22k, SM0603_big, F.Cu at (54.2, 287.8)
- added R13: 22k, SM0603_big, F.Cu at (121.2, 287.8)
- added R14: 22k, SM0603_big, F.Cu at (54.2, 339.8)
- added R14: 22k, SM0603_big, F.Cu at (121.2, 339.8)
- added R15: 22k, SM0603_big, F.Cu at (54.2, 325.8)
- added R15: 22k, SM0603_big, F.Cu at (121.2, 325.8)
- added R16: 22k, SM0603_big, F.Cu at (54.2, 311.8)
- added R16: 22k, SM0603_big, F.Cu at (121.2, 311.8)
- added R17: 22k, SM0603_big, F.Cu at (54.2, 297.8)
- added R17: 22k, SM0603_big, F.Cu at (121.2, 297.8)
- added R18: 120, SM0603_big, F.Cu at (61.2, 332.8)
- added R18: 120, SM0603_big, F.Cu at (128.2, 332.8)
- added R19: 120, SM0603_big, F.Cu at (61.2, 318.8)
- added R19: 120, SM0603_big, F.Cu at (128.2, 318.8)
- added R2: 22k, SM0603_big, F.Cu at (85.5, 88.2)
- added R2: 150, SM0805_big, F.Cu at (21.6, 71.0)
- added R2: 22k, SM0603_big, F.Cu at (155.5, 45.8)
- added R2: 22k, SM0603_big, F.Cu at (212.5, 185.2)
- added R2: 22k, SM0603_big, F.Cu at (102.5, 142.8)
- added R2: 22k, SM0603_big, F.Cu at (92.5, 185.2)
- added R2: 22k, SM0603_big, F.Cu at (122.5, 185.2)
- added R2: 22k, SM0603_big, F.Cu at (132.5, 142.8)
- added R2: 22k, SM0603_big, F.Cu at (162.5, 142.8)
- added R2: 22k, SM0603_big, F.Cu at (152.5, 185.2)
- added R2: 22k, SM0603_big, F.Cu at (182.5, 185.2)
- added R2: 22k, SM0603_big, F.Cu at (95.5, 45.8)
- added R2: 22k, SM0603_big, F.Cu at (192.5, 142.8)
- added R2: 22k, SM0603_big, F.Cu at (72.5, 142.8)
- added R2: 22k, SM0603_big, F.Cu at (62.5, 185.2)
- added R2: 150, SM0805_big, F.Cu at (40.6, 297.8)
- added R2: 150, SM0805_big, F.Cu at (107.6, 297.8)
- added R2: 22k, SM0603_big, F.Cu at (42.5, 142.8)
- added R2: 22k, SM0603_big, F.Cu at (145.5, 88.2)
- added R2: 22k, SM0603_big, F.Cu at (125.5, 45.8)
- added R2: 22k, SM0603_big, F.Cu at (115.5, 88.2)
- added R2: 22k, SM0603_big, F.Cu at (175.5, 88.2)
- added R2: 22k, SM0603_big, F.Cu at (185.5, 45.8)
- added R2: 22k, SM0603_big, F.Cu at (55.5, 88.2)
- added R2: 22k, SM0603_big, F.Cu at (65.5, 45.8)
- added R2: 150, SM0805_big, F.Cu at (201.6, 71.0)
- added R20: 120, SM0603_big, F.Cu at (61.2, 304.6)
- added R20: 120, SM0603_big, F.Cu at (128.2, 304.6)
- added R21: 120, SM0603_big, F.Cu at (61.2, 290.8)
- added R21: 120, SM0603_big, F.Cu at (128.2, 290.8)
- added R22: 22k, SM0603_big, F.Cu at (54.2, 273.8)
- added R22: 22k, SM0603_big, F.Cu at (121.2, 273.8)
- added R23: 22k, SM0603_big, F.Cu at (54.2, 259.8)
- added R23: 22k, SM0603_big, F.Cu at (121.2, 259.8)
- added R24: 22k, SM0603_big, F.Cu at (54.2, 245.8)
- added R24: 22k, SM0603_big, F.Cu at (121.2, 245.8)
- added R25: 22k, SM0603_big, F.Cu at (54.2, 231.8)
- added R25: 22k, SM0603_big, F.Cu at (121.2, 231.8)
- added R26: 22k, SM0603_big, F.Cu at (54.2, 283.8)
- added R26: 22k, SM0603_big, F.Cu at (121.2, 283.8)
- added R27: 22k, SM0603_big, F.Cu at (54.2, 269.8)
- added R27: 22k, SM0603_big, F.Cu at (121.2, 269.8)
- added R28: 22k, SM0603_big, F.Cu at (54.2, 255.8)
- added R28: 22k, SM0603_big, F.Cu at (121.2, 255.8)
- added R29: 22k, SM0603_big, F.Cu at (54.2, 241.8)
- added R29: 22k, SM0603_big, F.Cu at (121.2, 241.8)
- added R3: 22k, SM0603_big, F.Cu at (90.5, 88.2)
- added R3: 10k, SM0603_big, F.Cu at (36.0, 56.3)
- added R3: 22k, SM0603_big, F.Cu at (150.5, 45.8)
- added R3: 22k, SM0603_big, F.Cu at (217.5, 185.2)
- added R3: 22k, SM0603_big, F.Cu at (97.5, 142.8)
- added R3: 22k, SM0603_big, F.Cu at (97.5, 185.2)
- added R3: 22k, SM0603_big, F.Cu at (127.5, 185.2)
- added R3: 22k, SM0603_big, F.Cu at (127.5, 142.8)
- added R3: 22k, SM0603_big, F.Cu at (157.5, 142.8)
- added R3: 22k, SM0603_big, F.Cu at (157.5, 185.2)
- added R3: 22k, SM0603_big, F.Cu at (187.5, 185.2)
- added R3: 22k, SM0603_big, F.Cu at (90.5, 45.8)
- added R3: 22k, SM0603_big, F.Cu at (187.5, 142.8)
- added R3: 22k, SM0603_big, F.Cu at (67.5, 142.8)
- added R3: 22k, SM0603_big, F.Cu at (67.5, 185.2)
- added R3: 150, SM0805_big, F.Cu at (40.6, 300.2)
- added R3: 150, SM0805_big, F.Cu at (107.6, 300.2)
- added R3: 22k, SM0603_big, F.Cu at (37.5, 142.8)
- added R3: 22k, SM0603_big, F.Cu at (150.5, 88.2)
- added R3: 22k, SM0603_big, F.Cu at (120.5, 45.8)
- added R3: 22k, SM0603_big, F.Cu at (120.5, 88.2)
- added R3: 22k, SM0603_big, F.Cu at (180.5, 88.2)
- added R3: 22k, SM0603_big, F.Cu at (180.5, 45.8)
- added R3: 22k, SM0603_big, F.Cu at (60.5, 88.2)
- added R3: 22k, SM0603_big, F.Cu at (60.5, 45.8)
- added R3: 10k, SM0603_big, F.Cu at (216.0, 56.3)
- added R30: 120, SM0603_big, F.Cu at (61.2, 276.8)
- added R30: 120, SM0603_big, F.Cu at (128.2, 276.8)
- added R31: 120, SM0603_big, F.Cu at (61.2, 262.8)
- added R31: 120, SM0603_big, F.Cu at (128.2, 262.8)
- added R32: 120, SM0603_big, F.Cu at (61.2, 248.8)
- added R32: 120, SM0603_big, F.Cu at (128.2, 248.8)
- added R33: 120, SM0603_big, F.Cu at (61.2, 234.8)
- added R33: 120, SM0603_big, F.Cu at (128.2, 234.8)
- added R34: 0, SM0805_big, F.Cu at (68.2, 218.0)
- added R34: 0, SM0805_big, F.Cu at (135.2, 218.0)
- added R4: 120, SM0603_big, F.Cu at (88.8, 92.0)
- added R4: 22k, SM0603_big, F.Cu at (36.0, 49.8)
- added R4: 120, SM0603_big, F.Cu at (152.2, 42.0)
- added R4: 120, SM0603_big, F.Cu at (215.8, 189.0)
- added R4: 120, SM0603_big, F.Cu at (99.2, 139.0)
- added R4: 120, SM0603_big, F.Cu at (95.8, 189.0)
- added R4: 120, SM0603_big, F.Cu at (125.8, 189.0)
- added R4: 120, SM0603_big, F.Cu at (129.2, 139.0)
- added R4: 120, SM0603_big, F.Cu at (159.2, 139.0)
- added R4: 120, SM0603_big, F.Cu at (155.8, 189.0)
- added R4: 120, SM0603_big, F.Cu at (185.8, 189.0)
- added R4: 120, SM0603_big, F.Cu at (92.2, 42.0)
- added R4: 120, SM0603_big, F.Cu at (189.2, 139.0)
- added R4: 120, SM0603_big, F.Cu at (69.2, 139.0)
- added R4: 120, SM0603_big, F.Cu at (65.8, 189.0)
- added R4: 150, SM0805_big, F.Cu at (40.6, 302.6)
- added R4: 150, SM0805_big, F.Cu at (107.6, 302.6)
- added R4: 120, SM0603_big, F.Cu at (39.2, 139.0)
- added R4: 120, SM0603_big, F.Cu at (148.8, 92.0)
- added R4: 120, SM0603_big, F.Cu at (122.2, 42.0)
- added R4: 120, SM0603_big, F.Cu at (118.8, 92.0)
- added R4: 120, SM0603_big, F.Cu at (178.8, 92.0)
- added R4: 120, SM0603_big, F.Cu at (182.2, 42.0)
- added R4: 120, SM0603_big, F.Cu at (58.8, 92.0)
- added R4: 120, SM0603_big, F.Cu at (62.2, 42.0)
- added R4: 22k, SM0603_big, F.Cu at (216.0, 49.8)
- added R5: 22k, SM0603_big, F.Cu at (203.0, 50.0)
- added R5: 22k, SM0603_big, F.Cu at (23.0, 50.0)
- added R5: 150, SM0805_big, F.Cu at (40.6, 305.0)
- added R5: 150, SM0805_big, F.Cu at (107.6, 305.0)
- added R6: 120, SM0603_big, F.Cu at (205.5, 47.5)
- added R6: 120, SM0603_big, F.Cu at (25.5, 47.5)
- added R6: 2k2, SM0603_big, F.Cu at (39.6, 318.4)
- added R6: 2k2, SM0603_big, F.Cu at (106.6, 318.4)
- added R7: 2k2, SM0603_big, F.Cu at (209.4, 90.2)
- added R7: 2k2, SM0603_big, F.Cu at (29.4, 90.2)
- added R7: 2k2, SM0603_big, F.Cu at (39.6, 328.4)
- added R7: 2k2, SM0603_big, F.Cu at (106.6, 328.4)
- added R8: 2k2, SM0603_big, F.Cu at (213.2, 90.2)
- added R8: 2k2, SM0603_big, F.Cu at (33.2, 90.2)
- added R8: 150, SM0805_big, F.Cu at (37.0, 257.0)
- added R8: 150, SM0805_big, F.Cu at (104.0, 257.0)
- added R9: 10k, SM0603_big, F.Cu at (50.0, 285.0)
- added R9: 10k, SM0603_big, F.Cu at (117.0, 285.0)
- added SW1: SW_RESET, Taster_6mm, F.Cu at (204.0, 41.5)
- added SW1: SW_RESET, Taster_6mm, F.Cu at (24.0, 41.5)
- added SW1: SW1, Taster_6mm, F.Cu at (38.0, 312.2)
- added SW1: SW1, Taster_6mm, F.Cu at (105.0, 312.2)
- added SW2: SCHALTER_2POL, DIP_Schalter_2pol, F.Cu at (36.8, 323.4)
- added SW2: SCHALTER_2POL, DIP_Schalter_2pol, F.Cu at (103.8, 323.4)
- added SW3: SW_RESET, Taster_6mm, F.Cu at (38.0, 334.6)
- added SW3: SW_RESET, Taster_6mm, F.Cu at (105.0, 334.6)
- added U1: TSIC50XF, Tsic_TO92, F.Cu at (83.0, 41.5)
- added U1: ST485, st485, F.Cu at (30.0, 52.0)
- added U1: TSIC50XF, Tsic_TO92, F.Cu at (158.0, 92.5)
- added U1: TSIC50XF, Tsic_TO92, F.Cu at (210.0, 138.5)
- added U1: TSIC50XF, Tsic_TO92, F.Cu at (105.0, 189.5)
- added U1: TSIC50XF, Tsic_TO92, F.Cu at (90.0, 138.5)
- added U1: TSIC50XF, Tsic_TO92, F.Cu at (120.0, 138.5)
- added U1: TSIC50XF, Tsic_TO92, F.Cu at (135.0, 189.5)
- added U1: TSIC50XF, Tsic_TO92, F.Cu at (165.0, 189.5)
- added U1: TSIC50XF, Tsic_TO92, F.Cu at (150.0, 138.5)
- added U1: TSIC50XF, Tsic_TO92, F.Cu at (180.0, 138.5)
- added U1: TSIC50XF, Tsic_TO92, F.Cu at (98.0, 92.5)
- added U1: TSIC50XF, Tsic_TO92, F.Cu at (195.0, 189.5)
- added U1: TSIC50XF, Tsic_TO92, F.Cu at (75.0, 189.5)
- added U1: TSIC50XF, Tsic_TO92, F.Cu at (60.0, 138.5)
- added U1: LM7805, lm7805_lying, F.Cu at (39.0, 220.0)
- added U1: LM7805, lm7805_lying, F.Cu at (106.0, 220.0)
- added U1: TSIC50XF, Tsic_TO92, F.Cu at (45.0, 189.5)
- added U1: TSIC50XF, Tsic_TO92, F.Cu at (143.0, 41.5)
- added U1: TSIC50XF, Tsic_TO92, F.Cu at (128.0, 92.5)
- added U1: TSIC50XF, Tsic_TO92, F.Cu at (113.0, 41.5)
- added U1: TSIC50XF, Tsic_TO92, F.Cu at (173.0, 41.5)
- added U1: TSIC50XF, Tsic_TO92, F.Cu at (188.0, 92.5)
- added U1: TSIC50XF, Tsic_TO92, F.Cu at (53.0, 41.5)
- added U1: TSIC50XF, Tsic_TO92, F.Cu at (68.0, 92.5)
- added U1: ST485, st485, F.Cu at (210.0, 52.0)
- added U2: ST485, st485, F.Cu at (83.0, 82.2)
- added U2: HYT271, HYT271, F.Cu at (30.0, 118.5)
- added U2: ST485, st485, F.Cu at (158.0, 51.8)
- added U2: ST485, st485, F.Cu at (210.0, 179.2)
- added U2: ST485, st485, F.Cu at (105.0, 148.8)
- added U2: ST485, st485, F.Cu at (90.0, 179.2)
- added U2: ST485, st485, F.Cu at (120.0, 179.2)
- added U2: ST485, st485, F.Cu at (135.0, 148.8)
- added U2: ST485, st485, F.Cu at (165.0, 148.8)
- added U2: ST485, st485, F.Cu at (150.0, 179.2)
- added U2: ST485, st485, F.Cu at (180.0, 179.2)
- added U2: ST485, st485, F.Cu at (98.0, 51.8)
- added U2: ST485, st485, F.Cu at (195.0, 148.8)
- added U2: ST485, st485, F.Cu at (75.0, 148.8)
- added U2: ST485, st485, F.Cu at (60.0, 179.2)
- added U2: ST485, st485, F.Cu at (53.2, 334.8)
- added U2: ST485, st485, F.Cu at (120.2, 334.8)
- added U2: ST485, st485, F.Cu at (45.0, 148.8)
- added U2: ST485, st485, F.Cu at (143.0, 82.2)
- added U2: ST485, st485, F.Cu at (128.0, 51.8)
- added U2: ST485, st485, F.Cu at (113.0, 82.2)
- added U2: ST485, st485, F.Cu at (173.0, 82.2)
- added U2: ST485, st485, F.Cu at (188.0, 51.8)
- added U2: ST485, st485, F.Cu at (53.0, 82.2)
- added U2: ST485, st485, F.Cu at (68.0, 51.8)
- added U2: HYT271, HYT271, F.Cu at (210.0, 118.5)
- added U3: ST485, st485, F.Cu at (53.2, 320.8)
- added U3: ST485, st485, F.Cu at (120.2, 320.8)
- added U4: ST485, st485, F.Cu at (53.2, 306.8)
- added U4: ST485, st485, F.Cu at (120.2, 306.8)
- added U5: ST485, st485, F.Cu at (53.2, 292.8)
- added U5: ST485, st485, F.Cu at (120.2, 292.8)
- added U6: ST485, st485, F.Cu at (53.2, 278.8)
- added U6: ST485, st485, F.Cu at (120.2, 278.8)
- added U7: ST485, st485, F.Cu at (53.2, 264.8)
- added U7: ST485, st485, F.Cu at (120.2, 264.8)
- added U8: ST485, st485, F.Cu at (53.2, 250.8)
- added U8: ST485, st485, F.Cu at (120.2, 250.8)
- added U9: ST485, st485, F.Cu at (53.2, 236.8)
- added U9: ST485, st485, F.Cu at (120.2, 236.8)
- added X1: 20MHz, HC-49_quarz_big, F.Cu at (35.6, 276.3)
- added X1: 20MHz, HC-49_quarz_big, F.Cu at (102.6, 276.3)
- added m3_loch: VAL**, m3_loch, F.Cu at (88.0, 73.8)
- added m3_loch: VAL**, m3_loch, F.Cu at (168.0, 89.8)
- added m3_loch: VAL**, m3_loch, F.Cu at (183.0, 60.2)
- added m3_loch: VAL**, m3_loch, F.Cu at (193.0, 44.2)
- added m3_loch: VAL**, m3_loch, F.Cu at (58.0, 73.8)
- added m3_loch: VAL**, m3_loch, F.Cu at (48.0, 89.8)
- added m3_loch: VAL**, m3_loch, F.Cu at (63.0, 60.2)
- added m3_loch: VAL**, m3_loch, F.Cu at (73.0, 44.2)
- added m3_loch: VAL**, m3_loch, F.Cu at (215.0, 42.5)
- added m3_loch: VAL**, m3_loch, F.Cu at (205.0, 84.0)
- added m3_loch: VAL**, m3_loch, F.Cu at (35.0, 42.5)
- added m3_loch: VAL**, m3_loch, F.Cu at (78.0, 89.8)
- added m3_loch: VAL**, m3_loch, F.Cu at (25.0, 84.0)
- added m3_loch: VAL**, m3_loch, F.Cu at (163.0, 44.2)
- added m3_loch: VAL**, m3_loch, F.Cu at (153.0, 60.2)
- added m3_loch: VAL**, m3_loch, F.Cu at (215.0, 170.8)
- added m3_loch: VAL**, m3_loch, F.Cu at (205.0, 186.8)
- added m3_loch: VAL**, m3_loch, F.Cu at (100.0, 157.2)
- added m3_loch: VAL**, m3_loch, F.Cu at (110.0, 141.2)
- added m3_loch: VAL**, m3_loch, F.Cu at (85.0, 186.8)
- added m3_loch: VAL**, m3_loch, F.Cu at (95.0, 170.8)
- added m3_loch: VAL**, m3_loch, F.Cu at (125.0, 170.8)
- added m3_loch: VAL**, m3_loch, F.Cu at (93.0, 60.2)
- added m3_loch: VAL**, m3_loch, F.Cu at (115.0, 186.8)
- added m3_loch: VAL**, m3_loch, F.Cu at (140.0, 141.2)
- added m3_loch: VAL**, m3_loch, F.Cu at (130.0, 157.2)
- added m3_loch: VAL**, m3_loch, F.Cu at (160.0, 157.2)
- added m3_loch: VAL**, m3_loch, F.Cu at (170.0, 141.2)
- added m3_loch: VAL**, m3_loch, F.Cu at (145.0, 186.8)
- added m3_loch: VAL**, m3_loch, F.Cu at (155.0, 170.8)
- added m3_loch: VAL**, m3_loch, F.Cu at (185.0, 170.8)
- added m3_loch: VAL**, m3_loch, F.Cu at (175.0, 186.8)
- added m3_loch: VAL**, m3_loch, F.Cu at (200.0, 141.2)
- added m3_loch: VAL**, m3_loch, F.Cu at (103.0, 44.2)
- added m3_loch: VAL**, m3_loch, F.Cu at (190.0, 157.2)
- added m3_loch: VAL**, m3_loch, F.Cu at (70.0, 157.2)
- added m3_loch: VAL**, m3_loch, F.Cu at (80.0, 141.2)
- added m3_loch: VAL**, m3_loch, F.Cu at (55.0, 186.8)
- added m3_loch: VAL**, m3_loch, F.Cu at (65.0, 170.8)
- added m3_loch: VAL**, m3_loch, F.Cu at (26.0, 218.0)
- added m3_loch: VAL**, m3_loch, F.Cu at (26.0, 345.0)
- added m3_loch: VAL**, m3_loch, F.Cu at (78.0, 345.0)
- added m3_loch: VAL**, m3_loch, F.Cu at (145.0, 345.0)
- added m3_loch: VAL**, m3_loch, F.Cu at (93.0, 345.0)
- added m3_loch: VAL**, m3_loch, F.Cu at (133.0, 44.2)
- added m3_loch: VAL**, m3_loch, F.Cu at (93.0, 218.0)
- added m3_loch: VAL**, m3_loch, F.Cu at (50.0, 141.2)
- added m3_loch: VAL**, m3_loch, F.Cu at (40.0, 157.2)
- added m3_loch: VAL**, m3_loch, F.Cu at (138.0, 89.8)
- added m3_loch: VAL**, m3_loch, F.Cu at (148.0, 73.8)
- added m3_loch: VAL**, m3_loch, F.Cu at (123.0, 60.2)
- added m3_loch: VAL**, m3_loch, F.Cu at (108.0, 89.8)
- added m3_loch: VAL**, m3_loch, F.Cu at (118.0, 73.8)
- added m3_loch: VAL**, m3_loch, F.Cu at (178.0, 73.8)
- moved C1 288.4 mm to (22.8, 169.5)
- moved C2 288.4 mm to (37.2, 178.2)
- moved C3 288.4 mm to (37.2, 181.8)
- moved C4 288.4 mm to (31.8, 189.0)
- moved J1 288.4 mm to (30.0, 195.0)
- moved R1 288.4 mm to (22.8, 173.5)
- moved R2 288.4 mm to (32.5, 185.2)
- moved R3 288.4 mm to (37.5, 185.2)
- moved R4 288.4 mm to (35.8, 189.0)
- moved U1 288.4 mm to (30.0, 138.5)
- moved U2 288.4 mm to (30.0, 179.2)
- moved m3_loch 288.4 mm to (35.0, 170.8)
- moved m3_loch 288.4 mm to (25.0, 186.8)
- moved m3_loch 257.8 mm to (161.0, 345.0), turned to 0 degrees
- moved m3_loch 251.5 mm to (213.0, 345.0), turned to 0 degrees
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Routing:
- net GND: track 1927.7 -> 5935.8 mm, vias 23 -> 65
- net VCC: track 1267.8 -> 3394.3 mm, vias 19 -> 86
- net N-000007: track 195.7 -> 1065.2 mm
- net N-0000010: track 161.4 -> 908.5 mm
- net /zb: track 155.1 -> 628.7 mm
- net /za: track 154.8 -> 613.0 mm
- net /Vi2c: track 146.2 -> 438.6 mm, vias 1 -> 3
- net /RESET: track 218.5 -> 432.3 mm, vias 6 -> 10
- net /Vreg: track 65.1 -> 195.3 mm
- net /ZAC_08: track 63.7 -> 191.1 mm
- net +12V: track 53.8 -> 161.3 mm
- net /MOSI: track 73.2 -> 172.4 mm, vias 4 -> 8
- net /TX: track 60.8 -> 157.9 mm, vias 2 -> 6
- net /ZAC_01: track 47.2 -> 141.6 mm
- net /RX: track 66.5 -> 159.2 mm, vias 2 -> 6
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Other:
- board size 310 x 251.6 mm -> 200 x 330 mm
- rule pad_to_mask_clearance: 0.15 -> 0
- board text added: "v1.1"
